File: CONN.sch (KiCad schematic (older format))
At the start: 1 part, among them J3 174518-7

Commit message: restart a third time
Parts:
- removed J3: 174518-7, speeduino_connector_automotive:174518-7, symbol speeduino_connector_automotive:174518-7
- added H1, H2, H3, H4: MountingHole_Pad, MountingHole:MountingHole_5mm_Pad_TopOnly, symbol Mechanical:MountingHole_Pad
- added J1: Delphi_Sicma_24, speeduino_connector_automotive:Delphi_Sicma_24_Black, symbol speeduino_connector_automotive:Delphi_Sicma_24
Connections:
- net labels removed: 12v-SW, 5v, AC-FAN-OUT, AC-IN, AC-OUT, CAM-IN, CLT-IN, CLUTCH-IN, CRANK-IN, FAN-OUT, FP-OUT, IAT-IN, IDLE-OUT, IGN-1-OUT, IGN-2-OUT, INJ-1, INJ-2, INJ-3, INJ-4, O2-IN, ST_SIG, TACH-OUT, TPS-IN, VBAT, VSS-IN
- wire segments 0 -> 9
Other:
- note removed: "CYL-1-4\n"
- note removed: "CYL-2-3"
Changed lines of the file:
@@
 $Descr A4 11693 8268
 encoding utf-8
-Sheet 10 10
+Sheet 10 11
 Title ""
 Date ""
@@
 $EndDescr
 $Comp
-L speeduino_connector_automotive:174518-7 J3
-U 1 1 5EEDF806
-P 4600 2350
-F 0 "J3" H 5100 2615 50  0000 C CNN
-F 1 "174518-7" H 5100 2524 50  0000 C CNN
-F 2 "speeduino_connector_automotive:174518-7" H 5450 2450 50  0001 L CNN
-F 3 "https://componentsearchengine.com/Datasheets/1/174518-7.pdf" H 5450 2350 50  0001 L CNN
-F 4 "Conn Wire to Board RCP 64 POS Solder RA Thru-Hole Automotive Tube" H 5450 2250 50  0001 L CNN "Description"
-F 5 "21.9" H 5450 2150 50  0001 L CNN "Height"
-F 6 "571-174518-7" H 5450 2050 50  0001 L CNN "Mouser Part Number"
-F 7 "https://www.mouser.com/Search/Refine.aspx?Keyword=571-174518-7" H 5450 1950 50  0001 L CNN "Mouser Price/Stock"
-F 8 "TE Connectivity" H 5450 1850 50  0001 L CNN "Manufacturer_Name"
-F 9 "174518-7" H 5450 1750 50  0001 L CNN "Manufacturer_Part_Number"
-	1    4600 2350
+L Mechanical:MountingHole_Pad H1
+U 1 1 6036F829
+P 7100 4100
+F 0 "H1" V 7054 4250 50  0000 L CNN
+F 1 "MountingHole_Pad" V 7145 4250 50  0000 L CNN
+F 2 "MountingHole:MountingHole_5mm_Pad_TopOnly" H 7100 4100 50  0001 C CNN
+F 3 "~" H 7100 4100 50  0001 C CNN
+	1    7100 4100
 	1    0    0    -1
 $EndComp
-Text HLabel 5600 2950 2    50   Output ~ 0
-VBAT
-Text HLabel 5600 3050 2    50   Output ~ 0
-12v-SW
-Text HLabel 4600 5450 0    50   Output ~ 0
-IGN-2-OUT
-Text Notes 3750 5500 0    50   ~ 0
-CYL-2-3
-Text HLabel 4600 5050 0    50   Output ~ 0
-IGN-1-OUT
-Text Notes 3750 5100 0    50   ~ 0
-CYL-1-4\n
-Text HLabel 5600 5350 2    50   Output ~ 0
-AC-OUT
-Text HLabel 4600 5350 0    50   Output ~ 0
-FAN-OUT
-Text HLabel 5600 2850 2    50   Output ~ 0
-CLUTCH-IN
-Text HLabel 5600 4750 2    50   Output ~ 0
-AC-IN
-Text HLabel 5600 4850 2    50   Output ~ 0
-VSS-IN
-Text HLabel 4600 2350 0    50   Output ~ 0
-INJ-3
-Text HLabel 5600 2450 2    50   Output ~ 0
-INJ-4
-Text HLabel 5600 2350 2    50   Output ~ 0
-IDLE-OUT
-Text HLabel 4600 2450 0    50   Output ~ 0
-INJ-1
-Text HLabel 5600 2550 2    50   Output ~ 0
-INJ-2
-Text HLabel 4600 3150 0    50   Output ~ 0
-AC-FAN-OUT
-Text HLabel 4600 3550 0    50   Output ~ 0
-FP-OUT
-Text HLabel 5600 3150 2    50   Output ~ 0
-CLT-IN
-Text HLabel 5600 3250 2    50   Output ~ 0
-TPS-IN
-Text HLabel 4600 3350 0    50   Output ~ 0
-5v
-Text HLabel 5600 3350 2    50   Output ~ 0
-TACH-OUT
-Text HLabel 4600 3450 0    50   Output ~ 0
-CAM-IN
-Text HLabel 5600 3450 2    50   Output ~ 0
-CRANK-IN
-Text HLabel 4600 3650 0    50   Output ~ 0
-IAT-IN
-Text HLabel 4600 3750 0    50   Output ~ 0
-O2-IN
 $Comp
-L power:GND #PWR0154
-U 1 1 5EEEB3A2
-P 4600 2650
-F 0 "#PWR0154" H 4600 2400 50  0001 C CNN
-F 1 "GND" V 4605 2522 50  0000 R CNN
-F 2 "" H 4600 2650 50  0001 C CNN
-F 3 "" H 4600 2650 50  0001 C CNN
-	1    4600 2650
-	0    1    1    0
+L Mechanical:MountingHole_Pad H2
+U 1 1 60370D30
+P 7300 4100
+F 0 "H2" V 7254 4250 50  0000 L CNN
+F 1 "MountingHole_Pad" V 7345 4250 50  0000 L CNN
+F 2 "MountingHole:MountingHole_5mm_Pad_TopOnly" H 7300 4100 50  0001 C CNN
+F 3 "~" H 7300 4100 50  0001 C CNN
+	1    7300 4100
+	1    0    0    -1
 $EndComp
 $Comp
-L power:GND #PWR0155
-U 1 1 5EEEB4BB
-P 4600 2750
-F 0 "#PWR0155" H 4600 2500 50  0001 C CNN
-F 1 "GND" V 4605 2622 50  0000 R CNN
-F 2 "" H 4600 2750 50  0001 C CNN
-F 3 "" H 4600 2750 50  0001 C CNN
-	1    4600 2750
-	0    1    1    0
+L Mechanical:MountingHole_Pad H3
+U 1 1 6037123A
+P 7500 4100
+F 0 "H3" V 7454 4250 50  0000 L CNN
+F 1 "MountingHole_Pad" V 7545 4250 50  0000 L CNN
+F 2 "MountingHole:MountingHole_5mm_Pad_TopOnly" H 7500 4100 50  0001 C CNN
+F 3 "~" H 7500 4100 50  0001 C CNN
+	1    7500 4100
+	1    0    0    -1
 $EndComp
 $Comp
-L power:GND #PWR0156
-U 1 1 5EEEB674
-P 5600 2650
-F 0 "#PWR0156" H 5600 2400 50  0001 C CNN
-F 1 "GND" V 5605 2522 50  0000 R CNN
-F 2 "" H 5600 2650 50  0001 C CNN
-F 3 "" H 5600 2650 50  0001 C CNN
-	1    5600 2650
-	0    -1   -1   0
+L Mechanical:MountingHole_Pad H4
+U 1 1 6037162A
+P 7700 4100
+F 0 "H4" V 7654 4250 50  0000 L CNN
+F 1 "MountingHole_Pad" V 7745 4250 50  0000 L CNN
+F 2 "MountingHole:MountingHole_5mm_Pad_TopOnly" H 7700 4100 50  0001 C CNN
+F 3 "~" H 7700 4100 50  0001 C CNN
+	1    7700 4100
+	1    0    0    -1
 $EndComp
 $Comp
-L power:GND #PWR0157
-U 1 1 5EEEC019
-P 5600 2750
-F 0 "#PWR0157" H 5600 2500 50  0001 C CNN
-F 1 "GND" V 5605 2622 50  0000 R CNN
-F 2 "" H 5600 2750 50  0001 C CNN
-F 3 "" H 5600 2750 50  0001 C CNN
-	1    5600 2750
-	0    -1   -1   0
+L power:GND #PWR0158
+U 1 1 60376F19
+P 7400 4400
+F 0 "#PWR0158" H 7400 4150 50  0001 C CNN
+F 1 "GND" H 7405 4227 50  0000 C CNN
+F 2 "" H 7400 4400 50  0001 C CNN
+F 3 "" H 7400 4400 50  0001 C CNN
+	1    7400 4400
+	1    0    0    -1
 $EndComp
-Text HLabel 4600 2950 0    50   Output ~ 0
-ST_SIG
+Wire Wire Line
+	7100 4200 7100 4300
+Wire Wire Line
+	7100 4300 7300 4300
+Wire Wire Line
+	7400 4300 7400 4400
+Wire Wire Line
+	7700 4200 7700 4300
+Wire Wire Line
+	7700 4300 7500 4300
+Connection ~ 7400 4300
+Wire Wire Line
+	7300 4200 7300 4300
+Connection ~ 7300 4300
+Wire Wire Line
+	7300 4300 7400 4300
+Wire Wire Line
+	7500 4200 7500 4300
+Connection ~ 7500 4300
+Wire Wire Line
+	7500 4300 7400 4300
+$Comp
+L speeduino_connector_automotive:Delphi_Sicma_24 J1
+U 1 1 607DEB42
+P 2100 1900
+F 0 "J1" H 2100 2565 50  0000 C CNN
+F 1 "Delphi_Sicma_24" H 2100 2474 50  0000 C CNN
+F 2 "speeduino_connector_automotive:Delphi_Sicma_24_Black" H 2100 1900 50  0001 C CNN
+F 3 "" H 2100 1900 50  0001 C CNN
+	1    2100 1900
+	1    0    0    -1
+$EndComp
 $EndSCHEMATC
