File: Power+Reset.sch (KiCad schematic (older format))
At the start: 25 parts

Commit message: Starting on layout
Parts:
- removed SW?: SW_Push_DPDT, symbol Switch:SW_Push_DPDT
- added SW1: MLL1200S, mll1200s:SW_MLL1200S, symbol mll1200s:MLL1200S
- C28: renamed from C?; footprint (none) -> Capacitor_SMD:C_0805_2012Metric_Pad1.15x1.40mm_HandSolder; DIGIKEY (none) -> 311-1133-1-ND; LCSC_FP (none) -> 0803; LCSC_PN (none) -> C1779
- C29: renamed from C?; footprint (none) -> Capacitor_SMD:C_0805_2012Metric_Pad1.15x1.40mm_HandSolder; DIGIKEY (none) -> 1276-1047-1-ND; LCSC_FP (none) -> 0805; LCSC_PN (none) -> C1804
- D21: renamed from D?; footprint (none) -> Diode_SMD:D_SOD-323_HandSoldering; DIGIKEY (none) -> B0540WSDICT-ND; LCSC_FP (none) -> SOD-323; LCSC_PN (none) -> C98664
- R59, R60, R61: renamed from R?; footprint (none) -> Resistor_SMD:R_0603_1608Metric_Pad1.05x0.95mm_HandSolder
- gave numbers to parts that had none: 18
Connections:
- wire segments 75 -> 72
Other:
- moved on the sheet: C28, C29, R61

Commit message: restart a third time
Parts:
- C20, C22, C28, C29: footprint Capacitor_SMD:C_0805_2012Metric_Pad1.15x1.40mm_HandSolder -> Capacitor_SMD:C_0805_2012Metric_Pad1.18x1.45mm_HandSolder
- C21, C24, C25: footprint Capacitor_SMD:C_1206_3216Metric_Pad1.42x1.75mm_HandSolder -> Capacitor_SMD:C_1206_3216Metric_Pad1.33x1.80mm_HandSolder
- D17: value 1N4007 -> 1N4007W; footprint Diode_THT:D_DO-41_SOD81_P10.16mm_Horizontal -> Diode_SMD:D_SOD-123; DIGIKEY (none) -> S1MB-FDITR-ND; LCSC_FP (none) -> SOD-123; LCSC_PN (none) -> C108803
- D18: value 1N5818 -> B5818W-TP; footprint Diode_THT:D_DO-41_SOD81_P10.16mm_Horizontal -> Diode_SMD:D_SOD-123; DIGIKEY 1N5818-TPCT-ND -> B5818W-TPMSCT-ND; LCSC_FP (none) -> SOD-123_1.6x2.6; LCSC_PN (none) -> C183502; MOUSER 833-1N5818-TP -> (none)
- D19, D20: value 1N5919BG -> ZMM5V6; footprint Diode_THT:D_DO-41_SOD81_P7.62mm_Horizontal -> Diode_SMD:D_MiniMELF; DIGIKEY 1N5919BGOS-ND -> (none); LCSC_FP (none) -> LL-34; LCSC_PN (none) -> C8062; MOUSER 863-1N5919BG -> (none)
- D21: value D_Schottky -> B0540WS-7; DIGIKEY B0540WSDICT-ND -> (none)
- R59, R60, R61: footprint Resistor_SMD:R_0603_1608Metric_Pad1.05x0.95mm_HandSolder -> Resistor_SMD:R_0201_0603Metric_Pad0.64x0.40mm_HandSolder
Changed lines of the file:
@@
 $Descr A4 11693 8268
 encoding utf-8
-Sheet 9 10
+Sheet 9 11
 Title ""
 Date ""
@@
 P 2300 1150
 F 0 "D18" H 2300 933 50  0000 C CNN
-F 1 "1N5818" H 2300 1024 50  0000 C CNN
-F 2 "Diode_THT:D_DO-41_SOD81_P10.16mm_Horizontal" H 2300 975 50  0001 C CNN
-F 3 "http://www.vishay.com/docs/88525/1n5817.pdf" H 2300 1150 50  0001 C CNN
-F 4 "1N5818-TPCT-ND" H 2300 1150 50  0001 C CNN "DIGIKEY"
-F 5 "833-1N5818-TP" H 2300 1150 50  0001 C CNN "MOUSER"
+F 1 "B5818W-TP" H 2300 1024 50  0000 C CNN
+F 2 "Diode_SMD:D_SOD-123" H 2300 975 50  0001 C CNN
+F 3 "1810231731_ROHM-Semicon-RB160M-30TR_C183502.pdf" H 2300 1150 50  0001 C CNN
+F 4 "C183502" H 2300 1150 50  0001 C CNN "LCSC_PN"
+F 5 "SOD-123_1.6x2.6" H 2300 1150 50  0001 C CNN "LCSC_FP"
+F 6 "B5818W-TPMSCT-ND" H 2300 1150 50  0001 C CNN "DIGIKEY"
 	1    2300 1150
 	-1   0    0    1
@@
 F 0 "C21" H 2265 1346 50  0000 L CNN
 F 1 "50v 0.1uf" H 2265 1255 50  0000 L CNN
-F 2 "Capacitor_SMD:C_1206_3216Metric_Pad1.42x1.75mm_HandSolder" H 2188 1150 50  0001 C CNN
+F 2 "Capacitor_SMD:C_1206_3216Metric_Pad1.33x1.80mm_HandSolder" H 2188 1150 50  0001 C CNN
 F 3 "https://www.mouser.com/datasheet/2/212/KEM_C1002_X7R_SMD-1102033.pdf" H 2150 1300 50  0001 C CNN
 F 4 "399-C1206C104K5RAC7800CT-ND" H 2150 1300 50  0001 C CNN "DIGIKEY"
@@
 P 5300 1400
 F 0 "D20" V 5254 1480 50  0000 L CNN
-F 1 "1N5919BG" V 5345 1480 50  0000 L CNN
-F 2 "Diode_THT:D_DO-41_SOD81_P7.62mm_Horizontal" H 5300 1400 50  0001 C CNN
-F 3 "~" H 5300 1400 50  0001 C CNN
-F 4 "1N5919BGOS-ND" V 5300 1400 50  0001 C CNN "DIGIKEY"
-F 5 "863-1N5919BG " V 5300 1400 50  0001 C CNN "MOUSER"
+F 1 "ZMM5V6" V 5345 1480 50  0000 L CNN
+F 2 "Diode_SMD:D_MiniMELF" H 5300 1400 50  0001 C CNN
+F 3 "https://datasheet.lcsc.com/szlcsc/Semtech-ZMM5V6_C8062.pdf" H 5300 1400 50  0001 C CNN
+F 4 "C8062" V 5300 1400 50  0001 C CNN "LCSC_PN"
+F 5 "LL-34" V 5300 1400 50  0001 C CNN "LCSC_FP"
 	1    5300 1400
 	0    1    1    0
@@
 F 0 "C22" H 2365 2846 50  0000 L CNN
 F 1 "0.1uf" H 2365 2755 50  0000 L CNN
-F 2 "Capacitor_SMD:C_0805_2012Metric_Pad1.15x1.40mm_HandSolder" H 2288 2650 50  0001 C CNN
+F 2 "Capacitor_SMD:C_0805_2012Metric_Pad1.18x1.45mm_HandSolder" H 2288 2650 50  0001 C CNN
 F 3 "https://datasheet.lcsc.com/szlcsc/YAGEO-CC0805KRX7R9BB104_C49678.pdf" H 2250 2800 50  0001 C CNN
 F 4 "311-1140-1-ND" H 2250 2800 50  0001 C CNN "DIGIKEY"
@@
 P 7200 1100
 F 0 "D21" H 7200 1317 50  0000 C CNN
-F 1 "D_Schottky" H 7200 1226 50  0000 C CNN
+F 1 "B0540WS-7" H 7200 1226 50  0000 C CNN
 F 2 "Diode_SMD:D_SOD-323_HandSoldering" H 7200 1100 50  0001 C CNN
-F 3 "https://www.diodes.com/assets/Datasheets/B0540WS.pdf" H 7200 1100 50  0001 C CNN
-F 4 "B0540WSDICT-ND" H 7200 1100 50  0001 C CNN "DIGIKEY"
-F 5 "C98664" H 7200 1100 50  0001 C CNN "LCSC_PN"
-F 6 "SOD-323" H 7200 1100 50  0001 C CNN "LCSC_FP"
+F 3 "https://datasheet.lcsc.com/szlcsc/Diodes-Incorporated-B0540WS-7_C98664.pdf" H 7200 1100 50  0001 C CNN
+F 4 "C98664" H 7200 1100 50  0001 C CNN "LCSC_PN"
+F 5 "SOD-323" H 7200 1100 50  0001 C CNN "LCSC_FP"
 	1    7200 1100
 	1    0    0    -1
@@
 F 0 "R59" V 6993 1450 50  0000 C CNN
 F 1 "10k" V 7084 1450 50  0000 C CNN
-F 2 "Resistor_SMD:R_0603_1608Metric_Pad1.05x0.95mm_HandSolder" V 7130 1450 50  0001 C CNN
+F 2 "Resistor_SMD:R_0201_0603Metric_Pad0.64x0.40mm_HandSolder" V 7130 1450 50  0001 C CNN
 F 3 "~" H 7200 1450 50  0001 C CNN
 	1    7200 1450
@@
 F 0 "R60" V 7407 1800 50  0000 C CNN
 F 1 "120k" V 7316 1800 50  0000 C CNN
-F 2 "Resistor_SMD:R_0603_1608Metric_Pad1.05x0.95mm_HandSolder" V 7130 1800 50  0001 C CNN
+F 2 "Resistor_SMD:R_0201_0603Metric_Pad0.64x0.40mm_HandSolder" V 7130 1800 50  0001 C CNN
 F 3 "~" H 7200 1800 50  0001 C CNN
 	1    7200 1800
@@
 F 0 "C28" H 9115 1546 50  0000 L CNN
 F 1 "4.7nf" H 9115 1455 50  0000 L CNN
-F 2 "Capacitor_SMD:C_0805_2012Metric_Pad1.15x1.40mm_HandSolder" H 9038 1350 50  0001 C CNN
+F 2 "Capacitor_SMD:C_0805_2012Metric_Pad1.18x1.45mm_HandSolder" H 9038 1350 50  0001 C CNN
 F 3 "~" H 9000 1500 50  0001 C CNN
 F 4 "311-1133-1-ND" H 9000 1500 50  0001 C CNN "DIGIKEY"
@@
 P 1300 4050
 F 0 "D17" H 1300 3833 50  0000 C CNN
-F 1 "1N4007" H 1300 3924 50  0000 C CNN
-F 2 "Diode_THT:D_DO-41_SOD81_P10.16mm_Horizontal" H 1300 3875 50  0001 C CNN
-F 3 "http://www.vishay.com/docs/88503/1n4001.pdf" H 1300 4050 50  0001 C CNN
+F 1 "1N4007W" H 1300 3924 50  0000 C CNN
+F 2 "Diode_SMD:D_SOD-123" H 1300 3875 50  0001 C CNN
+F 3 "https://datasheet.lcsc.com/szlcsc/Shandong-Jingdao-Microelectronics-1N4007W_C108803.pdf" H 1300 4050 50  0001 C CNN
+F 4 "C108803" H 1300 4050 50  0001 C CNN "LCSC_PN"
+F 5 "SOD-123" H 1300 4050 50  0001 C CNN "LCSC_FP"
+F 6 "S1MB-FDITR-ND" H 1300 4050 50  0001 C CNN "DIGIKEY"
 	1    1300 4050
 	-1   0    0    1
@@
 F 0 "C29" H 9565 1546 50  0000 L CNN
 F 1 "22p" H 9565 1455 50  0000 L CNN
-F 2 "Capacitor_SMD:C_0805_2012Metric_Pad1.15x1.40mm_HandSolder" H 9488 1350 50  0001 C CNN
+F 2 "Capacitor_SMD:C_0805_2012Metric_Pad1.18x1.45mm_HandSolder" H 9488 1350 50  0001 C CNN
 F 3 "~" H 9450 1500 50  0001 C CNN
 F 4 "1276-1047-1-ND " H 9450 1500 50  0001 C CNN "DIGIKEY"
@@
 F 0 "R61" H 9520 1146 50  0000 L CNN
 F 1 "10k" H 9520 1055 50  0000 L CNN
-F 2 "Resistor_SMD:R_0603_1608Metric_Pad1.05x0.95mm_HandSolder" V 9380 1100 50  0001 C CNN
+F 2 "Resistor_SMD:R_0201_0603Metric_Pad0.64x0.40mm_HandSolder" V 9380 1100 50  0001 C CNN
 F 3 "~" H 9450 1100 50  0001 C CNN
 	1    9450 1100
@@
 F 0 "C25" H 4165 1446 50  0000 L CNN
 F 1 "50v 0.1uf" H 4165 1355 50  0000 L CNN
-F 2 "Capacitor_SMD:C_1206_3216Metric_Pad1.42x1.75mm_HandSolder" H 4088 1250 50  0001 C CNN
+F 2 "Capacitor_SMD:C_1206_3216Metric_Pad1.33x1.80mm_HandSolder" H 4088 1250 50  0001 C CNN
 F 3 "https://www.mouser.com/datasheet/2/212/KEM_C1002_X7R_SMD-1102033.pdf" H 4050 1400 50  0001 C CNN
 F 4 "399-C1206C104K5RAC7800CT-ND" H 4050 1400 50  0001 C CNN "DIGIKEY"
@@
 P 5200 2800
 F 0 "D19" V 5154 2880 50  0000 L CNN
-F 1 "1N5919BG" V 5245 2880 50  0000 L CNN
-F 2 "Diode_THT:D_DO-41_SOD81_P7.62mm_Horizontal" H 5200 2800 50  0001 C CNN
-F 3 "~" H 5200 2800 50  0001 C CNN
-F 4 "1N5919BGOS-ND" V 5200 2800 50  0001 C CNN "DIGIKEY"
-F 5 "863-1N5919BG " V 5200 2800 50  0001 C CNN "MOUSER"
+F 1 "ZMM5V6" V 5245 2880 50  0000 L CNN
+F 2 "Diode_SMD:D_MiniMELF" H 5200 2800 50  0001 C CNN
+F 3 "https://datasheet.lcsc.com/szlcsc/Semtech-ZMM5V6_C8062.pdf" H 5200 2800 50  0001 C CNN
+F 4 "C8062" V 5200 2800 50  0001 C CNN "LCSC_PN"
+F 5 "LL-34" V 5200 2800 50  0001 C CNN "LCSC_FP"
 	1    5200 2800
 	0    1    1    0
@@
 F 0 "C24" H 4065 2846 50  0000 L CNN
 F 1 "50v 0.1uf" H 4065 2755 50  0000 L CNN
-F 2 "Capacitor_SMD:C_1206_3216Metric_Pad1.42x1.75mm_HandSolder" H 3988 2650 50  0001 C CNN
+F 2 "Capacitor_SMD:C_1206_3216Metric_Pad1.33x1.80mm_HandSolder" H 3988 2650 50  0001 C CNN
 F 3 "https://www.mouser.com/datasheet/2/212/KEM_C1002_X7R_SMD-1102033.pdf" H 3950 2800 50  0001 C CNN
 F 4 "399-C1206C104K5RAC7800CT-ND" H 3950 2800 50  0001 C CNN "DIGIKEY"
@@
 F 0 "C20" H 2015 4246 50  0000 L CNN
 F 1 "0.1uf" H 2015 4155 50  0000 L CNN
-F 2 "Capacitor_SMD:C_0805_2012Metric_Pad1.15x1.40mm_HandSolder" H 1938 4050 50  0001 C CNN
+F 2 "Capacitor_SMD:C_0805_2012Metric_Pad1.18x1.45mm_HandSolder" H 1938 4050 50  0001 C CNN
 F 3 "https://datasheet.lcsc.com/szlcsc/YAGEO-CC0805KRX7R9BB104_C49678.pdf" H 1900 4200 50  0001 C CNN
 F 4 "311-1140-1-ND" H 1900 4200 50  0001 C CNN "DIGIKEY"
