File: speeduino-aio-na6-pnp.kicad_pcb (KiCad board)
At the start: 2 copper layers, 127 x 101.6 mm, 133 parts, among them J1 Conn_02x03_Odd_Even, J2 Conn_01x06, J3 174518-7, Q1 Q_PNP_BEC, SW1 MLL1200S, U1 ATmega2560-16AU, U10 MPX4250, U11 MC33814, U12 AMS1117-5.0, U2 VNLD5090, U3 VNLD5090, U4 VNLD5090, U5 VNLD5090, U6 VNLD5090, U7 TC4424A, U8 TC4424A, U9 SP720, Y1 Crystal_GND2

Commit message: restart a third time
Parts:
- removed JP2, JP3: Jumper_3_Open, Connector_PinHeader_2.54mm:PinHeader_1x03_P2.54mm_Vertical_SMD_Pin1Left
- removed SW1: MLL1200S, mll1200s:SW_MLL1200S
- added C30: 100n, Capacitor_SMD:C_0402_1005Metric_Pad0.74x0.62mm_HandSolder, F.Cu at (151.8, 113.5)
- added C31: 100n, Capacitor_SMD:C_0402_1005Metric_Pad0.74x0.62mm_HandSolder, F.Cu at (151.8, 111.5)
- added C32: 100n, Capacitor_SMD:C_0402_1005Metric_Pad0.74x0.62mm_HandSolder, F.Cu at (167.3, 118.5)
- added C33: 100n, Capacitor_SMD:C_0402_1005Metric_Pad0.74x0.62mm_HandSolder, F.Cu at (155.6, 108.9)
- added C34: 100n, Capacitor_SMD:C_0402_1005Metric_Pad0.74x0.62mm_HandSolder, F.Cu at (159.6, 124.8)
- added C35: 100n, Capacitor_SMD:C_0402_1005Metric_Pad0.74x0.62mm_HandSolder, F.Cu at (162.9, 124.8)
- added C36: 100n, Capacitor_SMD:C_0402_1005Metric_Pad0.74x0.62mm_HandSolder, F.Cu at (167.3, 120.5)
- added C37: 100n, Capacitor_SMD:C_0402_1005Metric_Pad0.74x0.62mm_HandSolder, F.Cu at (155.6, 110.9)
- added C38: 100n, Capacitor_SMD:C_0402_1005Metric_Pad0.74x0.62mm_HandSolder, F.Cu at (154.1, 134.1)
- added C39: 100n, Capacitor_SMD:C_0402_1005Metric_Pad0.74x0.62mm_HandSolder, F.Cu at (170.5, 116.6)
- added C40: 100n, Capacitor_SMD:C_0402_1005Metric_Pad0.74x0.62mm_HandSolder, F.Cu at (170.5, 118.6)
- added C41: 100n, Capacitor_SMD:C_0402_1005Metric_Pad0.74x0.62mm_HandSolder, F.Cu at (151.8, 115.5)
- added C42: 100n, Capacitor_SMD:C_0402_1005Metric_Pad0.74x0.62mm_HandSolder, F.Cu at (162.8, 126.8)
- added C43: 1u, Capacitor_SMD:C_0402_1005Metric_Pad0.74x0.62mm_HandSolder, F.Cu at (157.3, 130.1)
- added C44: 10n, Capacitor_SMD:C_0402_1005Metric_Pad0.74x0.62mm_HandSolder, F.Cu at (150.9, 117.9)
- added C45: 22u, Capacitor_SMD:CP_Elec_4x4.5, F.Cu at (137.6, 145.1)
- added C46: 47u, Capacitor_SMD:CP_Elec_5x5.8, F.Cu at (129.3, 145.6)
- added C47: 0.1, Capacitor_SMD:C_0805_2012Metric_Pad1.18x1.45mm_HandSolder, F.Cu at (132.3, 153.9)
- added C48: 10u, Capacitor_Tantalum_SMD:CP_EIA-7343-20_Kemet-V_Pad2.25x2.55mm_HandSolder, F.Cu at (135.7, 139.3)
- added C49: 0.1u, Capacitor_SMD:C_1206_3216Metric_Pad1.33x1.80mm_HandSolder, F.Cu at (143.8, 138.0)
- added C50: 0.1u, Capacitor_SMD:C_1206_3216Metric_Pad1.33x1.80mm_HandSolder, F.Cu at (127.8, 150.7)
- added C51: 0.1u, Capacitor_SMD:C_1206_3216Metric_Pad1.33x1.80mm_HandSolder, F.Cu at (136.8, 149.7)
- added F1: 250mA, Fuse:Fuse_1206_3216Metric_Pad1.42x1.75mm_HandSolder, F.Cu at (155.2, 120.4)
- added FB1: 600 @ 600MHz, Inductor_SMD:L_0805_2012Metric_Pad1.05x1.20mm_HandSolder, F.Cu at (145.7, 131.3)
- added H1: MountingHole_Pad, MountingHole:MountingHole_4.3mm_M4_Pad_Via, F.Cu at (167.8, 39.4)
- added H2: MountingHole_Pad, MountingHole:MountingHole_4.3mm_M4_Pad_Via, F.Cu at (29.5, 94.8)
- added H3: MountingHole_Pad, MountingHole:MountingHole_4.3mm_M4_Pad_Via, F.Cu at (26.5, 37.7)
- added H4: MountingHole_Pad, MountingHole:MountingHole_4.3mm_M4_Pad_Via, F.Cu at (167.5, 96.7)
- added L1: 15u, Inductor_SMD:L_Sunlord_MWSA0518_5.4x5.2mm, F.Cu at (135.8, 110.0)
- added L2: 15u, Inductor_SMD:L_Sunlord_MWSA0518_5.4x5.2mm, F.Cu at (133.1, 116.7)
- added L3: 39n, Inductor_SMD:L_0402_1005Metric_Pad0.77x0.64mm_HandSolder, F.Cu at (138.9, 134.2)
- added P1: USB_C_Plug_USB2.0, Connector_USB:USB_C_Receptacle_Amphenol_12401548E4-2A, F.Cu at (97.2, 25.9)
- added Q2: Q_PNP_BEC, Package_TO_SOT_SMD:SOT-23, F.Cu at (143.7, 144.9)
- added R62: 1k, Resistor_SMD:R_0603_1608Metric_Pad0.98x0.95mm_HandSolder, F.Cu at (57.5, 108.3)
- added R63: 1k, Resistor_SMD:R_0603_1608Metric_Pad0.98x0.95mm_HandSolder, F.Cu at (54.3, 108.3)
- added R64: 100k, Resistor_SMD:R_0603_1608Metric_Pad0.98x0.95mm_HandSolder, F.Cu at (55.9, 108.3)
- added R65: 100k, Resistor_SMD:R_0603_1608Metric_Pad0.98x0.95mm_HandSolder, F.Cu at (71.8, 108.3)
- added R66: 1k, Resistor_SMD:R_0603_1608Metric_Pad0.98x0.95mm_HandSolder, F.Cu at (70.2, 108.3)
- added R67: 1k, Resistor_SMD:R_0603_1608Metric_Pad0.98x0.95mm_HandSolder, F.Cu at (67.0, 108.3)
- added R68: 100k, Resistor_SMD:R_0603_1608Metric_Pad0.98x0.95mm_HandSolder, F.Cu at (68.6, 108.3)
- added R69: 2.4k, Resistor_SMD:R_0603_1608Metric_Pad0.98x0.95mm_HandSolder, F.Cu at (65.0, 100.6)
- added R70: 2.4k, Resistor_SMD:R_0603_1608Metric_Pad0.98x0.95mm_HandSolder, F.Cu at (63.0, 100.6)
- added R71: 2.4k, Resistor_SMD:R_0603_1608Metric_Pad0.98x0.95mm_HandSolder, F.Cu at (77.6, 100.7)
- added R72: 2.4k, Resistor_SMD:R_0603_1608Metric_Pad0.98x0.95mm_HandSolder, F.Cu at (75.5, 100.7)
- added TP1: TP_TACH, TestPoint:TestPoint_Pad_D1.0mm, F.Cu at (68.0, 175.2)
- added TP10: TestPoint_Small, TestPoint:TestPoint_Pad_D1.0mm, F.Cu at (167.3, 123.0)
- added TP11: TestPoint_Small, TestPoint:TestPoint_Pad_D1.0mm, F.Cu at (157.3, 132.6)
- added TP12: TP_VREG, TestPoint:TestPoint_Pad_D1.0mm, F.Cu at (144.3, 148.7)
- added TP13: TP_VPPREF, TestPoint:TestPoint_Pad_D1.0mm, F.Cu at (141.3, 152.6)
- added TP14: TP_VPPSENS, TestPoint:TestPoint_Pad_D1.0mm, F.Cu at (141.3, 149.6)
- added TP15: TP_VPROT, TestPoint:TestPoint_Pad_D1.0mm, F.Cu at (136.2, 152.9)
- added TP16: TP_CRANK, TestPoint:TestPoint_Pad_D1.0mm, F.Cu at (68.9, 151.6)
- added TP17: TP_CAM, TestPoint:TestPoint_Pad_D1.0mm, F.Cu at (64.8, 151.4)
- added TP2: TP_IAT, TestPoint:TestPoint_Pad_D1.0mm, F.Cu at (40.7, 149.5)
- added TP3: TP_VBAT, TestPoint:TestPoint_Pad_D1.0mm, F.Cu at (172.0, 159.8)
- added TP4: TP_CLT, TestPoint:TestPoint_Pad_D1.0mm, F.Cu at (48.8, 149.5)
- added TP5: TP_MAP, TestPoint:TestPoint_Pad_D1.0mm, F.Cu at (97.3, 148.7)
- added TP6: TP_TPS, TestPoint:TestPoint_Pad_D1.0mm, F.Cu at (53.0, 149.5)
- added TP7: TP_FLEX, TestPoint:TestPoint_Pad_D1.0mm, F.Cu at (37.0, 149.5)
- added TP8: TP_O2, TestPoint:TestPoint_Pad_D1.0mm, F.Cu at (56.9, 149.5)
- added TP9: TP_NRST, TestPoint:TestPoint_Pad_D1.0mm, F.Cu at (154.9, 113.4)
- added U13: VNLD5090, Package_SO:SOIC-8_3.9x4.9mm_P1.27mm, F.Cu at (62.1, 112.8)
- added U14: VNLD5090, Package_SO:SOIC-8_3.9x4.9mm_P1.27mm, F.Cu at (74.8, 112.8)
- added U15: MC33814, Package_QFP:LQFP-48-1EP_7x7mm_P0.5mm_EP3.6x3.6mm_ThermalVias, F.Cu at (64.5, 73.9)
- C1: value 1uf -> 0.1uf; footprint Capacitor_Tantalum_SMD:CP_EIA-7343-31_Kemet-D -> Capacitor_SMD:C_0805_2012Metric_Pad1.18x1.45mm_HandSolder
- C10: value 470pf -> 0.1uf; footprint Capacitor_SMD:C_0805_2012Metric_Pad1.15x1.40mm_HandSolder -> Capacitor_SMD:C_0805_2012Metric_Pad1.18x1.45mm_HandSolder
- C11, C15, C3: value 0.1uf -> 0.22uf; footprint Capacitor_SMD:C_0805_2012Metric_Pad1.15x1.40mm_HandSolder -> Capacitor_SMD:C_0805_2012Metric_Pad1.18x1.45mm_HandSolder
- C12, C5: value 0.22uf -> 0.1uf; footprint Capacitor_SMD:C_0805_2012Metric_Pad1.15x1.40mm_HandSolder -> Capacitor_SMD:C_0805_2012Metric_Pad1.18x1.45mm_HandSolder
- C13, C14, C2, C4, C6: footprint Capacitor_SMD:C_0805_2012Metric_Pad1.15x1.40mm_HandSolder -> Capacitor_SMD:C_0805_2012Metric_Pad1.18x1.45mm_HandSolder
- C16: value 0.22uf -> 10u; footprint Capacitor_SMD:C_0805_2012Metric_Pad1.15x1.40mm_HandSolder -> Capacitor_SMD:C_1206_3216Metric_Pad1.33x1.80mm_HandSolder
- C17: value EEE-FK0J220R 16v 22uf -> 10u; footprint Capacitor_SMD:CP_Elec_4x3 -> Capacitor_SMD:C_1206_3216Metric_Pad1.33x1.80mm_HandSolder
- C18: value 47uf -> 0.1u; footprint Capacitor_SMD:CP_Elec_6.3x5.8 -> Capacitor_SMD:C_0603_1608Metric_Pad1.08x0.95mm_HandSolder
- C19: value 35v 10uf -> 0.1u; footprint Capacitor_Tantalum_SMD:CP_EIA-7343-31_Kemet-D_Pad2.25x2.55mm_HandSolder -> Capacitor_SMD:C_0603_1608Metric_Pad1.08x0.95mm_HandSolder
- C20: value 0.1uf -> 10u; footprint Capacitor_SMD:C_0805_2012Metric_Pad1.15x1.40mm_HandSolder -> Capacitor_SMD:C_0603_1608Metric_Pad1.08x0.95mm_HandSolder
- C21: value 50v 0.1uf -> 220u; footprint Capacitor_SMD:C_1206_3216Metric_Pad1.42x1.75mm_HandSolder -> Capacitor_SMD:CP_Elec_10x14.3
- C22: value 0.1uf -> 220u; footprint Capacitor_SMD:C_0805_2012Metric_Pad1.15x1.40mm_HandSolder -> Capacitor_SMD:CP_Elec_10x14.3
- C23: value 47uf -> 0.1u; footprint Capacitor_SMD:CP_Elec_6.3x5.8 -> Capacitor_SMD:C_0402_1005Metric_Pad0.74x0.62mm_HandSolder
- C24: value 50v 0.1uf -> 100p; footprint Capacitor_SMD:C_1206_3216Metric_Pad1.42x1.75mm_HandSolder -> Capacitor_SMD:C_0402_1005Metric_Pad0.74x0.62mm_HandSolder
- C25: value 50v 0.1uf -> 12p; footprint Capacitor_SMD:C_1206_3216Metric_Pad1.42x1.75mm_HandSolder -> Capacitor_SMD:C_0402_1005Metric_Pad0.74x0.62mm_HandSolder
- C26: value 10v 47uf -> 12p; footprint Capacitor_Tantalum_SMD:CP_EIA-3528-21_Kemet-B_Pad1.50x2.35mm_HandSolder -> Capacitor_SMD:C_0402_1005Metric_Pad0.74x0.62mm_HandSolder
- C27: value 10v 47uf -> 2u2; footprint Capacitor_Tantalum_SMD:CP_EIA-3528-21_Kemet-B_Pad1.50x2.35mm_HandSolder -> Capacitor_SMD:C_0603_1608Metric_Pad1.08x0.95mm_HandSolder
- C28: value 4.7nf -> 2u2; footprint Capacitor_SMD:C_0805_2012Metric_Pad1.15x1.40mm_HandSolder -> Capacitor_SMD:C_0603_1608Metric_Pad1.08x0.95mm_HandSolder
- C29: value 22p -> 4u7; footprint Capacitor_SMD:C_0805_2012Metric_Pad1.15x1.40mm_HandSolder -> Capacitor_SMD:C_0603_1608Metric_Pad1.08x0.95mm_HandSolder
- C7: value 0.1uf -> 1uf; footprint Capacitor_SMD:C_0805_2012Metric_Pad1.15x1.40mm_HandSolder -> Capacitor_SMD:C_0805_2012Metric_Pad1.18x1.45mm_HandSolder
- C8: value 1uf -> 0.22uf; footprint Capacitor_SMD:C_0805_2012Metric_Pad1.15x1.40mm_HandSolder -> Capacitor_SMD:C_0805_2012Metric_Pad1.18x1.45mm_HandSolder
- C9: value 0.22uf -> 470pf; footprint Capacitor_SMD:C_0805_2012Metric_Pad1.15x1.40mm_HandSolder -> Capacitor_SMD:C_0805_2012Metric_Pad1.18x1.45mm_HandSolder
- D1, D3, D4: footprint LED_SMD:LED_0805_2012Metric_Pad1.15x1.40mm_HandSolder -> LED_SMD:LED_0603_1608Metric_Pad1.05x0.95mm_HandSolder
- D10: value 1n41001 -> B5819W
- D11: value LED -> B5819W; footprint LED_SMD:LED_0603_1608Metric -> Diode_SMD:D_SOD-123
- D12, D13, D14: footprint LED_SMD:LED_0603_1608Metric -> LED_SMD:LED_0603_1608Metric_Pad1.05x0.95mm_HandSolder
- D15: value MM3Zxx -> LED; footprint Diode_SMD:D_SOD-323_HandSoldering -> LED_SMD:LED_0603_1608Metric_Pad1.05x0.95mm_HandSolder
- D16: value MM3Zxx -> 1N4448WS
- D17: value 1N4007 -> 1N4448WS; footprint Diode_THT:D_DO-41_SOD81_P10.16mm_Horizontal -> Diode_SMD:D_SOD-323_HandSoldering
- D18: value 1N5818 -> 1N4448WS; footprint Diode_THT:D_DO-41_SOD81_P10.16mm_Horizontal -> Diode_SMD:D_SOD-323_HandSoldering
- D19: value 1N5919BG -> 1N4448WS; footprint Diode_THT:D_DO-41_SOD81_P7.62mm_Horizontal -> Diode_SMD:D_SOD-323_HandSoldering
- D2: value LED -> 1n41001; footprint LED_SMD:LED_0805_2012Metric_Pad1.15x1.40mm_HandSolder -> Diode_SMD:D_SOD-123
- D20: value 1N5919BG -> MM3Zxx; footprint Diode_THT:D_DO-41_SOD81_P7.62mm_Horizontal -> Diode_SMD:D_SOD-323_HandSoldering
- D21: value D_Schottky -> MM3Zxx
- D5, D6: value D -> LED; footprint Diode_SMD:D_SOD-323_HandSoldering -> LED_SMD:LED_0603_1608Metric_Pad1.05x0.95mm_HandSolder
- D7, D8: value D -> MM3Zxx
- D9: value LED -> B5819W; footprint LED_SMD:LED_0805_2012Metric_Pad1.15x1.40mm_HandSolder -> Diode_SMD:D_SOD-123
- J1: value Conn_02x03_Odd_Even -> CONN_BLACK; footprint Connector_PinHeader_2.54mm:PinHeader_2x03_P2.54mm_Vertical_SMD -> speeduino_connector_automotive:Delphi_Sicma_24_Black
- J2: value Conn_01x06 -> CONN_GREY; footprint Connector_PinHeader_2.54mm:PinHeader_1x06_P2.54mm_Vertical_SMD_Pin1Left -> speeduino_connector_automotive:Delphi_Sicma_24_Grey
- J3: value 174518-7 -> SWD; footprint speeduino_connector_automotive:174518-7 -> Connector_PinSocket_1.27mm:PinSocket_2x05_P1.27mm_Vertical_SMD
- JP1: footprint Connector_PinHeader_2.54mm:PinHeader_1x02_P2.54mm_Vertical_SMD_Pin1Right -> Jumper:SolderJumper-2_P1.3mm_Open_RoundedPad1.0x1.5mm
- Q1: value Q_PNP_BEC -> AO3401A; footprint Package_TO_SOT_SMD:SOT-23_Handsoldering -> Package_TO_SOT_SMD:SOT-23
- R1: value 1m -> 1k; footprint Resistor_SMD:R_0603_1608Metric_Pad1.05x0.95mm_HandSolder -> Resistor_SMD:R_0603_1608Metric_Pad0.98x0.95mm_HandSolder
- R10, R13, R17: value 2.4k -> 1k; footprint Resistor_SMD:R_0603_1608Metric_Pad1.05x0.95mm_HandSolder -> Resistor_SMD:R_0603_1608Metric_Pad0.98x0.95mm_HandSolder
- R11, R12: value 2.4k -> 100k; footprint Resistor_SMD:R_0603_1608Metric_Pad1.05x0.95mm_HandSolder -> Resistor_SMD:R_0603_1608Metric_Pad0.98x0.95mm_HandSolder
- R14, R2, R20, R21: footprint Resistor_SMD:R_0603_1608Metric_Pad1.05x0.95mm_HandSolder -> Resistor_SMD:R_0603_1608Metric_Pad0.98x0.95mm_HandSolder
- R15, R5, R6, R9: value 100k -> 1k; footprint Resistor_SMD:R_0603_1608Metric_Pad1.05x0.95mm_HandSolder -> Resistor_SMD:R_0603_1608Metric_Pad0.98x0.95mm_HandSolder
- R16: value 10k -> 1k; footprint Resistor_SMD:R_0603_1608Metric_Pad1.05x0.95mm_HandSolder -> Resistor_SMD:R_0603_1608Metric_Pad0.98x0.95mm_HandSolder
- R18, R19, R7, R8: value 1k -> 100k; footprint Resistor_SMD:R_0603_1608Metric_Pad1.05x0.95mm_HandSolder -> Resistor_SMD:R_0603_1608Metric_Pad0.98x0.95mm_HandSolder
- R22, R23: value 1k -> 10; footprint Resistor_SMD:R_0603_1608Metric_Pad1.05x0.95mm_HandSolder -> Resistor_SMD:R_0603_1608Metric_Pad0.98x0.95mm_HandSolder
- R24, R25: value 100k -> 10; footprint Resistor_SMD:R_0603_1608Metric_Pad1.05x0.95mm_HandSolder -> Resistor_SMD:R_0603_1608Metric_Pad0.98x0.95mm_HandSolder
- R26, R27, R28, R29, R4: value 1k -> 2.4k; footprint Resistor_SMD:R_0603_1608Metric_Pad1.05x0.95mm_HandSolder -> Resistor_SMD:R_0603_1608Metric_Pad0.98x0.95mm_HandSolder
- R3, R52: value 1k -> 10k; footprint Resistor_SMD:R_0603_1608Metric_Pad1.05x0.95mm_HandSolder -> Resistor_SMD:R_0603_1608Metric_Pad0.98x0.95mm_HandSolder
- R30: footprint Resistor_SMD:R_0603_1608Metric_Pad1.05x0.95mm_HandSolder -> Resistor_SMD:R_0805_2012Metric_Pad1.20x1.40mm_HandSolder
- R31: value 100k -> 2.49k; footprint Resistor_SMD:R_0603_1608Metric_Pad1.05x0.95mm_HandSolder -> Resistor_SMD:R_0805_2012Metric_Pad1.20x1.40mm_HandSolder
- R32: value 100k -> 3.9k; footprint Resistor_SMD:R_0603_1608Metric_Pad1.05x0.95mm_HandSolder -> Resistor_SMD:R_0805_2012Metric_Pad1.20x1.40mm_HandSolder
- R33: value 100k -> 1k; footprint Resistor_SMD:R_0603_1608Metric_Pad1.05x0.95mm_HandSolder -> Resistor_SMD:R_0805_2012Metric_Pad1.20x1.40mm_HandSolder
- R34: value 100k -> 470; footprint Resistor_SMD:R_0603_1608Metric_Pad1.05x0.95mm_HandSolder -> Resistor_SMD:R_0805_2012Metric_Pad1.20x1.40mm_HandSolder
- R35, R37, R38: value 2.4k -> 470; footprint Resistor_SMD:R_0603_1608Metric_Pad1.05x0.95mm_HandSolder -> Resistor_SMD:R_0805_2012Metric_Pad1.20x1.40mm_HandSolder
- R36: value 2.4k -> 2.49k; footprint Resistor_SMD:R_0603_1608Metric_Pad1.05x0.95mm_HandSolder -> Resistor_SMD:R_0805_2012Metric_Pad1.20x1.40mm_HandSolder
- R39, R40: value 10 -> 1k; footprint Resistor_SMD:R_0603_1608Metric_Pad1.05x0.95mm_HandSolder -> Resistor_SMD:R_0805_2012Metric_Pad1.20x1.40mm_HandSolder
- R41: value 10 -> 470; footprint Resistor_SMD:R_0603_1608Metric_Pad1.05x0.95mm_HandSolder -> Resistor_SMD:R_0805_2012Metric_Pad1.20x1.40mm_HandSolder
- R42: value 10 -> 220; footprint Resistor_SMD:R_0603_1608Metric_Pad1.05x0.95mm_HandSolder -> Resistor_SMD:R_0805_2012Metric_Pad1.20x1.40mm_HandSolder
- R43: value 1k -> 220; footprint Resistor_SMD:R_0603_1608Metric_Pad1.05x0.95mm_HandSolder -> Resistor_SMD:R_0805_2012Metric_Pad1.20x1.40mm_HandSolder
- R44: value 2.49k -> 470; footprint Resistor_SMD:R_0603_1608Metric_Pad1.05x0.95mm_HandSolder -> Resistor_SMD:R_0805_2012Metric_Pad1.20x1.40mm_HandSolder
- R45: value 3.9k -> 2.4k; footprint Resistor_SMD:R_0603_1608Metric_Pad1.05x0.95mm_HandSolder -> Resistor_SMD:R_0805_2012Metric_Pad1.20x1.40mm_HandSolder
- R46: value 1k -> null; footprint Resistor_SMD:R_0603_1608Metric_Pad1.05x0.95mm_HandSolder -> Resistor_SMD:R_0603_1608Metric_Pad0.98x0.95mm_HandSolder
- R47, R54, R57: value 470 -> null; footprint Resistor_SMD:R_0603_1608Metric_Pad1.05x0.95mm_HandSolder -> Resistor_SMD:R_0603_1608Metric_Pad0.98x0.95mm_HandSolder
- R48, R51: value 470 -> 5.1k; footprint Resistor_SMD:R_0603_1608Metric_Pad1.05x0.95mm_HandSolder -> Resistor_SMD:R_0402_1005Metric_Pad0.72x0.64mm_HandSolder
- R49: value 2.49k -> 22; footprint Resistor_SMD:R_0603_1608Metric_Pad1.05x0.95mm_HandSolder -> Resistor_SMD:R_0402_1005Metric_Pad0.72x0.64mm_HandSolder
- R50: value 470 -> 22; footprint Resistor_SMD:R_0603_1608Metric_Pad1.05x0.95mm_HandSolder -> Resistor_SMD:R_0402_1005Metric_Pad0.72x0.64mm_HandSolder
- R53: value 1k -> 3.24k; footprint Resistor_SMD:R_0603_1608Metric_Pad1.05x0.95mm_HandSolder -> Resistor_SMD:R_0603_1608Metric_Pad0.98x0.95mm_HandSolder
- R55: value 220 -> 10k; footprint Resistor_SMD:R_0603_1608Metric_Pad1.05x0.95mm_HandSolder -> Resistor_SMD:R_0603_1608Metric_Pad0.98x0.95mm_HandSolder
- R56: value 220 -> 3.24k; footprint Resistor_SMD:R_0603_1608Metric_Pad1.05x0.95mm_HandSolder -> Resistor_SMD:R_0603_1608Metric_Pad0.98x0.95mm_HandSolder
- R58: value 2.4k -> 60; footprint Resistor_SMD:R_0603_1608Metric_Pad1.05x0.95mm_HandSolder -> Resistor_SMD:R_0402_1005Metric_Pad0.72x0.64mm_HandSolder
- R59: value 10k -> 47; footprint Resistor_SMD:R_0603_1608Metric_Pad1.05x0.95mm_HandSolder -> Resistor_SMD:R_0402_1005Metric_Pad0.72x0.64mm_HandSolder
- R60: value 120k -> 10k; footprint Resistor_SMD:R_0603_1608Metric_Pad1.05x0.95mm_HandSolder -> Resistor_SMD:R_0402_1005Metric_Pad0.72x0.64mm_HandSolder
- R61: value 10k -> 100k; footprint Resistor_SMD:R_0603_1608Metric_Pad1.05x0.95mm_HandSolder -> Resistor_SMD:R_0603_1608Metric_Pad0.98x0.95mm_HandSolder
- RV1: value V14D220 -> Varistor
- U1: value ATmega2560-16AU -> VNLD5090; footprint Package_QFP:TQFP-100_14x14mm_P0.5mm -> Package_SO:SOIC-8_3.9x4.9mm_P1.27mm
- U10: value MPX4250 -> USBLC6-2SC6; footprint speeduino_misc:MPX4250 -> Package_TO_SOT_SMD:SOT-23-6
- U11: value MC33814 -> MCP2551-I-SN; footprint Package_QFP:LQFP-48-1EP_7x7mm_P0.5mm_EP3.6x3.6mm_ThermalVias -> Package_SO:SOIC-8_3.9x4.9mm_P1.27mm
- U12: value AMS1117-5.0 -> STM32F429ZGTx; footprint Package_TO_SOT_SMD:SOT-223-3_TabPin2 -> Package_QFP:LQFP-144_20x20mm_P0.5mm
- U2, U3: footprint Package_SO:SO-8_3.9x4.9mm_P1.27mm -> Package_SO:SOIC-8_3.9x4.9mm_P1.27mm
- U4, U5: value VNLD5090 -> TC4424A; footprint Package_SO:SO-8_3.9x4.9mm_P1.27mm -> Package_SO:SOIC-8_3.9x4.9mm_P1.27mm
- U6: value VNLD5090 -> SP720; footprint Package_SO:SO-8_3.9x4.9mm_P1.27mm -> Package_SO:SOIC-16_3.9x9.9mm_P1.27mm
- U7: value TC4424A -> MPX4250; footprint Package_SO:SOIC-8_3.9x4.9mm_P1.27mm -> speeduino_misc:MPX4250
- U8: value TC4424A -> TPS5430DDA; footprint Package_SO:SOIC-8_3.9x4.9mm_P1.27mm -> Package_SO:TI_SO-PowerPAD-8_ThermalVias
- U9: value SP720 -> TPS5430DDA; footprint Package_SO:SOIC-16_3.9x9.9mm_P1.27mm -> Package_SO:TI_SO-PowerPAD-8_ThermalVias
- Y1: value Crystal_GND2 -> 25mhz
- moved R21 427.3 mm to (30.3, 108.3), turned to 270 degrees
- moved R20 419.6 mm to (33.5, 108.3), turned to 90 degrees
- moved R18 416.4 mm to (46.3, 108.3), turned to 90 degrees
- moved U5 416.0 mm to (36.9, 112.8)
- moved R19 414.4 mm to (43.1, 108.3), turned to 270 degrees
- moved D8 405.3 mm to (38.7, 133.3), turned to 90 degrees
- moved D6 392.0 mm to (35.1, 104.9), turned to 270 degrees
- moved D5 390.0 mm to (38.3, 104.9), turned to 270 degrees
- moved D4 388.9 mm to (49.5, 104.9), turned to 270 degrees
- moved D7 386.7 mm to (60.9, 152.4), turned to 90 degrees
- moved D3 373.3 mm to (52.7, 104.9), turned to 270 degrees
- moved J2 373.2 mm to (59.6, 180.0)
- moved R9 362.2 mm to (84.3, 108.3), turned to 90 degrees
- moved R11 357.9 mm to (82.7, 108.3), turned to 90 degrees
- moved R10 355.3 mm to (81.1, 108.3), turned to 90 degrees
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Connections:
- C1 pad 1: CONN_VPROT -> IAT
- C10 pad 1: GND -> TPS
- C10 pad 2: ADC-CLAMP-6 -> GND
- C11 pad 1: CONN_TPS-IN -> ADC-CLAMP-3
- C12 pad 1: ADC-CLAMP-3 -> GND
- C12 pad 2: GND -> ADC-CLAMP-10
- C13 pad 1: GND -> ADC-CLAMP-9
- C13 pad 2: ADC-CLAMP-8 -> GND
- C14 pad 1: ADC-CLAMP-9 -> O2
- C15 pad 1: CONN_O2-IN -> ADC-CLAMP-4
- C16 pad 1: ADC-CLAMP-4 -> BUCK_IN
- C17 pad 1: /Power+Reset/VPPSENS -> +5V
- C18 pad 2: GND -> Net-(C18-Pad2)
- C19 pad 1: CONN_VBAT -> Net-(C19-Pad1)
- C19 pad 2: GND -> Net-(C19-Pad2)
- C2 pad 1: CONN_IAT-IN -> Net-(C2-Pad1)
- C20 pad 1: Net-(C18-Pad1) -> BUCK_IN
- C20 pad 2: GND -> Net-(C20-Pad2)
- C21 pad 1: CONN_VBAT -> +3V3
- C22 pad 1: /Power+Reset/VPPSENS -> +5V
- C23 pad 1: CONN_5v -> +3V3
- C24 pad 1: CONN_VPROT -> CANH
- C24 pad 2: GND -> CANL
- C25 pad 1: CONN_5v -> HSE_OUT
- C26 pad 1: CONN_VPROT -> Net-(C26-Pad1)
- C27 pad 1: CONN_5v -> Net-(C27-Pad1)
- C28 pad 1: /Power+Reset/RESET -> Net-(C28-Pad1)
- C29 pad 1: /Power+Reset/RESET -> +3V3
- C3 pad 1: Net-(C3-Pad1) -> ADC-CLAMP-1
- C4 pad 1: ADC-CLAMP-1 -> ADC-CLAMP-5
- C5 pad 1: ADC-CLAMP-5 -> VPROT
- C6 pad 1: CONN_VPROT -> CLT
- C7 pad 1: CONN_CLT-IN -> VPROT
- C8 pad 1: CONN_VPROT -> ADC-CLAMP-2
- C9 pad 1: ADC-CLAMP-2 -> GND
- C9 pad 2: GND -> ADC-CLAMP-6
- D1 pad 1: Net-(D1-Pad1) -> GND
- D10 pad 1: CONN_12v-SW -> GND
- D10 pad 2: CONN_IDLE-OUT -> Net-(C18-Pad1)
- D11 pad 2: Net-(D11-Pad2) -> Net-(C19-Pad1)
- D12 pad 1: GND -> Net-(D12-Pad1)
- D13 pad 1: GND -> Net-(D13-Pad1)
- D14 pad 1: GND -> Net-(D14-Pad1)
- D15 pad 1: /Sensors/CPU-D12 -> Net-(D15-Pad1)
- D15 pad 2: GND -> Net-(D15-Pad2)
- D16 pad 1: GND -> INJ-1
- D16 pad 2: CONN_5v -> Net-(D12-Pad1)
- D17 pad 1: Net-(C18-Pad1) -> INJ-2
- D17 pad 2: CONN_VBAT -> Net-(D13-Pad1)
- D18 pad 1: /mc33814/VREG-IN -> INJ-3
- D18 pad 2: CONN_VBAT -> Net-(D14-Pad1)
- D19 pad 1: CONN_VPROT -> INJ-4
- D19 pad 2: GND -> Net-(D15-Pad1)
- D2 pad 1: Net-(D2-Pad1) -> 12v-SW
- D2 pad 2: Net-(D2-Pad2) -> IDLE
- D20 pad 1: CONN_5v -> VPROT
- D21 pad 1: CONN_5v -> VREG
- D21 pad 2: Net-(D21-Pad2) -> VBAT
- D3 pad 1: Net-(D3-Pad1) -> GND
- D4 pad 1: Net-(D4-Pad1) -> GND
- D5 pad 1: CONN_INJ-1-OUT -> GND
- D5 pad 2: Net-(D1-Pad1) -> Net-(D5-Pad2)
- D6 pad 1: CONN_INJ-2-OUT -> GND
- D6 pad 2: Net-(D2-Pad1) -> Net-(D6-Pad2)
- D7 pad 1: CONN_INJ-3-OUT -> /Sensors/MCU-CLUTCH
- D7 pad 2: Net-(D3-Pad1) -> GND
- D8 pad 1: CONN_INJ-4-OUT -> GND
- D8 pad 2: Net-(D4-Pad1) -> +5V
- D9 pad 1: GND -> Net-(D9-Pad1)
- D9 pad 2: Net-(D9-Pad2) -> USB_CONN_VBUS
- J3 pad 1: CONN_INJ-3-OUT -> +3V3
- J3 pad 10: GND -> NRST
- J3 pad 2: CONN_IDLE-OUT -> SWDIO
- J3 pad 3: CONN_INJ-1-OUT -> GND
- J3 pad 4: CONN_INJ-4-OUT -> SWCLK
- J3 pad 5: Net-(J3-Pad5) -> GND
- J3 pad 6: CONN_INJ-2-OUT -> SWO
- J3 pad 7: GND -> Net-(J3-Pad7)
- J3 pad 8: GND -> Net-(J3-Pad8)
- JP1 pad 2: CONN_TACH-OUT -> TACH
- Q1 pad 1: /Power+Reset/VPPREF -> GND
- Q1 pad 2: /mc33814/VREG-IN -> Net-(D9-Pad1)
- Q1 pad 3: /Power+Reset/VPPSENS -> Net-(F1-Pad1)
- R1 pad 2: Net-(R1-Pad2) -> /FuelPump/MCU-FP
- R10 pad 1: Net-(D1-Pad2) -> Net-(R10-Pad1)
- R10 pad 2: CONN_12v-SW -> /FAN+TACH/MCU-TACH
- R11 pad 1: Net-(D2-Pad2) -> Net-(R11-Pad1)
- R11 pad 2: CONN_12v-SW -> GND
- R12 pad 1: Net-(D3-Pad2) -> GND
- R12 pad 2: CONN_12v-SW -> Net-(R10-Pad1)
- R13 pad 1: Net-(D4-Pad2) -> 12v-SW
- R13 pad 2: CONN_12v-SW -> Net-(JP1-Pad1)
- R14 pad 2: /FuelPump/CPU-D37 -> /Ignitors/MCU-IGN-3
- R15 pad 1: Net-(R14-Pad1) -> Net-(R15-Pad1)
- R15 pad 2: GND -> /Ignitors/MCU-IGN-4
- R16 pad 2: GND -> /Ignitors/MCU-IGN-1
- R17 pad 1: Net-(D9-Pad2) -> Net-(R17-Pad1)
- R17 pad 2: CONN_ST_SIG -> /Ignitors/MCU-IGN-2
- R18 pad 1: Net-(R18-Pad1) -> Net-(R14-Pad1)
- R18 pad 2: /IDLE+BOOST/CPU-D2 -> GND
- R19 pad 1: Net-(R19-Pad1) -> GND
- R19 pad 2: /IDLE+BOOST/CPU-D4 -> Net-(R15-Pad1)
- R2 pad 1: GND -> Net-(R1-Pad1)
- R2 pad 2: /Injectors/CPU-D10 -> GND
- R20 pad 1: Net-(R18-Pad1) -> Net-(R16-Pad1)
- R21 pad 2: Net-(R19-Pad1) -> Net-(R17-Pad1)
- R22 pad 1: Net-(R22-Pad1) -> IGN-3
- R22 pad 2: /FAN+TACH/CPU-D35 -> Net-(R22-Pad2)
- R23 pad 2: /FAN+TACH/CPU-D49 -> IGN-4
- R24 pad 1: Net-(R22-Pad1) -> IGN-1
- R24 pad 2: GND -> Net-(R24-Pad2)
- R25 pad 1: GND -> Net-(R25-Pad1)
- R25 pad 2: Net-(R23-Pad1) -> IGN-2
- R26 pad 1: CONN_12v-SW -> Net-(R22-Pad2)
- R26 pad 2: Net-(JP1-Pad1) -> Net-(D3-Pad2)
- R27 pad 1: Net-(R27-Pad1) -> Net-(D4-Pad2)
- R27 pad 2: /Ignitors/CPU-D32 -> Net-(R23-Pad1)
- R28 pad 1: Net-(R28-Pad1) -> Net-(R24-Pad2)
- R28 pad 2: /Ignitors/CPU-D33 -> Net-(D5-Pad2)
- R29 pad 1: Net-(R29-Pad1) -> Net-(D6-Pad2)
- R29 pad 2: /Ignitors/CPU-D39 -> Net-(R25-Pad1)
- R3 pad 2: /Injectors/CPU-D10 -> GND
- R30 pad 1: Net-(R30-Pad1) -> Net-(C2-Pad1)
- R30 pad 2: /Ignitors/CPU-D41 -> GND
- R31 pad 1: Net-(R27-Pad1) -> VPROT
- R31 pad 2: GND -> IAT
- R32 pad 1: GND -> VBAT
- R32 pad 2: Net-(R28-Pad1) -> Net-(C2-Pad1)
- R33 pad 1: Net-(R29-Pad1) -> /Sensors/MCU-CLUTCH
- R33 pad 2: GND -> CLUTCH
- R34 pad 1: GND -> ADC-CLAMP-1
- R34 pad 2: Net-(R30-Pad1) -> IAT
- R35 pad 1: Net-(R35-Pad1) -> ADC-CLAMP-5
- R35 pad 2: Net-(D11-Pad2) -> Net-(C2-Pad1)
- R36 pad 1: Net-(D12-Pad2) -> VPROT
- R36 pad 2: Net-(R36-Pad2) -> CLT
- R37 pad 1: Net-(JP2-Pad1) -> ADC-CLAMP-2
- R37 pad 2: Net-(D13-Pad2) -> CLT
- R38 pad 1: Net-(D14-Pad2) -> Net-(R38-Pad1)
- R38 pad 2: Net-(JP3-Pad1) -> ADC-CLAMP-6
- R39 pad 1: Net-(R35-Pad1) -> CRANK
- R39 pad 2: Net-(JP2-Pad3) -> VPROT
- R4 pad 1: Net-(R4-Pad1) -> Net-(D1-Pad2)
- R4 pad 2: /Injectors/CPU-D11 -> ST_SIG
- R40 pad 1: Net-(JP3-Pad3) -> CAM
- R40 pad 2: Net-(R36-Pad2) -> VPROT
- R41 pad 1: Net-(JP2-Pad1) -> ADC-CLAMP-3
- R41 pad 2: CONN_IGN-1-OUT -> TPS
- R42 pad 1: CONN_IGN-2-OUT -> ADC-CLAMP-10
- R42 pad 2: Net-(JP3-Pad1) -> CRANK
- R43 pad 1: Net-(C3-Pad1) -> ADC-CLAMP-9
- R43 pad 2: GND -> CAM
- R44 pad 1: CONN_VPROT -> ADC-CLAMP-4
- R44 pad 2: CONN_IAT-IN -> O2
- R45 pad 1: CONN_VBAT -> +5V
- R45 pad 2: Net-(C3-Pad1) -> ADC-CLAMP-8
- R46 pad 1: /Sensors/CPU-D12 -> BUCK_IN
- R46 pad 2: CONN_CLUTCH-IN -> BUCK_EN
- R47 pad 1: ADC-CLAMP-1 -> BUCK_EN
- R47 pad 2: CONN_IAT-IN -> GND
- R48 pad 1: ADC-CLAMP-5 -> Net-(P1-PadB5)
- R48 pad 2: Net-(C3-Pad1) -> GND
- R49 pad 1: CONN_VPROT -> USB_CONN_D-
- R49 pad 2: CONN_CLT-IN -> Net-(P1-PadA7)
- R5 pad 1: GND -> Net-(R5-Pad1)
- R5 pad 2: /Injectors/CPU-D11 -> /IDLE+BOOST/MCU-IDLE
- R50 pad 1: ADC-CLAMP-2 -> USB_CONN_D+
- R50 pad 2: CONN_CLT-IN -> Net-(P1-PadA6)
- R51 pad 1: Net-(R51-Pad1) -> Net-(P1-PadA5)
- R51 pad 2: ADC-CLAMP-6 -> GND
- R52 pad 1: CONN_CRANK-IN -> Net-(R52-Pad1)
- R52 pad 2: CONN_VPROT -> +3V3
- R53 pad 1: CONN_CAM-IN -> Net-(R53-Pad1)
- R53 pad 2: CONN_VPROT -> Net-(R52-Pad1)
- R54 pad 1: ADC-CLAMP-3 -> GND
- R54 pad 2: CONN_TPS-IN -> Net-(R53-Pad1)
- R55 pad 1: ADC-CLAMP-8 -> Net-(R55-Pad1)
- R55 pad 2: CONN_CRANK-IN -> +5V
- R56 pad 1: ADC-CLAMP-9 -> Net-(R56-Pad1)
- R56 pad 2: CONN_CAM-IN -> Net-(R55-Pad1)
- R57 pad 1: ADC-CLAMP-4 -> GND
- R57 pad 2: CONN_O2-IN -> Net-(R56-Pad1)
- R58 pad 1: CONN_5v -> CANL
- R58 pad 2: ADC-CLAMP-10 -> CANH
- R59 pad 1: Net-(D21-Pad2) -> Net-(C26-Pad1)
- R59 pad 2: CONN_5v -> HSE_IN
- R6 pad 1: GND -> Net-(R6-Pad1)
- R6 pad 2: /Injectors/CPU-D9 -> /IDLE+BOOST/MCU-BOOST
- R60 pad 1: CONN_5v -> Net-(R60-Pad1)
- R60 pad 2: Net-(R60-Pad2) -> +3V3
- R61 pad 1: CONN_5v -> GND
- R61 pad 2: /Power+Reset/RESET -> /Injectors/MCU-INJ-1
- R7 pad 1: Net-(R7-Pad1) -> Net-(R5-Pad1)
- R7 pad 2: /Injectors/CPU-D9 -> GND
- R8 pad 1: Net-(R8-Pad1) -> GND
- R8 pad 2: /Injectors/CPU-D8 -> Net-(R6-Pad1)
- R9 pad 1: GND -> Net-(R11-Pad1)
- R9 pad 2: /Injectors/CPU-D8 -> /FAN+TACH/MCU-FAN
- RV1 pad 1: CONN_VBAT -> GND
- RV1 pad 2: GND -> VBAT
- U1 pad 1: /IDLE+BOOST/CPU-D4 -> GND
- U1 pad 2: Net-(J2-Pad3) -> Net-(R1-Pad1)
- U1 pad 3: Net-(J2-Pad2) -> Net-(U1-Pad3)
- U1 pad 4: Net-(U1-Pad4) -> Net-(R3-Pad1)
- U1 pad 5: Net-(U1-Pad5) -> 12v-SW
- U1 pad 6: /IDLE+BOOST/CPU-D2 -> ST_SIG
- U1 pad 7: ADC-CLAMP-10 -> ST_SIG
- U1 pad 8: Net-(U1-Pad8) -> 12v-SW
- U10 pad 1: Net-(R51-Pad1) -> USB_CONN_D-
- U10 pad 3: CONN_VPROT -> USB_CONN_D+
- U10 pad 4: (no net) -> USB_D+
- U10 pad 5: (no net) -> USB_CONN_VBUS
- U10 pad 6: (no net) -> USB_D-
- U11 pad 1: Net-(U11-Pad1) -> MCU-CAN-TX
- U11 pad 2: Net-(U11-Pad2) -> GND
- U11 pad 3: Net-(U11-Pad3) -> +3V3
- U11 pad 4: Net-(U11-Pad4) -> MCU-CAN-RX
- U11 pad 5: Net-(U11-Pad5) -> +3V3
- U11 pad 6: Net-(U11-Pad6) -> CANL
- U11 pad 7: Net-(U11-Pad7) -> CANH
- U11 pad 8: Net-(U11-Pad8) -> GND
- U12 pad 1: GND -> Net-(U12-Pad1)
- U12 pad 2: CONN_5v -> Net-(U12-Pad2)
- U12 pad 3: Net-(C18-Pad1) -> Net-(U12-Pad3)
- U2 pad 1: Net-(R3-Pad1) -> Net-(R5-Pad1)
- U2 pad 3: Net-(R4-Pad1) -> Net-(R6-Pad1)
- U2 pad 6: CONN_INJ-2-OUT -> BOOST
- U2 pad 8: CONN_INJ-1-OUT -> IDLE
- U3 pad 1: Net-(R7-Pad1) -> Net-(R11-Pad1)
- U3 pad 3: Net-(R8-Pad1) -> Net-(R10-Pad1)
- U3 pad 6: CONN_INJ-4-OUT -> Net-(JP1-Pad1)
- U3 pad 8: CONN_INJ-3-OUT -> FAN
- U4 pad 1: GND -> Net-(U4-Pad1)
- U4 pad 3: Net-(U4-Pad3) -> GND
- U4 pad 4: Net-(R16-Pad1) -> Net-(R15-Pad1)
- U4 pad 5: CONN_12v-SW -> Net-(R23-Pad1)
- U4 pad 6: CONN_ST_SIG -> +5V
- U4 pad 7: CONN_ST_SIG -> Net-(R22-Pad2)
- U4 pad 8: CONN_12v-SW -> Net-(U4-Pad8)
- U5 pad 1: Net-(R18-Pad1) -> Net-(U5-Pad1)
- U5 pad 2: Net-(U5-Pad2) -> Net-(R16-Pad1)
- U5 pad 3: Net-(R19-Pad1) -> GND
- U5 pad 4: Net-(U5-Pad4) -> Net-(R17-Pad1)
- U5 pad 5: GND -> Net-(R25-Pad1)
- U5 pad 6: CONN_BOOST-OUT -> +5V
- U5 pad 7: GND -> Net-(R24-Pad2)
- U5 pad 8: CONN_IDLE-OUT -> Net-(U5-Pad8)
- U6 pad 1: Net-(R22-Pad1) -> ADC-CLAMP-1
- U6 pad 2: Net-(U6-Pad2) -> ADC-CLAMP-2
- U6 pad 3: Net-(R23-Pad1) -> ADC-CLAMP-3
- U6 pad 4: Net-(U6-Pad4) -> ADC-CLAMP-4
- U6 pad 5: GND -> ADC-CLAMP-5
- U6 pad 6: Net-(JP1-Pad1) -> ADC-CLAMP-6
- U6 pad 7: GND -> Net-(U6-Pad7)
- U6 pad 8: CONN_FAN-OUT -> GND
- U7 pad 1: Net-(U7-Pad1) -> Net-(R38-Pad1)
- U7 pad 2: Net-(R27-Pad1) -> GND
- U7 pad 3: GND -> VPROT
- U7 pad 4: Net-(R28-Pad1) -> (no net)
- U7 pad 5: Net-(R36-Pad2) -> (no net)
- U7 pad 6: CONN_5v -> (no net)
- U8 pad 1: Net-(U8-Pad1) -> Net-(C18-Pad2)
- U8 pad 2: Net-(R29-Pad1) -> Net-(U8-Pad2)
- U8 pad 3: GND -> Net-(U8-Pad3)
- U8 pad 4: Net-(R30-Pad1) -> Net-(R52-Pad1)
- U8 pad 5: Net-(JP3-Pad1) -> BUCK_EN
- U8 pad 6: CONN_5v -> GND
- U8 pad 7: Net-(JP2-Pad1) -> +5V
- U8 pad 8: Net-(U8-Pad8) -> Net-(C18-Pad1)
- U9 pad 1: ADC-CLAMP-1 -> Net-(C19-Pad2)
- U9 pad 2: ADC-CLAMP-2 -> Net-(U9-Pad2)
- U9 pad 3: ADC-CLAMP-3 -> Net-(U9-Pad3)
- U9 pad 4: ADC-CLAMP-4 -> Net-(R55-Pad1)
- U9 pad 5: ADC-CLAMP-5 -> BUCK_EN
- U9 pad 6: ADC-CLAMP-6 -> GND
- U9 pad 7: Net-(U9-Pad7) -> BUCK_IN
- U9 pad 8: GND -> Net-(C19-Pad1)
- U9 pad 9: Net-(U9-Pad9) -> GND
- Y1 pad 1: Net-(R1-Pad1) -> HSE_OUT
- Y1 pad 3: Net-(R1-Pad2) -> Net-(C26-Pad1)
- Y1 pad 4: (no net) -> GND
Routing:
- net GND: track 0.00 -> 76.9 mm, vias 0 -> 16
- net ADC-CLAMP-8: track 0.00 -> 46.3 mm
- net ADC-CLAMP-10: track 0.00 -> 38.8 mm
- net ADC-CLAMP-9: track 0.00 -> 35.3 mm
- net ADC-CLAMP-4: track 0.00 -> 29.7 mm, vias 0 -> 1
- net ADC-CLAMP-3: track 0.00 -> 27.7 mm, vias 0 -> 1
- net ADC-CLAMP-2: track 0.00 -> 24.1 mm, vias 0 -> 1
- net IAT: track 0.00 -> 21.8 mm
- net ADC-CLAMP-1: track 0.00 -> 19.1 mm, vias 0 -> 1
- net CLT: track 0.00 -> 18.1 mm
- net CANL: track 0.00 -> 15.2 mm
- net TPS: track 0.00 -> 13.4 mm
- net CANH: track 0.00 -> 12.7 mm
- net CRANK: track 0.00 -> 12.3 mm
- net O2: track 0.00 -> 11.4 mm
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Other:
- board size 127 x 101.6 mm -> 154 x 160 mm
- copper layers 2 -> 4

Commit message: Layout p much finished.. Time for some stretch goals..?
Parts:
- removed C42: 100n, Capacitor_SMD:C_0402_1005Metric_Pad0.74x0.62mm_HandSolder
- removed P1: USB_C_Plug_USB2.0, Connector_USB:USB_C_Receptacle_Amphenol_12401548E4-2A
- removed R48, R51: 5.1k, Resistor_SMD:R_0402_1005Metric_Pad0.72x0.64mm_HandSolder
- removed R49, R50: 22, Resistor_SMD:R_0402_1005Metric_Pad0.72x0.64mm_HandSolder
- added J4: USB_B, Connector_USB:USB_B_Amphenol_MUSB-D511_Vertical_Rugged, F.Cu at (109.0, 34.2)
- added J5: USB_EXT, Connector_PinHeader_2.54mm:PinHeader_1x05_P2.54mm_Vertical_SMD_Pin1Left, F.Cu at (121.5, 47.4)
- added REF**: PinHeader_1x09_P2.54mm_Vertical_SMD_Pin1Left, Connector_PinHeader_2.54mm:PinHeader_1x09_P2.54mm_Vertical_SMD_Pin1Left, F.Cu at (140.3, 39.5)
- added REF**: PinHeader_1x02_P2.54mm_Vertical, Connector_PinHeader_2.54mm:PinHeader_1x02_P2.54mm_Vertical, F.Cu at (110.2, 47.5)
- added REF**: PinHeader_1x02_P2.54mm_Vertical, Connector_PinHeader_2.54mm:PinHeader_1x02_P2.54mm_Vertical, F.Cu at (61.1, 55.5)
- added REF**: PinHeader_1x02_P2.54mm_Vertical, Connector_PinHeader_2.54mm:PinHeader_1x02_P2.54mm_Vertical, F.Cu at (40.5, 55.6)
- added REF**: microSD_HC_Hirose_DM3D-SF, Connector_Card:microSD_HC_Hirose_DM3D-SF, F.Cu at (141.0, 29.2)
- added REF**: BatteryHolder_ComfortableElectronic_CH273-2450_1x2450, Battery:BatteryHolder_ComfortableElectronic_CH273-2450_1x2450, F.Cu at (40.5, 51.8)
- added TP18: TP_BUCK_EN, TestPoint:TestPoint_Pad_D1.0mm, F.Cu at (124.7, 107.7)
- added TP19: TP_PWR_GND2, TestPoint:TestPoint_Pad_D1.0mm, F.Cu at (115.8, 90.8)
- added TP20: TP_PWR_GND1, TestPoint:TestPoint_Pad_D1.0mm, F.Cu at (115.8, 88.7)
- added TP21: TP_BUCK_IN, TestPoint:TestPoint_Pad_D1.0mm, F.Cu at (126.8, 107.7)
- TP10: value TestPoint_Small -> TP_5V
- TP11: value TestPoint_Small -> TP_3V
- moved TP3 153.7 mm to (26.8, 109.5)
- moved C4 153.7 mm to (26.8, 112.4)
- moved C2 148.2 mm to (27.9, 117.5), turned to 180 degrees
- moved R30 147.3 mm to (27.9, 115.3), turned to 180 degrees
- moved R32 144.1 mm to (30.9, 112.3), turned to 270 degrees
- moved R35 143.3 mm to (28.9, 112.3), turned to 270 degrees
- moved R17 128.8 mm to (157.3, 115.5), turned to 180 degrees
- moved R21 127.1 mm to (157.3, 114.0), turned to 0 degrees
- moved R16 125.5 mm to (157.3, 112.3), turned to 180 degrees
- moved U5 125.0 mm to (161.8, 107.3), turned to 90 degrees
- moved R20 123.8 mm to (157.3, 110.8), turned to 180 degrees
- moved R29 122.2 mm to (157.3, 109.2), turned to 0 degrees
- moved R25 120.6 mm to (157.3, 107.5), turned to 180 degrees
- moved C39 119.0 mm to (61.2, 69.5), turned to 180 degrees
- moved R28 119.0 mm to (157.3, 106.0), turned to 180 degrees
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Connections:
- C20 pad 2: Net-(C20-Pad2) -> GND
- C46 pad 2: GND -> Net-(C46-Pad2)
- C50 pad 2: GND -> Net-(C46-Pad2)
- C51 pad 2: GND -> Net-(C46-Pad2)
- D20 pad 2: GND -> Net-(C46-Pad2)
- J1 pad B1: GND -> ST_SIG
- J1 pad B8: ST_SIG -> GND
- J1 pad C1: INJ-1 -> IGN-2
- J1 pad C2: INJ-2 -> IGN-1
- J1 pad C3: INJ-3 -> IGN-4
- J1 pad C4: INJ-4 -> IGN-3
- J1 pad C5: IGN-1 -> INJ-2
- J1 pad C6: IGN-2 -> INJ-1
- J1 pad C7: IGN-3 -> INJ-4
- J1 pad C8: IGN-4 -> INJ-3
- J2 pad A8: FP -> Net-(J2-PadA8)
- J2 pad B3: GND -> FP
- J2 pad C1: FAN -> TACH
- J2 pad C2: TACH -> FAN
Routing:
- net GND: track 76.9 -> 328.4 mm, vias 16 -> 80
- net +5V: track 9.22 -> 250.9 mm, vias 3 -> 14
- net BOOST: track 0.00 -> 212.5 mm, vias 0 -> 3
- net IDLE: track 1.72 -> 210.1 mm, vias 0 -> 3
- net 12v-SW: track 4.10 -> 211.1 mm, vias 0 -> 7
- net FAN: track 0.00 -> 203.4 mm, vias 0 -> 3
- net VBAT: track 0.00 -> 195.7 mm, vias 0 -> 1
- net Net-(JP1-Pad1): track 5.74 -> 191.4 mm, vias 0 -> 2
- net /FuelPump/MCU-FP: track 0.00 -> 157.0 mm, vias 0 -> 3
- net NRST: track 0.00 -> 149.3 mm, vias 0 -> 5
- net MCU-CAN-TX: track 3.23 -> 147.5 mm, vias 1 -> 3
- net MCU-CAN-RX: track 3.26 -> 146.0 mm, vias 1 -> 3
- net VPROT: track 4.52 -> 141.1 mm, vias 0 -> 5
- net /FAN+TACH/MCU-TACH: track 0.00 -> 122.7 mm, vias 0 -> 2
- net ADC-CLAMP-6: track 6.64 -> 127.5 mm, vias 1 -> 3
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- added copper zone on In2.Cu, net +3V3
- added copper zone on In2.Cu, net +5V
- added copper zone on In2.Cu, net 12v-SW
- added copper zone on B.Cu, net GND
- added copper zone on F.Cu, net GND
- added copper zone on In1.Cu, net GND
- added copper zone on In2.Cu, net USB_CONN_VBUS
Other:
- board size 154 x 160 mm -> 160 x 117.5 mm
- board text added: "FUEL"
- board text added: "IGN1"
- board text added: "IGN2"
- board text added: "IGN3"
- board text added: "IGN4"
- board text added: "INJ1"
- board text added: "INJ2"
- board text added: "INJ3"
- board text added: "INJ4"
