File: FuelPump.sch (KiCad schematic (older format))
At the start: 1 part

Commit message: Almost finished w/ schematic
Parts:
- removed U?: VN5160S-E, Package_SO:SO-8_3.9x4.9mm_P1.27mm, symbol speeduino_ic_automotive:VN5160S-E
- added C?: 1uf, symbol Device:C
- added D?: LED, LED_SMD:LED_0805_2012Metric_Pad1.15x1.40mm_HandSolder, symbol Device:LED
- added R?: 10k, symbol Device:R
- added R?: 1k, symbol Device:R
- added R?: 2.4k, symbol Device:R
- added R?: 100k, symbol Device:R
- added U?: VNLD5090, Package_SO:SO-8_3.9x4.9mm_P1.27mm, symbol speeduino_ic_automotive:VNLD5090
Connections:
- net labels added: 12v-SW, CPU-D37, GND, ST_Sig, VPROT
- wire segments 0 -> 24
Changed lines of the file:
@@
 $Descr A4 11693 8268
 encoding utf-8
-Sheet 2 2
+Sheet 3 9
 Title ""
 Date ""
@@
 Comment4 ""
 $EndDescr
-$Comp
-L speeduino_ic_automotive:VN5160S-E U?
-U 1 1 5EF1A4E9
+Text HLabel 3250 3600 0    50   Input ~ 0
+CPU-D37
+$Comp
+L power:GND #PWR0108
+U 1 1 5EEB0693
+P 3650 3200
+F 0 "#PWR0108" H 3650 2950 50  0001 C CNN
+F 1 "GND" V 3655 3072 50  0000 R CNN
+F 2 "" H 3650 3200 50  0001 C CNN
+F 3 "" H 3650 3200 50  0001 C CNN
+	1    3650 3200
+	0    1    1    0
+$EndComp
+Text HLabel 5450 3250 1    50   Input ~ 0
+12v-SW
+Text HLabel 6950 3600 2    50   Output ~ 0
+ST_Sig
+Text HLabel 2600 3900 0    50   Input ~ 0
+VPROT
+$Comp
+L power:GND #PWR0109
+U 1 1 5EEB1B26
+P 4100 4250
+F 0 "#PWR0109" H 4100 4000 50  0001 C CNN
+F 1 "GND" V 4105 4122 50  0000 R CNN
+F 2 "" H 4100 4250 50  0001 C CNN
+F 3 "" H 4100 4250 50  0001 C CNN
+	1    4100 4250
+	1    0    0    -1
+$EndComp
+Wire Wire Line
+	5350 3900 5900 3900
+Wire Wire Line
+	5450 3450 5450 3250
+$Comp
+L power:GND #PWR0110
+U 1 1 5EEB672C
+P 6650 4500
+F 0 "#PWR0110" H 6650 4250 50  0001 C CNN
+F 1 "GND" H 6655 4327 50  0000 C CNN
+F 2 "" H 6650 4500 50  0001 C CNN
+F 3 "" H 6650 4500 50  0001 C CNN
+	1    6650 4500
+	1    0    0    -1
+$EndComp
+Wire Wire Line
+	5350 3600 5450 3600
+Wire Wire Line
+	6650 3600 6650 3900
+Wire Wire Line
+	5350 3750 5450 3750
+Wire Wire Line
+	5450 3750 5450 3600
+Connection ~ 5450 3600
+Wire Wire Line
+	5450 3450 5350 3450
+Wire Wire Line
+	5450 3450 7500 3450
+Wire Wire Line
+	7500 3450 7500 4950
+Wire Wire Line
+	7500 4950 5900 4950
+Wire Wire Line
+	5900 4950 5900 3900
+Connection ~ 5450 3450
+Connection ~ 6650 3600
+Wire Wire Line
+	6650 3600 6950 3600
+Wire Wire Line
+	5450 3600 6650 3600
+$Comp
+L Device:R R?
+U 1 1 5EEBE5EA
+P 4100 4100
+F 0 "R?" H 4170 4146 50  0000 L CNN
+F 1 "10k" H 4170 4055 50  0000 L CNN
+F 2 "" V 4030 4100 50  0001 C CNN
+F 3 "~" H 4100 4100 50  0001 C CNN
+F 4 "311-10KARCT-ND" H 4100 4100 50  0001 C CNN "DIGIKEY"
+F 5 "C17414" H 4100 4100 50  0001 C CNN "LCSC_PN"
+F 6 "0805" H 4100 4100 50  0001 C CNN "LCSC_FP"
+	1    4100 4100
+	1    0    0    -1
+$EndComp
+Wire Wire Line
+	4350 3900 4100 3900
+Wire Wire Line
+	4100 3900 4100 3950
+Wire Wire Line
+	4350 3600 3900 3600
+Wire Wire Line
+	3250 3600 3450 3600
+Wire Wire Line
+	3900 3600 3900 3500
+Connection ~ 3900 3600
+Wire Wire Line
+	3900 3600 3750 3600
+Wire Wire Line
+	4350 3450 4350 3200
+Wire Wire Line
+	2700 4050 2700 3900
+Wire Wire Line
+	2700 3900 2600 3900
+$Comp
+L power:GND #PWR0111
+U 1 1 5EEC78A8
+P 2700 4350
+F 0 "#PWR0111" H 2700 4100 50  0001 C CNN
+F 1 "GND" V 2705 4222 50  0000 R CNN
+F 2 "" H 2700 4350 50  0001 C CNN
+F 3 "" H 2700 4350 50  0001 C CNN
+	1    2700 4350
+	1    0    0    -1
+$EndComp
+$Comp
+L Device:C C?
+U 1 1 5F880F36
+P 2700 4200
+AR Path="/5EFFD74E/5F880F36" Ref="C?"  Part="1"
+AR Path="/5EF12BA4/5F880F36" Ref="C?"  Part="1"
+F 0 "C?" H 2815 4246 50  0000 L CNN
+F 1 "1uf" H 2815 4155 50  0000 L CNN
+F 2 "" H 2738 4050 50  0001 C CNN
+F 3 "~" H 2700 4200 50  0001 C CNN
+F 4 "311-1365-1-ND" H 2700 4200 50  0001 C CNN "DIGIKEY"
+F 5 "C28323" H 2700 4200 50  0001 C CNN "LCSC_PN"
+F 6 "0805" H 2700 4200 50  0001 C CNN "LCSC_FP"
+	1    2700 4200
+	1    0    0    -1
+$EndComp
+$Comp
+L speeduino_ic_automotive:VNLD5090 U?
+U 1 1 5F889AF3
 P 4750 3650
-AR Path="/5EF1A4E9" Ref="U?"  Part="1"
-AR Path="/5EF12BA4/5EF1A4E9" Ref="U?"  Part="1"
+AR Path="/5F889AF3" Ref="U?"  Part="1"
+AR Path="/5EEDB4C5/5F889AF3" Ref="U?"  Part="1"
+AR Path="/5EFA5E54/5F889AF3" Ref="U?"  Part="1"
+AR Path="/5EF12BA4/5F889AF3" Ref="U?"  Part="1"
 F 0 "U?" H 4850 4217 50  0000 C CNN
-F 1 "VN5160S-E" H 4850 4126 50  0000 C CNN
+F 1 "VNLD5090" H 4850 4126 50  0000 C CNN
 F 2 "Package_SO:SO-8_3.9x4.9mm_P1.27mm" H 4950 2950 50  0001 C CNN
-F 3 "https://www.st.com/resource/en/datasheet/vn5160s-e.pdf" H 4750 3650 50  0001 C CNN
+F 3 "https://www.st.com/resource/en/datasheet/vnld5090-e.pdf" H 4750 3650 50  0001 C CNN
+F 4 "511-VNLD5090-E" H 4750 3650 50  0001 C CNN "MOUSER"
+F 5 "497-18682-ND" H 4750 3650 50  0001 C CNN "DIGIKEY"
 	1    4750 3650
 	1    0    0    -1
 $EndComp
+$Comp
+L Device:R R?
+U 1 1 5F88E440
+P 3600 3600
+AR Path="/5EEDB4C5/5F88E440" Ref="R?"  Part="1"
+AR Path="/5EFA5E54/5F88E440" Ref="R?"  Part="1"
+AR Path="/5EF12BA4/5F88E440" Ref="R?"  Part="1"
+F 0 "R?" V 3393 3600 50  0000 C CNN
+F 1 "1k" V 3484 3600 50  0000 C CNN
+F 2 "" V 3530 3600 50  0001 C CNN
+F 3 "~" H 3600 3600 50  0001 C CNN
+F 4 "311-1.00KCRCT-ND" V 3600 3600 50  0001 C CNN "DIGIKEY"
+F 5 "C17513" V 3600 3600 50  0001 C CNN "LCSC_PN"
+F 6 "0805" V 3600 3600 50  0001 C CNN "LCSC_FP"
+	1    3600 3600
+	0    1    1    0
+$EndComp
+$Comp
+L Device:R R?
+U 1 1 5F896E46
+P 6650 4050
+AR Path="/5EEDB4C5/5F896E46" Ref="R?"  Part="1"
+AR Path="/5EFC1D36/5F896E46" Ref="R?"  Part="1"
+AR Path="/5EF12BA4/5F896E46" Ref="R?"  Part="1"
+F 0 "R?" V 6443 4050 50  0000 C CNN
+F 1 "2.4k" V 6534 4050 50  0000 C CNN
+F 2 "" V 6580 4050 50  0001 C CNN
+F 3 "~" H 6650 4050 50  0001 C CNN
+F 4 "311-2.40KCRCT-ND" V 6650 4050 50  0001 C CNN "DIGIKEY"
+F 5 "C17526" V 6650 4050 50  0001 C CNN "LCSC_PN"
+F 6 "0805" V 6650 4050 50  0001 C CNN "LCSC_FP"
+	1    6650 4050
+	-1   0    0    1
+$EndComp
+$Comp
+L Device:R R?
+U 1 1 5F89C767
+P 3900 3350
+AR Path="/5EEDB4C5/5F89C767" Ref="R?"  Part="1"
+AR Path="/5EFC1D36/5F89C767" Ref="R?"  Part="1"
+AR Path="/5EF12BA4/5F89C767" Ref="R?"  Part="1"
+F 0 "R?" H 3830 3304 50  0000 R CNN
+F 1 "100k" H 3830 3395 50  0000 R CNN
+F 2 "" V 3830 3350 50  0001 C CNN
+F 3 "~" H 3900 3350 50  0001 C CNN
+F 4 "311-100KCRCT-ND" V 3900 3350 50  0001 C CNN "DIGIKEY"
+F 5 "C17407" V 3900 3350 50  0001 C CNN "LCSC_PN"
+F 6 "0805" V 3900 3350 50  0001 C CNN "LCSC_FP"
+	1    3900 3350
+	-1   0    0    1
+$EndComp
+Wire Wire Line
+	3650 3200 3900 3200
+Connection ~ 3900 3200
+Wire Wire Line
+	3900 3200 4350 3200
+$Comp
+L Device:LED D?
+U 1 1 5F8A89CE
+P 6650 4350
+AR Path="/5EEDB4C5/5F8A89CE" Ref="D?"  Part="1"
+AR Path="/5EF12BA4/5F8A89CE" Ref="D?"  Part="1"
+F 0 "D?" H 6643 4095 50  0000 C CNN
+F 1 "LED" H 6643 4186 50  0000 C CNN
+F 2 "LED_SMD:LED_0805_2012Metric_Pad1.15x1.40mm_HandSolder" H 6650 4350 50  0001 C CNN
+F 3 "~" H 6650 4350 50  0001 C CNN
+F 4 "475-1415-1-ND" H 6650 4350 50  0001 C CNN "DIGIKEY"
+F 5 "C84256" H 6650 4350 50  0001 C CNN "LCSC_PN"
+F 6 "LED_0805" H 6650 4350 50  0001 C CNN "LCSC_FP"
+	1    6650 4350
+	0    -1   -1   0
+$EndComp
 $EndSCHEMATC

Commit message: Starting on layout
Parts:
- C1: renamed from C?; footprint (none) -> Capacitor_Tantalum_SMD:CP_EIA-7343-31_Kemet-D; LCSC_FP 0805 -> CASE-D_7343; LCSC_PN C28323 -> C117038
- R14, R15, R16, R17: renamed from R?; footprint (none) -> Resistor_SMD:R_0603_1608Metric_Pad1.05x0.95mm_HandSolder
- gave numbers to parts that had none: 2
Changed lines of the file:
@@
 $Descr A4 11693 8268
 encoding utf-8
-Sheet 3 9
+Sheet 3 10
 Title ""
 Date ""
@@
 	5450 3600 6650 3600
 $Comp
-L Device:R R?
+L Device:R R16
 U 1 1 5EEBE5EA
 P 4100 4100
-F 0 "R?" H 4170 4146 50  0000 L CNN
+F 0 "R16" H 4170 4146 50  0000 L CNN
 F 1 "10k" H 4170 4055 50  0000 L CNN
-F 2 "" V 4030 4100 50  0001 C CNN
+F 2 "Resistor_SMD:R_0603_1608Metric_Pad1.05x0.95mm_HandSolder" V 4030 4100 50  0001 C CNN
 F 3 "~" H 4100 4100 50  0001 C CNN
 F 4 "311-10KARCT-ND" H 4100 4100 50  0001 C CNN "DIGIKEY"
@@
 P 2700 4200
 AR Path="/5EFFD74E/5F880F36" Ref="C?"  Part="1"
-AR Path="/5EF12BA4/5F880F36" Ref="C?"  Part="1"
-F 0 "C?" H 2815 4246 50  0000 L CNN
+AR Path="/5EF12BA4/5F880F36" Ref="C1"  Part="1"
+F 0 "C1" H 2815 4246 50  0000 L CNN
 F 1 "1uf" H 2815 4155 50  0000 L CNN
-F 2 "" H 2738 4050 50  0001 C CNN
-F 3 "~" H 2700 4200 50  0001 C CNN
+F 2 "Capacitor_Tantalum_SMD:CP_EIA-7343-31_Kemet-D" H 2738 4050 50  0001 C CNN
+F 3 "https://datasheet.lcsc.com/szlcsc/KEMET-T491D106K050AT_C117038.pdf" H 2700 4200 50  0001 C CNN
 F 4 "311-1365-1-ND" H 2700 4200 50  0001 C CNN "DIGIKEY"
-F 5 "C28323" H 2700 4200 50  0001 C CNN "LCSC_PN"
-F 6 "0805" H 2700 4200 50  0001 C CNN "LCSC_FP"
+F 5 "C117038" H 2700 4200 50  0001 C CNN "LCSC_PN"
+F 6 "CASE-D_7343" H 2700 4200 50  0001 C CNN "LCSC_FP"
 	1    2700 4200
 	1    0    0    -1
@@
 AR Path="/5EEDB4C5/5F889AF3" Ref="U?"  Part="1"
 AR Path="/5EFA5E54/5F889AF3" Ref="U?"  Part="1"
-AR Path="/5EF12BA4/5F889AF3" Ref="U?"  Part="1"
-F 0 "U?" H 4850 4217 50  0000 C CNN
+AR Path="/5EF12BA4/5F889AF3" Ref="U4"  Part="1"
+F 0 "U4" H 4850 4217 50  0000 C CNN
 F 1 "VNLD5090" H 4850 4126 50  0000 C CNN
 F 2 "Package_SO:SO-8_3.9x4.9mm_P1.27mm" H 4950 2950 50  0001 C CNN
@@
 AR Path="/5EEDB4C5/5F88E440" Ref="R?"  Part="1"
 AR Path="/5EFA5E54/5F88E440" Ref="R?"  Part="1"
-AR Path="/5EF12BA4/5F88E440" Ref="R?"  Part="1"
-F 0 "R?" V 3393 3600 50  0000 C CNN
+AR Path="/5EF12BA4/5F88E440" Ref="R14"  Part="1"
+F 0 "R14" V 3393 3600 50  0000 C CNN
 F 1 "1k" V 3484 3600 50  0000 C CNN
-F 2 "" V 3530 3600 50  0001 C CNN
+F 2 "Resistor_SMD:R_0603_1608Metric_Pad1.05x0.95mm_HandSolder" V 3530 3600 50  0001 C CNN
 F 3 "~" H 3600 3600 50  0001 C CNN
 F 4 "311-1.00KCRCT-ND" V 3600 3600 50  0001 C CNN "DIGIKEY"
@@
 AR Path="/5EEDB4C5/5F896E46" Ref="R?"  Part="1"
 AR Path="/5EFC1D36/5F896E46" Ref="R?"  Part="1"
-AR Path="/5EF12BA4/5F896E46" Ref="R?"  Part="1"
-F 0 "R?" V 6443 4050 50  0000 C CNN
+AR Path="/5EF12BA4/5F896E46" Ref="R17"  Part="1"
+F 0 "R17" V 6443 4050 50  0000 C CNN
 F 1 "2.4k" V 6534 4050 50  0000 C CNN
-F 2 "" V 6580 4050 50  0001 C CNN
+F 2 "Resistor_SMD:R_0603_1608Metric_Pad1.05x0.95mm_HandSolder" V 6580 4050 50  0001 C CNN
 F 3 "~" H 6650 4050 50  0001 C CNN
 F 4 "311-2.40KCRCT-ND" V 6650 4050 50  0001 C CNN "DIGIKEY"
@@
 AR Path="/5EEDB4C5/5F89C767" Ref="R?"  Part="1"
 AR Path="/5EFC1D36/5F89C767" Ref="R?"  Part="1"
-AR Path="/5EF12BA4/5F89C767" Ref="R?"  Part="1"
-F 0 "R?" H 3830 3304 50  0000 R CNN
+AR Path="/5EF12BA4/5F89C767" Ref="R15"  Part="1"
+F 0 "R15" H 3830 3304 50  0000 R CNN
 F 1 "100k" H 3830 3395 50  0000 R CNN
-F 2 "" V 3830 3350 50  0001 C CNN
+F 2 "Resistor_SMD:R_0603_1608Metric_Pad1.05x0.95mm_HandSolder" V 3830 3350 50  0001 C CNN
 F 3 "~" H 3900 3350 50  0001 C CNN
 F 4 "311-100KCRCT-ND" V 3900 3350 50  0001 C CNN "DIGIKEY"
@@
 P 6650 4350
 AR Path="/5EEDB4C5/5F8A89CE" Ref="D?"  Part="1"
-AR Path="/5EF12BA4/5F8A89CE" Ref="D?"  Part="1"
-F 0 "D?" H 6643 4095 50  0000 C CNN
+AR Path="/5EF12BA4/5F8A89CE" Ref="D9"  Part="1"
+F 0 "D9" H 6643 4095 50  0000 C CNN
 F 1 "LED" H 6643 4186 50  0000 C CNN
 F 2 "LED_SMD:LED_0805_2012Metric_Pad1.15x1.40mm_HandSolder" H 6650 4350 50  0001 C CNN

Commit message: restart a third time
Parts:
- removed C1: 1uf, Capacitor_Tantalum_SMD:CP_EIA-7343-31_Kemet-D, symbol Device:C
- D1: renamed from D9; footprint LED_SMD:LED_0805_2012Metric_Pad1.15x1.40mm_HandSolder -> LED_SMD:LED_0603_1608Metric_Pad1.05x0.95mm_HandSolder
- R1: renamed from R14; footprint Resistor_SMD:R_0603_1608Metric_Pad1.05x0.95mm_HandSolder -> Resistor_SMD:R_0603_1608Metric_Pad0.98x0.95mm_HandSolder
- R2: renamed from R15; footprint Resistor_SMD:R_0603_1608Metric_Pad1.05x0.95mm_HandSolder -> Resistor_SMD:R_0603_1608Metric_Pad0.98x0.95mm_HandSolder
- R3: renamed from R16; footprint Resistor_SMD:R_0603_1608Metric_Pad1.05x0.95mm_HandSolder -> Resistor_SMD:R_0603_1608Metric_Pad0.98x0.95mm_HandSolder
- R4: renamed from R17; footprint Resistor_SMD:R_0603_1608Metric_Pad1.05x0.95mm_HandSolder -> Resistor_SMD:R_0603_1608Metric_Pad0.98x0.95mm_HandSolder
- U1: renamed from U4; footprint Package_SO:SO-8_3.9x4.9mm_P1.27mm -> Package_SO:SOIC-8_3.9x4.9mm_P1.27mm
Connections:
- net CPU-D37 renamed MCU-FP
Changed lines of the file:
@@
 $Descr A4 11693 8268
 encoding utf-8
-Sheet 3 10
-Title ""
-Date ""
-Rev ""
+Sheet 2 9
+Title "Speeduino STM32"
+Date "2021-04-20"
+Rev "v0.1"
 Comp ""
 Comment1 ""
@@
 $EndDescr
 Text HLabel 3250 3600 0    50   Input ~ 0
-CPU-D37
+MCU-FP
 $Comp
-L power:GND #PWR0108
+L power:GND #PWR05
 U 1 1 5EEB0693
 P 3650 3200
-F 0 "#PWR0108" H 3650 2950 50  0001 C CNN
+F 0 "#PWR05" H 3650 2950 50  0001 C CNN
 F 1 "GND" V 3655 3072 50  0000 R CNN
 F 2 "" H 3650 3200 50  0001 C CNN
@@
 Text HLabel 6950 3600 2    50   Output ~ 0
 ST_Sig
-Text HLabel 2600 3900 0    50   Input ~ 0
-VPROT
 $Comp
-L power:GND #PWR0109
+L power:GND #PWR06
 U 1 1 5EEB1B26
 P 4100 4250
-F 0 "#PWR0109" H 4100 4000 50  0001 C CNN
+F 0 "#PWR06" H 4100 4000 50  0001 C CNN
 F 1 "GND" V 4105 4122 50  0000 R CNN
 F 2 "" H 4100 4250 50  0001 C CNN
@@
 	5450 3450 5450 3250
 $Comp
-L power:GND #PWR0110
+L power:GND #PWR07
 U 1 1 5EEB672C
 P 6650 4500
-F 0 "#PWR0110" H 6650 4250 50  0001 C CNN
+F 0 "#PWR07" H 6650 4250 50  0001 C CNN
 F 1 "GND" H 6655 4327 50  0000 C CNN
 F 2 "" H 6650 4500 50  0001 C CNN
@@
 	5450 3600 6650 3600
 $Comp
-L Device:R R16
+L Device:R R3
 U 1 1 5EEBE5EA
 P 4100 4100
-F 0 "R16" H 4170 4146 50  0000 L CNN
+F 0 "R3" H 4170 4146 50  0000 L CNN
 F 1 "10k" H 4170 4055 50  0000 L CNN
-F 2 "Resistor_SMD:R_0603_1608Metric_Pad1.05x0.95mm_HandSolder" V 4030 4100 50  0001 C CNN
+F 2 "Resistor_SMD:R_0603_1608Metric_Pad0.98x0.95mm_HandSolder" V 4030 4100 50  0001 C CNN
 F 3 "~" H 4100 4100 50  0001 C CNN
 F 4 "311-10KARCT-ND" H 4100 4100 50  0001 C CNN "DIGIKEY"
@@
 Wire Wire Line
 	4350 3450 4350 3200
-Wire Wire Line
-	2700 4050 2700 3900
-Wire Wire Line
-	2700 3900 2600 3900
-$Comp
-L power:GND #PWR0111
-U 1 1 5EEC78A8
-P 2700 4350
-F 0 "#PWR0111" H 2700 4100 50  0001 C CNN
-F 1 "GND" V 2705 4222 50  0000 R CNN
-F 2 "" H 2700 4350 50  0001 C CNN
-F 3 "" H 2700 4350 50  0001 C CNN
-	1    2700 4350
-	1    0    0    -1
-$EndComp
-$Comp
-L Device:C C?
-U 1 1 5F880F36
-P 2700 4200
-AR Path="/5EFFD74E/5F880F36" Ref="C?"  Part="1"
-AR Path="/5EF12BA4/5F880F36" Ref="C1"  Part="1"
-F 0 "C1" H 2815 4246 50  0000 L CNN
-F 1 "1uf" H 2815 4155 50  0000 L CNN
-F 2 "Capacitor_Tantalum_SMD:CP_EIA-7343-31_Kemet-D" H 2738 4050 50  0001 C CNN
-F 3 "https://datasheet.lcsc.com/szlcsc/KEMET-T491D106K050AT_C117038.pdf" H 2700 4200 50  0001 C CNN
-F 4 "311-1365-1-ND" H 2700 4200 50  0001 C CNN "DIGIKEY"
-F 5 "C117038" H 2700 4200 50  0001 C CNN "LCSC_PN"
-F 6 "CASE-D_7343" H 2700 4200 50  0001 C CNN "LCSC_FP"
-	1    2700 4200
-	1    0    0    -1
-$EndComp
 $Comp
 L speeduino_ic_automotive:VNLD5090 U?
@@
 AR Path="/5EEDB4C5/5F889AF3" Ref="U?"  Part="1"
 AR Path="/5EFA5E54/5F889AF3" Ref="U?"  Part="1"
-AR Path="/5EF12BA4/5F889AF3" Ref="U4"  Part="1"
-F 0 "U4" H 4850 4217 50  0000 C CNN
+AR Path="/5EF12BA4/5F889AF3" Ref="U1"  Part="1"
+F 0 "U1" H 4850 4217 50  0000 C CNN
 F 1 "VNLD5090" H 4850 4126 50  0000 C CNN
-F 2 "Package_SO:SO-8_3.9x4.9mm_P1.27mm" H 4950 2950 50  0001 C CNN
+F 2 "Package_SO:SOIC-8_3.9x4.9mm_P1.27mm" H 4950 2950 50  0001 C CNN
 F 3 "https://www.st.com/resource/en/datasheet/vnld5090-e.pdf" H 4750 3650 50  0001 C CNN
 F 4 "511-VNLD5090-E" H 4750 3650 50  0001 C CNN "MOUSER"
@@
 AR Path="/5EEDB4C5/5F88E440" Ref="R?"  Part="1"
 AR Path="/5EFA5E54/5F88E440" Ref="R?"  Part="1"
-AR Path="/5EF12BA4/5F88E440" Ref="R14"  Part="1"
-F 0 "R14" V 3393 3600 50  0000 C CNN
+AR Path="/5EF12BA4/5F88E440" Ref="R1"  Part="1"
+F 0 "R1" V 3393 3600 50  0000 C CNN
 F 1 "1k" V 3484 3600 50  0000 C CNN
-F 2 "Resistor_SMD:R_0603_1608Metric_Pad1.05x0.95mm_HandSolder" V 3530 3600 50  0001 C CNN
+F 2 "Resistor_SMD:R_0603_1608Metric_Pad0.98x0.95mm_HandSolder" V 3530 3600 50  0001 C CNN
 F 3 "~" H 3600 3600 50  0001 C CNN
 F 4 "311-1.00KCRCT-ND" V 3600 3600 50  0001 C CNN "DIGIKEY"
@@
 AR Path="/5EEDB4C5/5F896E46" Ref="R?"  Part="1"
 AR Path="/5EFC1D36/5F896E46" Ref="R?"  Part="1"
-AR Path="/5EF12BA4/5F896E46" Ref="R17"  Part="1"
-F 0 "R17" V 6443 4050 50  0000 C CNN
+AR Path="/5EF12BA4/5F896E46" Ref="R4"  Part="1"
+F 0 "R4" V 6443 4050 50  0000 C CNN
 F 1 "2.4k" V 6534 4050 50  0000 C CNN
-F 2 "Resistor_SMD:R_0603_1608Metric_Pad1.05x0.95mm_HandSolder" V 6580 4050 50  0001 C CNN
+F 2 "Resistor_SMD:R_0603_1608Metric_Pad0.98x0.95mm_HandSolder" V 6580 4050 50  0001 C CNN
 F 3 "~" H 6650 4050 50  0001 C CNN
 F 4 "311-2.40KCRCT-ND" V 6650 4050 50  0001 C CNN "DIGIKEY"
@@
 AR Path="/5EEDB4C5/5F89C767" Ref="R?"  Part="1"
 AR Path="/5EFC1D36/5F89C767" Ref="R?"  Part="1"
-AR Path="/5EF12BA4/5F89C767" Ref="R15"  Part="1"
-F 0 "R15" H 3830 3304 50  0000 R CNN
+AR Path="/5EF12BA4/5F89C767" Ref="R2"  Part="1"
+F 0 "R2" H 3830 3304 50  0000 R CNN
 F 1 "100k" H 3830 3395 50  0000 R CNN
-F 2 "Resistor_SMD:R_0603_1608Metric_Pad1.05x0.95mm_HandSolder" V 3830 3350 50  0001 C CNN
+F 2 "Resistor_SMD:R_0603_1608Metric_Pad0.98x0.95mm_HandSolder" V 3830 3350 50  0001 C CNN
 F 3 "~" H 3900 3350 50  0001 C CNN
 F 4 "311-100KCRCT-ND" V 3900 3350 50  0001 C CNN "DIGIKEY"
@@
 P 6650 4350
 AR Path="/5EEDB4C5/5F8A89CE" Ref="D?"  Part="1"
-AR Path="/5EF12BA4/5F8A89CE" Ref="D9"  Part="1"
-F 0 "D9" H 6643 4095 50  0000 C CNN
+AR Path="/5EF12BA4/5F8A89CE" Ref="D1"  Part="1"
+F 0 "D1" H 6643 4095 50  0000 C CNN
 F 1 "LED" H 6643 4186 50  0000 C CNN
-F 2 "LED_SMD:LED_0805_2012Metric_Pad1.15x1.40mm_HandSolder" H 6650 4350 50  0001 C CNN
+F 2 "LED_SMD:LED_0603_1608Metric_Pad1.05x0.95mm_HandSolder" H 6650 4350 50  0001 C CNN
 F 3 "~" H 6650 4350 50  0001 C CNN
 F 4 "475-1415-1-ND" H 6650 4350 50  0001 C CNN "DIGIKEY"
