File: mc33814.sch (KiCad schematic (older format))
At the start: 1 part

Commit message: Starting on layout
Parts:
- gave numbers to parts that had none: 1
Changed lines of the file:
@@
 $Descr A4 11693 8268
 encoding utf-8
-Sheet 8 9
+Sheet 8 10
 Title ""
 Date ""
@@
 P 5950 3500
 AR Path="/5F2C7EEA" Ref="U?"  Part="1"
-AR Path="/5F2C75FB/5F2C7EEA" Ref="U?"  Part="1"
-F 0 "U?" H 7094 3546 50  0000 L CNN
+AR Path="/5F2C75FB/5F2C7EEA" Ref="U11"  Part="1"
+F 0 "U11" H 7094 3546 50  0000 L CNN
 F 1 "MC33814" H 7094 3455 50  0000 L CNN
 F 2 "Package_QFP:LQFP-48-1EP_7x7mm_P0.5mm_EP3.6x3.6mm_ThermalVias" H 5950 3500 50  0001 C CNN

Commit message: restart a third time
Parts:
- added C45: 22u, Capacitor_SMD:CP_Elec_4x4.5, symbol Device:CP_Small
- added C46: 47u, Capacitor_SMD:CP_Elec_5x5.8, symbol Device:CP_Small
- added C47: 0.1, Capacitor_SMD:C_0805_2012Metric_Pad1.18x1.45mm_HandSolder, symbol Device:C_Small
- added C48: 10u, Capacitor_Tantalum_SMD:CP_EIA-7343-20_Kemet-V_Pad2.25x2.55mm_HandSolder, symbol Device:CP_Small
- added C49, C50, C51: 0.1u, Capacitor_SMD:C_1206_3216Metric_Pad1.33x1.80mm_HandSolder, symbol Device:C_Small
- added D20, D21: MM3Zxx, Diode_SMD:D_SOD-323_HandSoldering, symbol Device:D_Small
- added Q2: Q_PNP_BEC, Package_TO_SOT_SMD:SOT-23, symbol Device:Q_PNP_BEC
- added RV1: Varistor, Varistor:RV_Disc_D15.5mm_W3.9mm_P7.5mm, symbol Device:Varistor
- added TP12: TP_VREG, TestPoint:TestPoint_Pad_D1.0mm, symbol Connector:TestPoint_Small
- added TP13: TP_VPPREF, TestPoint:TestPoint_Pad_D1.0mm, symbol Connector:TestPoint_Small
- added TP14: TP_VPPSENS, TestPoint:TestPoint_Pad_D1.0mm, symbol Connector:TestPoint_Small
- added TP15: TP_VPROT, TestPoint:TestPoint_Pad_D1.0mm, symbol Connector:TestPoint_Small
- renumbered U11 to U15
Connections:
- net GND: now also C45.2, C46.2, C47.2, C48.2, C49.2, C50.2, C51.2, D20.2 (A), RV1.1
- net VPPREF: now also Q2.1 (B), TP13.1
- net VPPSENS: now also C45.1, C47.1, Q2.3 (C), TP14.1
- net VPROT: now also C46.1, C50.1, C51.1, D20.1 (K), TP15.1
- net CPU-A10 renamed MCU-RIN2
- net CPU-A6 renamed MCU-SPI1-CS
- net CPU-A9 renamed MCU-RIN1
- net CPU-MISO renamed MCU-SPI1-MISO
- net CPU-MOSI renamed MCU-SPI1-MOSI
- net CPU-SCLK renamed MCU-SPI1-SCK
- net VREG-IN renamed VREG
- net VREG: now also D21.1 (K), Q2.2 (E), TP12.1
- new net VBAT: C48.1, C49.1, D21.2 (A), RV1.2
- no-connect marks 0 -> 29
Other:
- moved on the sheet: U15

Commit message: Layout p much finished.. Time for some stretch goals..?
Connections:
- net GND: no longer C46.2, C50.2, C51.2, D20.2 (A)
- new net: C46.2, C50.2, C51.2, D20.2 (A)
Other:
- moved on the sheet: C46, C50, C51, D20, TP15
Changed lines of the file:
@@
 Wire Wire Line
 	7750 4050 7750 3900
-Text GLabel 8500 2350 2    50   Input ~ 0
+Text GLabel 4750 5050 2    50   Input ~ 0
 VPROT
 Text GLabel 4300 3900 3    50   Input ~ 0
@@
 L Device:C_Small C50
 U 1 1 60B98827
-P 8100 2550
-F 0 "C50" H 8192 2596 50  0000 L CNN
-F 1 "0.1u" H 8192 2505 50  0000 L CNN
-F 2 "Capacitor_SMD:C_1206_3216Metric_Pad1.33x1.80mm_HandSolder" H 8100 2550 50  0001 C CNN
-F 3 "https://datasheet.lcsc.com/lcsc/1805021622_KEMET-C1206C104K5RAC7800_C141184.pdf" H 8100 2550 50  0001 C CNN
-F 4 "C141184" H 8100 2550 50  0001 C CNN "LCSC_PN"
-F 5 "1206" H 8100 2550 50  0001 C CNN "LCSC_FP"
-	1    8100 2550
+P 4350 5250
+F 0 "C50" H 4442 5296 50  0000 L CNN
+F 1 "0.1u" H 4442 5205 50  0000 L CNN
+F 2 "Capacitor_SMD:C_1206_3216Metric_Pad1.33x1.80mm_HandSolder" H 4350 5250 50  0001 C CNN
+F 3 "https://datasheet.lcsc.com/lcsc/1805021622_KEMET-C1206C104K5RAC7800_C141184.pdf" H 4350 5250 50  0001 C CNN
+F 4 "C141184" H 4350 5250 50  0001 C CNN "LCSC_PN"
+F 5 "1206" H 4350 5250 50  0001 C CNN "LCSC_FP"
+	1    4350 5250
 	1    0    0    -1
 $EndComp
@@
 L Device:CP_Small C46
 U 1 1 60B98E5B
-P 7750 2500
-F 0 "C46" H 7838 2546 50  0000 L CNN
-F 1 "47u" H 7838 2455 50  0000 L CNN
-F 2 "Capacitor_SMD:CP_Elec_5x5.8" H 7750 2500 50  0001 C CNN
-F 3 "https://datasheet.lcsc.com/lcsc/1912111437_PANASONIC-EEEFK0J470AR_C336380.pdf" H 7750 2500 50  0001 C CNN
-F 4 "C336380" H 7750 2500 50  0001 C CNN "LCSC_PN"
-F 5 "SMD,5x5.8mm" H 7750 2500 50  0001 C CNN "LCSC_FP"
-	1    7750 2500
+P 4000 5200
+F 0 "C46" H 4088 5246 50  0000 L CNN
+F 1 "47u" H 4088 5155 50  0000 L CNN
+F 2 "Capacitor_SMD:CP_Elec_5x5.8" H 4000 5200 50  0001 C CNN
+F 3 "https://datasheet.lcsc.com/lcsc/1912111437_PANASONIC-EEEFK0J470AR_C336380.pdf" H 4000 5200 50  0001 C CNN
+F 4 "C336380" H 4000 5200 50  0001 C CNN "LCSC_PN"
+F 5 "SMD,5x5.8mm" H 4000 5200 50  0001 C CNN "LCSC_FP"
+	1    4000 5200
 	1    0    0    -1
 $EndComp
@@
 L Device:D_Small D20
 U 1 1 60B9A71D
-P 7300 2500
-F 0 "D20" V 7254 2570 50  0000 L CNN
-F 1 "MM3Zxx" V 7345 2570 50  0000 L CNN
-F 2 "Diode_SMD:D_SOD-323_HandSoldering" V 7300 2500 50  0001 C CNN
-F 3 "https://diotec.com/tl_files/diotec/files/pdf/datasheets/mm3z2v4.pdf" V 7300 2500 50  0001 C CNN
-F 4 "C152524" V 7300 2500 50  0001 C CNN "LCSC_PN"
-F 5 "SOD-323" V 7300 2500 50  0001 C CNN "LCSC_FP"
-	1    7300 2500
+P 3550 5200
+F 0 "D20" V 3504 5270 50  0000 L CNN
+F 1 "MM3Zxx" V 3595 5270 50  0000 L CNN
+F 2 "Diode_SMD:D_SOD-323_HandSoldering" V 3550 5200 50  0001 C CNN
+F 3 "https://diotec.com/tl_files/diotec/files/pdf/datasheets/mm3z2v4.pdf" V 3550 5200 50  0001 C CNN
+F 4 "C152524" V 3550 5200 50  0001 C CNN "LCSC_PN"
+F 5 "SOD-323" V 3550 5200 50  0001 C CNN "LCSC_FP"
+	1    3550 5200
 	0    1    1    0
 $EndComp
 Wire Wire Line
-	8100 2650 8100 2750
+	4350 5350 4350 5450
 Wire Wire Line
-	8100 2350 8100 2450
+	4350 5050 4350 5150
 Wire Wire Line
-	7750 2350 7750 2400
+	4000 5050 4000 5100
 Wire Wire Line
-	7750 2350 8100 2350
+	4000 5050 4350 5050
 Wire Wire Line
-	7750 2350 7300 2350
+	4000 5050 3550 5050
 Wire Wire Line
-	7300 2350 7300 2400
-Connection ~ 7750 2350
+	3550 5050 3550 5100
+Connection ~ 4000 5050
 Wire Wire Line
-	8100 2750 7750 2750
+	4350 5450 4000 5450
 Wire Wire Line
-	7750 2750 7750 2600
+	4000 5450 4000 5300
 Wire Wire Line
-	7300 2600 7300 2750
+	3550 5300 3550 5450
 Wire Wire Line
-	7300 2750 7750 2750
-Connection ~ 7750 2750
-Connection ~ 8100 2350
+	3550 5450 4000 5450
+Connection ~ 4000 5450
+Connection ~ 4350 5050
 Wire Wire Line
 	7800 1850 7800 1550
@@
 Wire Wire Line
 	7300 2150 6950 2150
-Wire Wire Line
-	6950 2150 6950 2750
-Wire Wire Line
-	6950 2750 7300 2750
 Connection ~ 7300 2150
-Connection ~ 7300 2750
 Wire Wire Line
 	6800 1550 7300 1550
 Wire Wire Line
-	8100 2350 8400 2350
+	4350 5050 4650 5050
 Wire Wire Line
 	7600 2900 8300 2900
@@
 	7900 3300 8300 3300
 Wire Wire Line
-	6950 2750 6950 4050
-Wire Wire Line
 	6950 4050 7450 4050
-Connection ~ 6950 2750
 Connection ~ 6950 4050
 Wire Wire Line
@@
 L Device:C_Small C51
 U 1 1 60C40E4D
-P 8450 2550
-F 0 "C51" H 8542 2596 50  0000 L CNN
-F 1 "0.1u" H 8542 2505 50  0000 L CNN
-F 2 "Capacitor_SMD:C_1206_3216Metric_Pad1.33x1.80mm_HandSolder" H 8450 2550 50  0001 C CNN
-F 3 "https://datasheet.lcsc.com/lcsc/1805021622_KEMET-C1206C104K5RAC7800_C141184.pdf" H 8450 2550 50  0001 C CNN
-F 4 "C141184" H 8450 2550 50  0001 C CNN "LCSC_PN"
-F 5 "1206" H 8450 2550 50  0001 C CNN "LCSC_FP"
-	1    8450 2550
+P 4700 5250
+F 0 "C51" H 4792 5296 50  0000 L CNN
+F 1 "0.1u" H 4792 5205 50  0000 L CNN
+F 2 "Capacitor_SMD:C_1206_3216Metric_Pad1.33x1.80mm_HandSolder" H 4700 5250 50  0001 C CNN
+F 3 "https://datasheet.lcsc.com/lcsc/1805021622_KEMET-C1206C104K5RAC7800_C141184.pdf" H 4700 5250 50  0001 C CNN
+F 4 "C141184" H 4700 5250 50  0001 C CNN "LCSC_PN"
+F 5 "1206" H 4700 5250 50  0001 C CNN "LCSC_FP"
+	1    4700 5250
 	1    0    0    -1
 $EndComp
 Wire Wire Line
-	8450 2450 8450 2350
-Connection ~ 8450 2350
+	4700 5150 4700 5050
+Connection ~ 4700 5050
 Wire Wire Line
-	8450 2350 8500 2350
+	4700 5050 4750 5050
 Wire Wire Line
-	8450 2650 8450 2750
+	4700 5350 4700 5450
 Wire Wire Line
-	8450 2750 8100 2750
-Connection ~ 8100 2750
+	4700 5450 4350 5450
+Connection ~ 4350 5450
 $Comp
 L Connector:TestPoint_Small TP14
@@
 L Connector:TestPoint_Small TP15
 U 1 1 60D88AC9
-P 8450 2150
-F 0 "TP15" H 8498 2196 50  0000 L CNN
-F 1 "TP_VPROT" H 8498 2105 50  0000 L CNN
-F 2 "TestPoint:TestPoint_Pad_D1.0mm" H 8650 2150 50  0001 C CNN
-F 3 "~" H 8650 2150 50  0001 C CNN
-	1    8450 2150
+P 4700 4850
+F 0 "TP15" H 4748 4896 50  0000 L CNN
+F 1 "TP_VPROT" H 4748 4805 50  0000 L CNN
+F 2 "TestPoint:TestPoint_Pad_D1.0mm" H 4900 4850 50  0001 C CNN
+F 3 "~" H 4900 4850 50  0001 C CNN
+	1    4700 4850
 	1    0    0    -1
 $EndComp
 Wire Wire Line
-	8450 2150 8400 2150
+	4700 4850 4650 4850
 Wire Wire Line
-	8400 2150 8400 2350
-Connection ~ 8400 2350
+	4650 4850 4650 5050
+Connection ~ 4650 5050
 Wire Wire Line
-	8400 2350 8450 2350
+	4650 5050 4700 5050
 $Comp
 L Connector:TestPoint_Small TP13
@@
 Wire Wire Line
 	8300 2900 8500 2900
+Wire Wire Line
+	6950 2150 6950 4050
 $EndSCHEMATC

Commit message: Update Schematic with a bunch of extra stuff
Parts:
- removed C46: 47u, Capacitor_SMD:CP_Elec_5x5.8, symbol Device:CP_Small
- removed C48: 10u, Capacitor_Tantalum_SMD:CP_EIA-7343-20_Kemet-V_Pad2.25x2.55mm_HandSolder, symbol Device:CP_Small
- removed C49, C50, C51: 0.1u, Capacitor_SMD:C_1206_3216Metric_Pad1.33x1.80mm_HandSolder, symbol Device:C_Small
- removed D20, D21: MM3Zxx, Diode_SMD:D_SOD-323_HandSoldering, symbol Device:D_Small
- removed RV1: Varistor, Varistor:RV_Disc_D15.5mm_W3.9mm_P7.5mm, symbol Device:Varistor
- removed TP15: TP_VPROT, TestPoint:TestPoint_Pad_D1.0mm, symbol Connector:TestPoint_Small
Changed lines of the file:
@@
 $Descr A4 11693 8268
 encoding utf-8
-Sheet 9 9
-Title "Speeduino STM32"
+Sheet 9 10
+Title "DaveECU2"
 Date "2021-04-20"
 Rev "v0.1"
@@
 NoConn ~ 3050 2900
 $Comp
-L Device:Varistor RV1
-U 1 1 60B45CFD
-P 7300 1900
-F 0 "RV1" H 7179 1854 50  0000 R CNN
-F 1 "Varistor" H 7179 1945 50  0000 R CNN
-F 2 "Varistor:RV_Disc_D15.5mm_W3.9mm_P7.5mm" V 7230 1900 50  0001 C CNN
-F 3 "http://industrial.panasonic.com/www-cgi/jvcr13pz.cgi?E+PZ+3+AWA0002+ERZV14D220+7+WW" H 7300 1900 50  0001 C CNN
-F 4 "C1527916" H 7300 1900 50  0001 C CNN "LCSC_PN"
-F 5 "Disc15.5mm" H 7300 1900 50  0001 C CNN "LCSC_FP"
-F 6 "P7307-ND" H 7300 1900 50  0001 C CNN "DIGIKEY"
-	1    7300 1900
-	-1   0    0    1
-$EndComp
-$Comp
-L Device:C_Small C49
-U 1 1 60B470D5
-P 8100 1950
-F 0 "C49" H 8192 1996 50  0000 L CNN
-F 1 "0.1u" H 8192 1905 50  0000 L CNN
-F 2 "Capacitor_SMD:C_1206_3216Metric_Pad1.33x1.80mm_HandSolder" H 8100 1950 50  0001 C CNN
-F 3 "https://datasheet.lcsc.com/lcsc/1805021622_KEMET-C1206C104K5RAC7800_C141184.pdf" H 8100 1950 50  0001 C CNN
-F 4 "C141184" H 8100 1950 50  0001 C CNN "LCSC_PN"
-F 5 "1206" H 8100 1950 50  0001 C CNN "LCSC_FP"
-	1    8100 1950
-	1    0    0    -1
-$EndComp
-Text HLabel 6800 1550 0    50   Input ~ 0
-VBAT
-Wire Wire Line
-	7300 1550 7300 1750
-Wire Wire Line
-	7800 1550 7300 1550
-Connection ~ 7300 1550
-$Comp
 L Device:C_Small C47
 U 1 1 60B55285
@@
 	1    0    0    -1
 $EndComp
-$Comp
-L Device:D_Small D21
-U 1 1 60B5A34C
-P 8400 1550
-F 0 "D21" H 8400 1343 50  0000 C CNN
-F 1 "MM3Zxx" H 8400 1434 50  0000 C CNN
-F 2 "Diode_SMD:D_SOD-323_HandSoldering" V 8400 1550 50  0001 C CNN
-F 3 "https://datasheet.lcsc.com/lcsc/1809111719_ON-Semiconductor-SZMM3Z5V1ST1G_C152524.pdf" V 8400 1550 50  0001 C CNN
-F 4 "C152524" H 8400 1550 50  0001 C CNN "LCSC_PN"
-F 5 "SOD-323" H 8400 1550 50  0001 C CNN "LCSC_FP"
-	1    8400 1550
-	-1   0    0    1
-$EndComp
-Wire Wire Line
-	7800 1550 8100 1550
-Wire Wire Line
-	8100 1550 8100 1850
-Connection ~ 7800 1550
-Wire Wire Line
-	8100 1550 8300 1550
-Connection ~ 8100 1550
 Text GLabel 2950 3100 0    50   Input ~ 0
 VREG
-Text GLabel 8500 1550 2    50   Input ~ 0
-VREG
-Wire Wire Line
-	7300 2050 7300 2150
-Wire Wire Line
-	7300 2150 7800 2150
-Wire Wire Line
-	7800 2050 7800 2150
-Connection ~ 7800 2150
-Wire Wire Line
-	7800 2150 8100 2150
-Wire Wire Line
-	8100 2050 8100 2150
 $Comp
 L Device:Q_PNP_BEC Q2
@@
 Wire Wire Line
 	7750 4050 7750 3900
-Text GLabel 4750 5050 2    50   Input ~ 0
-VPROT
 Text GLabel 4300 3900 3    50   Input ~ 0
 VPROT
-$Comp
-L Device:C_Small C50
-U 1 1 60B98827
-P 4350 5250
-F 0 "C50" H 4442 5296 50  0000 L CNN
-F 1 "0.1u" H 4442 5205 50  0000 L CNN
-F 2 "Capacitor_SMD:C_1206_3216Metric_Pad1.33x1.80mm_HandSolder" H 4350 5250 50  0001 C CNN
-F 3 "https://datasheet.lcsc.com/lcsc/1805021622_KEMET-C1206C104K5RAC7800_C141184.pdf" H 4350 5250 50  0001 C CNN
-F 4 "C141184" H 4350 5250 50  0001 C CNN "LCSC_PN"
-F 5 "1206" H 4350 5250 50  0001 C CNN "LCSC_FP"
-	1    4350 5250
-	1    0    0    -1
-$EndComp
-$Comp
-L Device:CP_Small C46
-U 1 1 60B98E5B
-P 4000 5200
-F 0 "C46" H 4088 5246 50  0000 L CNN
-F 1 "47u" H 4088 5155 50  0000 L CNN
-F 2 "Capacitor_SMD:CP_Elec_5x5.8" H 4000 5200 50  0001 C CNN
-F 3 "https://datasheet.lcsc.com/lcsc/1912111437_PANASONIC-EEEFK0J470AR_C336380.pdf" H 4000 5200 50  0001 C CNN
-F 4 "C336380" H 4000 5200 50  0001 C CNN "LCSC_PN"
-F 5 "SMD,5x5.8mm" H 4000 5200 50  0001 C CNN "LCSC_FP"
-	1    4000 5200
-	1    0    0    -1
-$EndComp
-$Comp
-L Device:D_Small D20
-U 1 1 60B9A71D
-P 3550 5200
-F 0 "D20" V 3504 5270 50  0000 L CNN
-F 1 "MM3Zxx" V 3595 5270 50  0000 L CNN
-F 2 "Diode_SMD:D_SOD-323_HandSoldering" V 3550 5200 50  0001 C CNN
-F 3 "https://diotec.com/tl_files/diotec/files/pdf/datasheets/mm3z2v4.pdf" V 3550 5200 50  0001 C CNN
-F 4 "C152524" V 3550 5200 50  0001 C CNN "LCSC_PN"
-F 5 "SOD-323" V 3550 5200 50  0001 C CNN "LCSC_FP"
-	1    3550 5200
-	0    1    1    0
-$EndComp
-Wire Wire Line
-	4350 5350 4350 5450
-Wire Wire Line
-	4350 5050 4350 5150
-Wire Wire Line
-	4000 5050 4000 5100
-Wire Wire Line
-	4000 5050 4350 5050
-Wire Wire Line
-	4000 5050 3550 5050
-Wire Wire Line
-	3550 5050 3550 5100
-Connection ~ 4000 5050
-Wire Wire Line
-	4350 5450 4000 5450
-Wire Wire Line
-	4000 5450 4000 5300
-Wire Wire Line
-	3550 5300 3550 5450
-Wire Wire Line
-	3550 5450 4000 5450
-Connection ~ 4000 5450
-Connection ~ 4350 5050
-Wire Wire Line
-	7800 1850 7800 1550
-$Comp
-L Device:CP_Small C48
-U 1 1 60B4695A
-P 7800 1950
-F 0 "C48" H 7888 1996 50  0000 L CNN
-F 1 "10u" H 7888 1905 50  0000 L CNN
-F 2 "Capacitor_Tantalum_SMD:CP_EIA-7343-20_Kemet-V_Pad2.25x2.55mm_HandSolder" H 7800 1950 50  0001 C CNN
-F 3 "https://datasheet.lcsc.com/lcsc/1809200017_KEMET-T491D106K050AT_C117038.pdf" H 7800 1950 50  0001 C CNN
-F 4 "C117038" H 7800 1950 50  0001 C CNN "LCSC_PN"
-F 5 "CASE-D_7343" H 7800 1950 50  0001 C CNN "LCSC_FP"
-	1    7800 1950
-	1    0    0    -1
-$EndComp
-Wire Wire Line
-	7300 2150 6950 2150
-Connection ~ 7300 2150
-Wire Wire Line
-	6800 1550 7300 1550
-Wire Wire Line
-	4350 5050 4650 5050
 Wire Wire Line
 	7600 2900 8300 2900
@@
 Wire Wire Line
 	6950 4050 7450 4050
-Connection ~ 6950 4050
 Wire Wire Line
 	7450 4050 7750 4050
@@
 Wire Wire Line
 	6950 4050 6950 4100
-$Comp
-L Device:C_Small C51
-U 1 1 60C40E4D
-P 4700 5250
-F 0 "C51" H 4792 5296 50  0000 L CNN
-F 1 "0.1u" H 4792 5205 50  0000 L CNN
-F 2 "Capacitor_SMD:C_1206_3216Metric_Pad1.33x1.80mm_HandSolder" H 4700 5250 50  0001 C CNN
-F 3 "https://datasheet.lcsc.com/lcsc/1805021622_KEMET-C1206C104K5RAC7800_C141184.pdf" H 4700 5250 50  0001 C CNN
-F 4 "C141184" H 4700 5250 50  0001 C CNN "LCSC_PN"
-F 5 "1206" H 4700 5250 50  0001 C CNN "LCSC_FP"
-	1    4700 5250
-	1    0    0    -1
-$EndComp
-Wire Wire Line
-	4700 5150 4700 5050
-Connection ~ 4700 5050
-Wire Wire Line
-	4700 5050 4750 5050
-Wire Wire Line
-	4700 5350 4700 5450
-Wire Wire Line
-	4700 5450 4350 5450
-Connection ~ 4350 5450
 $Comp
 L Connector:TestPoint_Small TP14
@@
 	8300 3600 8500 3600
 $Comp
-L Connector:TestPoint_Small TP15
-U 1 1 60D88AC9
-P 4700 4850
-F 0 "TP15" H 4748 4896 50  0000 L CNN
-F 1 "TP_VPROT" H 4748 4805 50  0000 L CNN
-F 2 "TestPoint:TestPoint_Pad_D1.0mm" H 4900 4850 50  0001 C CNN
-F 3 "~" H 4900 4850 50  0001 C CNN
-	1    4700 4850
-	1    0    0    -1
-$EndComp
-Wire Wire Line
-	4700 4850 4650 4850
-Wire Wire Line
-	4650 4850 4650 5050
-Connection ~ 4650 5050
-Wire Wire Line
-	4650 5050 4700 5050
-$Comp
 L Connector:TestPoint_Small TP13
 U 1 1 60D8A8F2
@@
 Wire Wire Line
 	8300 2900 8500 2900
-Wire Wire Line
-	6950 2150 6950 4050
 $EndSCHEMATC
