File: Injectors.sch (KiCad schematic (older format))
At the start: 22 parts

Commit message: Starting on layout
Parts:
- R10, R11, R12, R13, R2, R3, R4, R5, R6, R7, R8, R9: renamed from R?; footprint (none) -> Resistor_SMD:R_0603_1608Metric_Pad1.05x0.95mm_HandSolder
- gave numbers to parts that had none: 10
Changed lines of the file:
@@
 $Descr A4 11693 8268
 encoding utf-8
-Sheet 2 9
+Sheet 2 10
 Title ""
 Date ""
@@
 P 2550 1950
 AR Path="/5EEDBC10" Ref="U?"  Part="1"
-AR Path="/5EEDB4C5/5EEDBC10" Ref="U?"  Part="1"
-F 0 "U?" H 2650 2517 50  0000 C CNN
+AR Path="/5EEDB4C5/5EEDBC10" Ref="U2"  Part="1"
+F 0 "U2" H 2650 2517 50  0000 C CNN
 F 1 "VNLD5090" H 2650 2426 50  0000 C CNN
 F 2 "Package_SO:SO-8_3.9x4.9mm_P1.27mm" H 2750 1250 50  0001 C CNN
@@
 $EndComp
 $Comp
-L Device:R R?
+L Device:R R3
 U 1 1 5EEDE368
 P 1500 1750
-F 0 "R?" V 1293 1750 50  0000 C CNN
+F 0 "R3" V 1293 1750 50  0000 C CNN
 F 1 "1k" V 1384 1750 50  0000 C CNN
-F 2 "" V 1430 1750 50  0001 C CNN
+F 2 "Resistor_SMD:R_0603_1608Metric_Pad1.05x0.95mm_HandSolder" V 1430 1750 50  0001 C CNN
 F 3 "~" H 1500 1750 50  0001 C CNN
 F 4 "311-1.00KCRCT-ND" V 1500 1750 50  0001 C CNN "DIGIKEY"
@@
 	1200 2050 1000 2050
 $Comp
-L Device:R R?
+L Device:R R2
 U 1 1 5EEE7DB3
 P 1500 900
-F 0 "R?" V 1293 900 50  0000 C CNN
+F 0 "R2" V 1293 900 50  0000 C CNN
 F 1 "100k" V 1384 900 50  0000 C CNN
-F 2 "" V 1430 900 50  0001 C CNN
+F 2 "Resistor_SMD:R_0603_1608Metric_Pad1.05x0.95mm_HandSolder" V 1430 900 50  0001 C CNN
 F 3 "~" H 1500 900 50  0001 C CNN
 F 4 "311-100KCRCT-ND" V 1500 900 50  0001 C CNN "DIGIKEY"
@@
 12v-SW
 $Comp
-L Device:R R?
+L Device:R R10
 U 1 1 5EF06411
 P 3900 1150
-F 0 "R?" V 3693 1150 50  0000 C CNN
+F 0 "R10" V 3693 1150 50  0000 C CNN
 F 1 "2.4k" V 3784 1150 50  0000 C CNN
-F 2 "" V 3830 1150 50  0001 C CNN
+F 2 "Resistor_SMD:R_0603_1608Metric_Pad1.05x0.95mm_HandSolder" V 3830 1150 50  0001 C CNN
 F 3 "~" H 3900 1150 50  0001 C CNN
 F 4 "311-2.40KCRCT-ND" V 3900 1150 50  0001 C CNN "DIGIKEY"
@@
 	3750 1150 3450 1150
 $Comp
-L Device:LED D?
+L Device:LED D1
 U 1 1 5EF06418
 P 4450 1150
-F 0 "D?" H 4443 895 50  0000 C CNN
+F 0 "D1" H 4443 895 50  0000 C CNN
 F 1 "LED" H 4443 986 50  0000 C CNN
 F 2 "LED_SMD:LED_0805_2012Metric_Pad1.15x1.40mm_HandSolder" H 4450 1150 50  0001 C CNN
@@
 	4300 1150 4050 1150
 $Comp
-L Device:D D?
+L Device:D D5
 U 1 1 5EF0641F
 P 5100 1150
-F 0 "D?" H 5100 933 50  0000 C CNN
+F 0 "D5" H 5100 933 50  0000 C CNN
 F 1 "D" H 5100 1024 50  0000 C CNN
 F 2 "Diode_SMD:D_SOD-323_HandSoldering" H 5100 1150 50  0001 C CNN
@@
 	5400 5100 5400 4500
 $Comp
-L Device:R R?
+L Device:R R11
 U 1 1 5F791B22
 P 3900 3200
-F 0 "R?" V 3693 3200 50  0000 C CNN
+F 0 "R11" V 3693 3200 50  0000 C CNN
 F 1 "2.4k" V 3784 3200 50  0000 C CNN
-F 2 "" V 3830 3200 50  0001 C CNN
+F 2 "Resistor_SMD:R_0603_1608Metric_Pad1.05x0.95mm_HandSolder" V 3830 3200 50  0001 C CNN
 F 3 "~" H 3900 3200 50  0001 C CNN
 F 4 "311-2.40KCRCT-ND" V 3900 3200 50  0001 C CNN "DIGIKEY"
@@
 $EndComp
 $Comp
-L Device:R R?
+L Device:R R5
 U 1 1 5F7933D6
 P 1500 2850
-F 0 "R?" V 1293 2850 50  0000 C CNN
+F 0 "R5" V 1293 2850 50  0000 C CNN
 F 1 "100k" V 1384 2850 50  0000 C CNN
-F 2 "" V 1430 2850 50  0001 C CNN
+F 2 "Resistor_SMD:R_0603_1608Metric_Pad1.05x0.95mm_HandSolder" V 1430 2850 50  0001 C CNN
 F 3 "~" H 1500 2850 50  0001 C CNN
 F 4 "311-100KCRCT-ND" V 1500 2850 50  0001 C CNN "DIGIKEY"
@@
 $EndComp
 $Comp
-L Device:R R?
+L Device:R R4
 U 1 1 5F794925
 P 1500 2050
-F 0 "R?" V 1293 2050 50  0000 C CNN
+F 0 "R4" V 1293 2050 50  0000 C CNN
 F 1 "1k" V 1384 2050 50  0000 C CNN
-F 2 "" V 1430 2050 50  0001 C CNN
+F 2 "Resistor_SMD:R_0603_1608Metric_Pad1.05x0.95mm_HandSolder" V 1430 2050 50  0001 C CNN
 F 3 "~" H 1500 2050 50  0001 C CNN
 F 4 "311-1.00KCRCT-ND" V 1500 2050 50  0001 C CNN "DIGIKEY"
@@
 $EndComp
 $Comp
-L Device:D D?
+L Device:D D6
 U 1 1 5F7960E4
 P 5100 3200
-F 0 "D?" H 5100 2983 50  0000 C CNN
+F 0 "D6" H 5100 2983 50  0000 C CNN
 F 1 "D" H 5100 3074 50  0000 C CNN
 F 2 "Diode_SMD:D_SOD-323_HandSoldering" H 5100 3200 50  0001 C CNN
@@
 Connection ~ 5250 3200
 $Comp
-L Device:LED D?
+L Device:LED D2
 U 1 1 5F797CCC
 P 4450 3200
-F 0 "D?" H 4443 2945 50  0000 C CNN
+F 0 "D2" H 4443 2945 50  0000 C CNN
 F 1 "LED" H 4443 3036 50  0000 C CNN
 F 2 "LED_SMD:LED_0805_2012Metric_Pad1.15x1.40mm_HandSolder" H 4450 3200 50  0001 C CNN
@@
 P 2700 5300
 AR Path="/5F79AB0C" Ref="U?"  Part="1"
-AR Path="/5EEDB4C5/5F79AB0C" Ref="U?"  Part="1"
-F 0 "U?" H 2800 5867 50  0000 C CNN
+AR Path="/5EEDB4C5/5F79AB0C" Ref="U3"  Part="1"
+F 0 "U3" H 2800 5867 50  0000 C CNN
 F 1 "VNLD5090" H 2800 5776 50  0000 C CNN
 F 2 "Package_SO:SO-8_3.9x4.9mm_P1.27mm" H 2900 4600 50  0001 C CNN
@@
 $EndComp
 $Comp
-L Device:D D?
+L Device:D D7
 U 1 1 5F79C130
 P 5250 4500
-F 0 "D?" H 5250 4283 50  0000 C CNN
+F 0 "D7" H 5250 4283 50  0000 C CNN
 F 1 "D" H 5250 4374 50  0000 C CNN
 F 2 "Diode_SMD:D_SOD-323_HandSoldering" H 5250 4500 50  0001 C CNN
@@
 $EndComp
 $Comp
-L Device:D D?
+L Device:D D8
 U 1 1 5F79C951
 P 5250 6550
-F 0 "D?" H 5250 6333 50  0000 C CNN
+F 0 "D8" H 5250 6333 50  0000 C CNN
 F 1 "D" H 5250 6424 50  0000 C CNN
 F 2 "Diode_SMD:D_SOD-323_HandSoldering" H 5250 6550 50  0001 C CNN
@@
 Connection ~ 5400 4500
 $Comp
-L Device:LED D?
+L Device:LED D3
 U 1 1 5F79FF70
 P 4600 4500
-F 0 "D?" H 4593 4245 50  0000 C CNN
+F 0 "D3" H 4593 4245 50  0000 C CNN
 F 1 "LED" H 4593 4336 50  0000 C CNN
 F 2 "LED_SMD:LED_0805_2012Metric_Pad1.15x1.40mm_HandSolder" H 4600 4500 50  0001 C CNN
@@
 $EndComp
 $Comp
-L Device:LED D?
+L Device:LED D4
 U 1 1 5F7A0421
 P 4600 6550
-F 0 "D?" H 4593 6295 50  0000 C CNN
+F 0 "D4" H 4593 6295 50  0000 C CNN
 F 1 "LED" H 4593 6386 50  0000 C CNN
 F 2 "LED_SMD:LED_0805_2012Metric_Pad1.15x1.40mm_HandSolder" H 4600 6550 50  0001 C CNN
@@
 $EndComp
 $Comp
-L Device:R R?
+L Device:R R12
 U 1 1 5F7AE86B
 P 4050 4500
-F 0 "R?" V 3843 4500 50  0000 C CNN
+F 0 "R12" V 3843 4500 50  0000 C CNN
 F 1 "2.4k" V 3934 4500 50  0000 C CNN
-F 2 "" V 3980 4500 50  0001 C CNN
+F 2 "Resistor_SMD:R_0603_1608Metric_Pad1.05x0.95mm_HandSolder" V 3980 4500 50  0001 C CNN
 F 3 "~" H 4050 4500 50  0001 C CNN
 F 4 "311-2.40KCRCT-ND" V 4050 4500 50  0001 C CNN "DIGIKEY"
@@
 $EndComp
 $Comp
-L Device:R R?
+L Device:R R13
 U 1 1 5F7AECAC
 P 4050 6550
-F 0 "R?" V 3843 6550 50  0000 C CNN
+F 0 "R13" V 3843 6550 50  0000 C CNN
 F 1 "2.4k" V 3934 6550 50  0000 C CNN
-F 2 "" V 3980 6550 50  0001 C CNN
+F 2 "Resistor_SMD:R_0603_1608Metric_Pad1.05x0.95mm_HandSolder" V 3980 6550 50  0001 C CNN
 F 3 "~" H 4050 6550 50  0001 C CNN
 F 4 "311-2.40KCRCT-ND" V 4050 6550 50  0001 C CNN "DIGIKEY"
@@
 $EndComp
 $Comp
-L Device:R R?
+L Device:R R9
 U 1 1 5F7B0FF1
 P 1650 6200
-F 0 "R?" V 1443 6200 50  0000 C CNN
+F 0 "R9" V 1443 6200 50  0000 C CNN
 F 1 "100k" V 1534 6200 50  0000 C CNN
-F 2 "" V 1580 6200 50  0001 C CNN
+F 2 "Resistor_SMD:R_0603_1608Metric_Pad1.05x0.95mm_HandSolder" V 1580 6200 50  0001 C CNN
 F 3 "~" H 1650 6200 50  0001 C CNN
 F 4 "311-100KCRCT-ND" V 1650 6200 50  0001 C CNN "DIGIKEY"
@@
 $EndComp
 $Comp
-L Device:R R?
+L Device:R R6
 U 1 1 5F7B3D3C
 P 1650 4250
-F 0 "R?" V 1443 4250 50  0000 C CNN
+F 0 "R6" V 1443 4250 50  0000 C CNN
 F 1 "100k" V 1534 4250 50  0000 C CNN
-F 2 "" V 1580 4250 50  0001 C CNN
+F 2 "Resistor_SMD:R_0603_1608Metric_Pad1.05x0.95mm_HandSolder" V 1580 4250 50  0001 C CNN
 F 3 "~" H 1650 4250 50  0001 C CNN
 F 4 "311-100KCRCT-ND" V 1650 4250 50  0001 C CNN "DIGIKEY"
@@
 $EndComp
 $Comp
-L Device:R R?
+L Device:R R7
 U 1 1 5F7B4559
 P 1650 5100
-F 0 "R?" V 1443 5100 50  0000 C CNN
+F 0 "R7" V 1443 5100 50  0000 C CNN
 F 1 "1k" V 1534 5100 50  0000 C CNN
-F 2 "" V 1580 5100 50  0001 C CNN
+F 2 "Resistor_SMD:R_0603_1608Metric_Pad1.05x0.95mm_HandSolder" V 1580 5100 50  0001 C CNN
 F 3 "~" H 1650 5100 50  0001 C CNN
 F 4 "311-1.00KCRCT-ND" V 1650 5100 50  0001 C CNN "DIGIKEY"
@@
 $EndComp
 $Comp
-L Device:R R?
+L Device:R R8
 U 1 1 5F7B74AF
 P 1650 5400
-F 0 "R?" V 1443 5400 50  0000 C CNN
+F 0 "R8" V 1443 5400 50  0000 C CNN
 F 1 "1k" V 1534 5400 50  0000 C CNN
-F 2 "" V 1580 5400 50  0001 C CNN
+F 2 "Resistor_SMD:R_0603_1608Metric_Pad1.05x0.95mm_HandSolder" V 1580 5400 50  0001 C CNN
 F 3 "~" H 1650 5400 50  0001 C CNN
 F 4 "311-1.00KCRCT-ND" V 1650 5400 50  0001 C CNN "DIGIKEY"

Commit message: restart a third time
Parts:
- D12: renamed from D1; footprint LED_SMD:LED_0805_2012Metric_Pad1.15x1.40mm_HandSolder -> LED_SMD:LED_0603_1608Metric_Pad1.05x0.95mm_HandSolder
- D13: renamed from D2; footprint LED_SMD:LED_0805_2012Metric_Pad1.15x1.40mm_HandSolder -> LED_SMD:LED_0603_1608Metric_Pad1.05x0.95mm_HandSolder
- D14: renamed from D3; footprint LED_SMD:LED_0805_2012Metric_Pad1.15x1.40mm_HandSolder -> LED_SMD:LED_0603_1608Metric_Pad1.05x0.95mm_HandSolder
- D15: renamed from D4; footprint LED_SMD:LED_0805_2012Metric_Pad1.15x1.40mm_HandSolder -> LED_SMD:LED_0603_1608Metric_Pad1.05x0.95mm_HandSolder
- D16: renamed from D5; value D -> 1N4448WS
- D17: renamed from D6; value D -> 1N4448WS
- D18: renamed from D7; value D -> 1N4448WS
- D19: renamed from D8; value D -> 1N4448WS
- R61: renamed from R2; footprint Resistor_SMD:R_0603_1608Metric_Pad1.05x0.95mm_HandSolder -> Resistor_SMD:R_0603_1608Metric_Pad0.98x0.95mm_HandSolder
- R62: renamed from R3; footprint Resistor_SMD:R_0603_1608Metric_Pad1.05x0.95mm_HandSolder -> Resistor_SMD:R_0603_1608Metric_Pad0.98x0.95mm_HandSolder
- R63: renamed from R4; footprint Resistor_SMD:R_0603_1608Metric_Pad1.05x0.95mm_HandSolder -> Resistor_SMD:R_0603_1608Metric_Pad0.98x0.95mm_HandSolder
- R64: renamed from R5; footprint Resistor_SMD:R_0603_1608Metric_Pad1.05x0.95mm_HandSolder -> Resistor_SMD:R_0603_1608Metric_Pad0.98x0.95mm_HandSolder
- R65: renamed from R6; footprint Resistor_SMD:R_0603_1608Metric_Pad1.05x0.95mm_HandSolder -> Resistor_SMD:R_0603_1608Metric_Pad0.98x0.95mm_HandSolder
- R66: renamed from R7; footprint Resistor_SMD:R_0603_1608Metric_Pad1.05x0.95mm_HandSolder -> Resistor_SMD:R_0603_1608Metric_Pad0.98x0.95mm_HandSolder
- R67: renamed from R8; footprint Resistor_SMD:R_0603_1608Metric_Pad1.05x0.95mm_HandSolder -> Resistor_SMD:R_0603_1608Metric_Pad0.98x0.95mm_HandSolder
- R68: renamed from R9; footprint Resistor_SMD:R_0603_1608Metric_Pad1.05x0.95mm_HandSolder -> Resistor_SMD:R_0603_1608Metric_Pad0.98x0.95mm_HandSolder
- R69: renamed from R10; footprint Resistor_SMD:R_0603_1608Metric_Pad1.05x0.95mm_HandSolder -> Resistor_SMD:R_0603_1608Metric_Pad0.98x0.95mm_HandSolder
- R70: renamed from R11; footprint Resistor_SMD:R_0603_1608Metric_Pad1.05x0.95mm_HandSolder -> Resistor_SMD:R_0603_1608Metric_Pad0.98x0.95mm_HandSolder
- R71: renamed from R12; footprint Resistor_SMD:R_0603_1608Metric_Pad1.05x0.95mm_HandSolder -> Resistor_SMD:R_0603_1608Metric_Pad0.98x0.95mm_HandSolder
- R72: renamed from R13; footprint Resistor_SMD:R_0603_1608Metric_Pad1.05x0.95mm_HandSolder -> Resistor_SMD:R_0603_1608Metric_Pad0.98x0.95mm_HandSolder
- U13: renamed from U2; footprint Package_SO:SO-8_3.9x4.9mm_P1.27mm -> Package_SO:SOIC-8_3.9x4.9mm_P1.27mm
- U14: renamed from U3; footprint Package_SO:SO-8_3.9x4.9mm_P1.27mm -> Package_SO:SOIC-8_3.9x4.9mm_P1.27mm
Connections:
- net CPU-D10 renamed MCU-INJ-1
- net CPU-D11 renamed MCU-INJ-2
- net CPU-D8 renamed MCU-INJ-4
- net CPU-D9 renamed MCU-INJ-3

Commit message: Update Schematic with a bunch of extra stuff
Connections:
- no-connect marks 0 -> 4
Changed lines of the file:
@@
 $Descr A4 11693 8268
 encoding utf-8
-Sheet 8 9
-Title "Speeduino STM32"
+Sheet 8 8
+Title "DaveECU2"
 Date "2021-04-20"
 Rev "v0.1"
@@
 Text HLabel 1150 5100 0    50   Input ~ 0
 MCU-INJ-3
+NoConn ~ 2150 1900
+NoConn ~ 2150 2200
+NoConn ~ 2300 5250
+NoConn ~ 2300 5550
 $EndSCHEMATC
