File: FAN+TACH.sch (KiCad schematic (older format))
At the start: 7 parts

Commit message: Starting on layout
Parts:
- JP1: renamed from JP?; footprint (none) -> Connector_PinHeader_2.54mm:PinHeader_1x02_P2.54mm_Vertical_SMD_Pin1Right
- R22, R23, R24, R25, R26: renamed from R?; footprint (none) -> Resistor_SMD:R_0603_1608Metric_Pad1.05x0.95mm_HandSolder
- gave numbers to parts that had none: 1
Changed lines of the file:
@@
 $Descr A4 11693 8268
 encoding utf-8
-Sheet 5 9
+Sheet 5 10
 Title ""
 Date ""
@@
 TACH-OUT
 $Comp
-L Device:Jumper JP?
+L Device:Jumper JP1
 U 1 1 5EFA7131
 P 7400 3350
-F 0 "JP?" H 7400 3614 50  0000 C CNN
+F 0 "JP1" H 7400 3614 50  0000 C CNN
 F 1 "Jumper" H 7400 3523 50  0000 C CNN
-F 2 "" H 7400 3350 50  0001 C CNN
+F 2 "Connector_PinHeader_2.54mm:PinHeader_1x02_P2.54mm_Vertical_SMD_Pin1Right" H 7400 3350 50  0001 C CNN
 F 3 "~" H 7400 3350 50  0001 C CNN
 	1    7400 3350
@@
 P 4150 3050
 AR Path="/5EEDB4C5/5F863141" Ref="R?"  Part="1"
-AR Path="/5EFA5E54/5F863141" Ref="R?"  Part="1"
-F 0 "R?" V 3943 3050 50  0000 C CNN
+AR Path="/5EFA5E54/5F863141" Ref="R22"  Part="1"
+F 0 "R22" V 3943 3050 50  0000 C CNN
 F 1 "1k" V 4034 3050 50  0000 C CNN
-F 2 "" V 4080 3050 50  0001 C CNN
+F 2 "Resistor_SMD:R_0603_1608Metric_Pad1.05x0.95mm_HandSolder" V 4080 3050 50  0001 C CNN
 F 3 "~" H 4150 3050 50  0001 C CNN
 F 4 "311-1.00KCRCT-ND" V 4150 3050 50  0001 C CNN "DIGIKEY"
@@
 P 4150 3350
 AR Path="/5EEDB4C5/5F865B33" Ref="R?"  Part="1"
-AR Path="/5EFA5E54/5F865B33" Ref="R?"  Part="1"
-F 0 "R?" V 3943 3350 50  0000 C CNN
+AR Path="/5EFA5E54/5F865B33" Ref="R23"  Part="1"
+F 0 "R23" V 3943 3350 50  0000 C CNN
 F 1 "1k" V 4034 3350 50  0000 C CNN
-F 2 "" V 4080 3350 50  0001 C CNN
+F 2 "Resistor_SMD:R_0603_1608Metric_Pad1.05x0.95mm_HandSolder" V 4080 3350 50  0001 C CNN
 F 3 "~" H 4150 3350 50  0001 C CNN
 F 4 "311-1.00KCRCT-ND" V 4150 3350 50  0001 C CNN "DIGIKEY"
@@
 P 4600 3750
 AR Path="/5EEDB4C5/5F86631A" Ref="R?"  Part="1"
-AR Path="/5EFA5E54/5F86631A" Ref="R?"  Part="1"
-F 0 "R?" H 4530 3704 50  0000 R CNN
+AR Path="/5EFA5E54/5F86631A" Ref="R25"  Part="1"
+F 0 "R25" H 4530 3704 50  0000 R CNN
 F 1 "100k" H 4530 3795 50  0000 R CNN
-F 2 "" V 4530 3750 50  0001 C CNN
+F 2 "Resistor_SMD:R_0603_1608Metric_Pad1.05x0.95mm_HandSolder" V 4530 3750 50  0001 C CNN
 F 3 "~" H 4600 3750 50  0001 C CNN
 F 4 "311-100KCRCT-ND" V 4600 3750 50  0001 C CNN "DIGIKEY"
@@
 P 4600 2750
 AR Path="/5EEDB4C5/5F868FC3" Ref="R?"  Part="1"
-AR Path="/5EFA5E54/5F868FC3" Ref="R?"  Part="1"
-F 0 "R?" H 4530 2704 50  0000 R CNN
+AR Path="/5EFA5E54/5F868FC3" Ref="R24"  Part="1"
+F 0 "R24" H 4530 2704 50  0000 R CNN
 F 1 "100k" H 4530 2795 50  0000 R CNN
-F 2 "" V 4530 2750 50  0001 C CNN
+F 2 "Resistor_SMD:R_0603_1608Metric_Pad1.05x0.95mm_HandSolder" V 4530 2750 50  0001 C CNN
 F 3 "~" H 4600 2750 50  0001 C CNN
 F 4 "311-100KCRCT-ND" V 4600 2750 50  0001 C CNN "DIGIKEY"
@@
 P 6950 3750
 AR Path="/5EEDB4C5/5F869342" Ref="R?"  Part="1"
-AR Path="/5EFA5E54/5F869342" Ref="R?"  Part="1"
-F 0 "R?" V 6743 3750 50  0000 C CNN
+AR Path="/5EFA5E54/5F869342" Ref="R26"  Part="1"
+F 0 "R26" V 6743 3750 50  0000 C CNN
 F 1 "1k" V 6834 3750 50  0000 C CNN
-F 2 "" V 6880 3750 50  0001 C CNN
+F 2 "Resistor_SMD:R_0603_1608Metric_Pad1.05x0.95mm_HandSolder" V 6880 3750 50  0001 C CNN
 F 3 "~" H 6950 3750 50  0001 C CNN
 F 4 "311-1.00KCRCT-ND" V 6950 3750 50  0001 C CNN "DIGIKEY"
@@
 AR Path="/5F8719C9" Ref="U?"  Part="1"
 AR Path="/5EEDB4C5/5F8719C9" Ref="U?"  Part="1"
-AR Path="/5EFA5E54/5F8719C9" Ref="U?"  Part="1"
-F 0 "U?" H 5500 3817 50  0000 C CNN
+AR Path="/5EFA5E54/5F8719C9" Ref="U6"  Part="1"
+F 0 "U6" H 5500 3817 50  0000 C CNN
 F 1 "VNLD5090" H 5500 3726 50  0000 C CNN
 F 2 "Package_SO:SO-8_3.9x4.9mm_P1.27mm" H 5600 2550 50  0001 C CNN

Commit message: restart a third time
Parts:
- added TP1: TP_TACH, TestPoint:TestPoint_Pad_D1.0mm, symbol Connector:TestPoint_Small
- JP1: footprint Connector_PinHeader_2.54mm:PinHeader_1x02_P2.54mm_Vertical_SMD_Pin1Right -> Jumper:SolderJumper-2_P1.3mm_Open_RoundedPad1.0x1.5mm
- R10: renamed from R23; footprint Resistor_SMD:R_0603_1608Metric_Pad1.05x0.95mm_HandSolder -> Resistor_SMD:R_0603_1608Metric_Pad0.98x0.95mm_HandSolder
- R11: renamed from R24; footprint Resistor_SMD:R_0603_1608Metric_Pad1.05x0.95mm_HandSolder -> Resistor_SMD:R_0603_1608Metric_Pad0.98x0.95mm_HandSolder
- R12: renamed from R25; footprint Resistor_SMD:R_0603_1608Metric_Pad1.05x0.95mm_HandSolder -> Resistor_SMD:R_0603_1608Metric_Pad0.98x0.95mm_HandSolder
- R13: renamed from R26; footprint Resistor_SMD:R_0603_1608Metric_Pad1.05x0.95mm_HandSolder -> Resistor_SMD:R_0603_1608Metric_Pad0.98x0.95mm_HandSolder
- R9: renamed from R22; footprint Resistor_SMD:R_0603_1608Metric_Pad1.05x0.95mm_HandSolder -> Resistor_SMD:R_0603_1608Metric_Pad0.98x0.95mm_HandSolder
- U3: renamed from U6; footprint Package_SO:SO-8_3.9x4.9mm_P1.27mm -> Package_SO:SOIC-8_3.9x4.9mm_P1.27mm
Connections:
- net TACH-OUT: now also TP1.1
- net CPU-D35 renamed MCU-FAN
- net CPU-D49 renamed MCU-TACH
Changed lines of the file:
@@
 $Descr A4 11693 8268
 encoding utf-8
-Sheet 5 10
-Title ""
-Date ""
-Rev ""
+Sheet 4 9
+Title "Speeduino STM32"
+Date "2021-04-20"
+Rev "v0.1"
 Comp ""
 Comment1 ""
@@
 12v-SW
 Text HLabel 3550 3050 0    50   Input ~ 0
-CPU-D35
+MCU-FAN
 Text HLabel 3550 3350 0    50   Input ~ 0
-CPU-D49
+MCU-TACH
 Text HLabel 7950 3000 2    50   Output ~ 0
 FAN-OUT
@@
 F 0 "JP1" H 7400 3614 50  0000 C CNN
 F 1 "Jumper" H 7400 3523 50  0000 C CNN
-F 2 "Connector_PinHeader_2.54mm:PinHeader_1x02_P2.54mm_Vertical_SMD_Pin1Right" H 7400 3350 50  0001 C CNN
+F 2 "Jumper:SolderJumper-2_P1.3mm_Open_RoundedPad1.0x1.5mm" H 7400 3350 50  0001 C CNN
 F 3 "~" H 7400 3350 50  0001 C CNN
 	1    7400 3350
@@
 $EndComp
 $Comp
-L power:GND #PWR0116
+L power:GND #PWR014
 U 1 1 5EFA7CCD
 P 6250 3750
-F 0 "#PWR0116" H 6250 3500 50  0001 C CNN
+F 0 "#PWR014" H 6250 3500 50  0001 C CNN
 F 1 "GND" H 6255 3577 50  0000 C CNN
 F 2 "" H 6250 3750 50  0001 C CNN
@@
 	6550 3350 7100 3350
 Connection ~ 6550 3350
-Wire Wire Line
-	7950 3350 7700 3350
-$Comp
-L power:GND #PWR0117
+$Comp
+L power:GND #PWR015
 U 1 1 5EFAD44E
 P 6550 3200
-F 0 "#PWR0117" H 6550 2950 50  0001 C CNN
+F 0 "#PWR015" H 6550 2950 50  0001 C CNN
 F 1 "GND" V 6555 3072 50  0000 R CNN
 F 2 "" H 6550 3200 50  0001 C CNN
@@
 Connection ~ 4600 3050
 $Comp
-L power:GND #PWR0118
+L power:GND #PWR012
 U 1 1 5EFB270F
 P 4600 2250
-F 0 "#PWR0118" H 4600 2000 50  0001 C CNN
+F 0 "#PWR012" H 4600 2000 50  0001 C CNN
 F 1 "GND" H 4605 2077 50  0000 C CNN
 F 2 "" H 4600 2250 50  0001 C CNN
@@
 	5000 3350 4600 3350
 $Comp
-L power:GND #PWR0119
+L power:GND #PWR013
 U 1 1 5EFB892E
 P 4600 4450
-F 0 "#PWR0119" H 4600 4200 50  0001 C CNN
+F 0 "#PWR013" H 4600 4200 50  0001 C CNN
 F 1 "GND" H 4605 4277 50  0000 C CNN
 F 2 "" H 4600 4450 50  0001 C CNN
@@
 P 4150 3050
 AR Path="/5EEDB4C5/5F863141" Ref="R?"  Part="1"
-AR Path="/5EFA5E54/5F863141" Ref="R22"  Part="1"
-F 0 "R22" V 3943 3050 50  0000 C CNN
+AR Path="/5EFA5E54/5F863141" Ref="R9"  Part="1"
+F 0 "R9" V 3943 3050 50  0000 C CNN
 F 1 "1k" V 4034 3050 50  0000 C CNN
-F 2 "Resistor_SMD:R_0603_1608Metric_Pad1.05x0.95mm_HandSolder" V 4080 3050 50  0001 C CNN
+F 2 "Resistor_SMD:R_0603_1608Metric_Pad0.98x0.95mm_HandSolder" V 4080 3050 50  0001 C CNN
 F 3 "~" H 4150 3050 50  0001 C CNN
 F 4 "311-1.00KCRCT-ND" V 4150 3050 50  0001 C CNN "DIGIKEY"
@@
 P 4150 3350
 AR Path="/5EEDB4C5/5F865B33" Ref="R?"  Part="1"
-AR Path="/5EFA5E54/5F865B33" Ref="R23"  Part="1"
-F 0 "R23" V 3943 3350 50  0000 C CNN
+AR Path="/5EFA5E54/5F865B33" Ref="R10"  Part="1"
+F 0 "R10" V 3943 3350 50  0000 C CNN
 F 1 "1k" V 4034 3350 50  0000 C CNN
-F 2 "Resistor_SMD:R_0603_1608Metric_Pad1.05x0.95mm_HandSolder" V 4080 3350 50  0001 C CNN
+F 2 "Resistor_SMD:R_0603_1608Metric_Pad0.98x0.95mm_HandSolder" V 4080 3350 50  0001 C CNN
 F 3 "~" H 4150 3350 50  0001 C CNN
 F 4 "311-1.00KCRCT-ND" V 4150 3350 50  0001 C CNN "DIGIKEY"
@@
 P 4600 3750
 AR Path="/5EEDB4C5/5F86631A" Ref="R?"  Part="1"
-AR Path="/5EFA5E54/5F86631A" Ref="R25"  Part="1"
-F 0 "R25" H 4530 3704 50  0000 R CNN
+AR Path="/5EFA5E54/5F86631A" Ref="R12"  Part="1"
+F 0 "R12" H 4530 3704 50  0000 R CNN
 F 1 "100k" H 4530 3795 50  0000 R CNN
-F 2 "Resistor_SMD:R_0603_1608Metric_Pad1.05x0.95mm_HandSolder" V 4530 3750 50  0001 C CNN
+F 2 "Resistor_SMD:R_0603_1608Metric_Pad0.98x0.95mm_HandSolder" V 4530 3750 50  0001 C CNN
 F 3 "~" H 4600 3750 50  0001 C CNN
 F 4 "311-100KCRCT-ND" V 4600 3750 50  0001 C CNN "DIGIKEY"
@@
 P 4600 2750
 AR Path="/5EEDB4C5/5F868FC3" Ref="R?"  Part="1"
-AR Path="/5EFA5E54/5F868FC3" Ref="R24"  Part="1"
-F 0 "R24" H 4530 2704 50  0000 R CNN
+AR Path="/5EFA5E54/5F868FC3" Ref="R11"  Part="1"
+F 0 "R11" H 4530 2704 50  0000 R CNN
 F 1 "100k" H 4530 2795 50  0000 R CNN
-F 2 "Resistor_SMD:R_0603_1608Metric_Pad1.05x0.95mm_HandSolder" V 4530 2750 50  0001 C CNN
+F 2 "Resistor_SMD:R_0603_1608Metric_Pad0.98x0.95mm_HandSolder" V 4530 2750 50  0001 C CNN
 F 3 "~" H 4600 2750 50  0001 C CNN
 F 4 "311-100KCRCT-ND" V 4600 2750 50  0001 C CNN "DIGIKEY"
@@
 P 6950 3750
 AR Path="/5EEDB4C5/5F869342" Ref="R?"  Part="1"
-AR Path="/5EFA5E54/5F869342" Ref="R26"  Part="1"
-F 0 "R26" V 6743 3750 50  0000 C CNN
+AR Path="/5EFA5E54/5F869342" Ref="R13"  Part="1"
+F 0 "R13" V 6743 3750 50  0000 C CNN
 F 1 "1k" V 6834 3750 50  0000 C CNN
-F 2 "Resistor_SMD:R_0603_1608Metric_Pad1.05x0.95mm_HandSolder" V 6880 3750 50  0001 C CNN
+F 2 "Resistor_SMD:R_0603_1608Metric_Pad0.98x0.95mm_HandSolder" V 6880 3750 50  0001 C CNN
 F 3 "~" H 6950 3750 50  0001 C CNN
 F 4 "311-1.00KCRCT-ND" V 6950 3750 50  0001 C CNN "DIGIKEY"
@@
 AR Path="/5F8719C9" Ref="U?"  Part="1"
 AR Path="/5EEDB4C5/5F8719C9" Ref="U?"  Part="1"
-AR Path="/5EFA5E54/5F8719C9" Ref="U6"  Part="1"
-F 0 "U6" H 5500 3817 50  0000 C CNN
+AR Path="/5EFA5E54/5F8719C9" Ref="U3"  Part="1"
+F 0 "U3" H 5500 3817 50  0000 C CNN
 F 1 "VNLD5090" H 5500 3726 50  0000 C CNN
-F 2 "Package_SO:SO-8_3.9x4.9mm_P1.27mm" H 5600 2550 50  0001 C CNN
+F 2 "Package_SO:SOIC-8_3.9x4.9mm_P1.27mm" H 5600 2550 50  0001 C CNN
 F 3 "https://www.st.com/resource/en/datasheet/vnld5090-e.pdf" H 5400 3250 50  0001 C CNN
 F 4 "511-VNLD5090-E" H 5400 3250 50  0001 C CNN "MOUSER"
@@
 	1    0    0    -1
 $EndComp
+$Comp
+L Connector:TestPoint_Small TP1
+U 1 1 60D91417
+P 7750 3550
+F 0 "TP1" H 7798 3596 50  0000 L CNN
+F 1 "TP_TACH" H 7798 3505 50  0000 L CNN
+F 2 "TestPoint:TestPoint_Pad_D1.0mm" H 7950 3550 50  0001 C CNN
+F 3 "~" H 7950 3550 50  0001 C CNN
+	1    7750 3550
+	1    0    0    -1
+$EndComp
+Wire Wire Line
+	7750 3550 7750 3350
+Wire Wire Line
+	7700 3350 7750 3350
+Connection ~ 7750 3350
+Wire Wire Line
+	7750 3350 7950 3350
 $EndSCHEMATC

Commit message: Update Schematic with a bunch of extra stuff
Parts:
- removed R10, R13, R9: 1k, Resistor_SMD:R_0603_1608Metric_Pad0.98x0.95mm_HandSolder, symbol Device:R
- removed R11, R12: 100k, Resistor_SMD:R_0603_1608Metric_Pad0.98x0.95mm_HandSolder, symbol Device:R
- removed U3: VNLD5090, Package_SO:SOIC-8_3.9x4.9mm_P1.27mm, symbol speeduino_ic_automotive:VNLD5090
- added Q? (x3): 2N7002, Package_TO_SOT_SMD:SOT-23, symbol Transistor_FET:2N7002
- added R?: 10k, Resistor_SMD:R_0603_1608Metric_Pad0.98x0.95mm_HandSolder, symbol Device:R
Connections:
- net 12v-SW: now also R?.2
- net FAN-OUT: now also Q?.3 (D)
- net GND: now also Q?.2 (S), Q?.2 (S), Q?.2 (S)
- net MCU-FAN: now also Q?.1 (G)
- net MCU-TACH: now also Q?.1 (G)
- net at JP1.1: now also Q?.3 (D), R?.1
- new net FUELPUMP-OUT: Q?.3 (D)
- new net MCU-FP: Q?.1 (G)
Other:
- moved on the sheet: JP1, TP1

Commit message: Start rerouting again
Parts:
- gave numbers to parts that had none: 4
Changed lines of the file:
@@
 	3700 2850 3900 2850
 $Comp
-L Transistor_FET:2N7002 Q?
+L Transistor_FET:2N7002 Q2
 U 1 1 61AFCA1D
 P 2450 4450
-F 0 "Q?" H 2654 4496 50  0000 L CNN
+F 0 "Q2" H 2654 4496 50  0000 L CNN
 F 1 "2N7002" H 2654 4405 50  0000 L CNN
 F 2 "Package_TO_SOT_SMD:SOT-23" H 2650 4375 50  0001 L CIN
@@
 P 2200 2850
 AR Path="/5EEDB4C5/61B00181" Ref="R?"  Part="1"
-AR Path="/5EFA5E54/61B00181" Ref="R?"  Part="1"
-F 0 "R?" V 1993 2850 50  0000 C CNN
+AR Path="/5EFA5E54/61B00181" Ref="R1"  Part="1"
+F 0 "R1" V 1993 2850 50  0000 C CNN
 F 1 "10k" V 2084 2850 50  0000 C CNN
 F 2 "Resistor_SMD:R_0603_1608Metric_Pad0.98x0.95mm_HandSolder" V 2130 2850 50  0001 C CNN
@@
 	2550 4200 3200 4200
 $Comp
-L power:GND #PWR?
+L power:GND #PWR01
 U 1 1 61B06797
 P 2550 4650
-F 0 "#PWR?" H 2550 4400 50  0001 C CNN
+F 0 "#PWR01" H 2550 4400 50  0001 C CNN
 F 1 "GND" H 2555 4477 50  0000 C CNN
 F 2 "" H 2550 4650 50  0001 C CNN
@@
 $EndComp
 $Comp
-L Transistor_FET:2N7002 Q?
+L Transistor_FET:2N7002 Q3
 U 1 1 61B06C55
 P 2600 3150
-F 0 "Q?" H 2804 3196 50  0000 L CNN
+F 0 "Q3" H 2804 3196 50  0000 L CNN
 F 1 "2N7002" H 2804 3105 50  0000 L CNN
 F 2 "Package_TO_SOT_SMD:SOT-23" H 2800 3075 50  0001 L CIN
@@
 	2700 2850 2700 2950
 $Comp
-L power:GND #PWR?
+L power:GND #PWR02
 U 1 1 61B0F0BA
 P 2700 3350
-F 0 "#PWR?" H 2700 3100 50  0001 C CNN
+F 0 "#PWR02" H 2700 3100 50  0001 C CNN
 F 1 "GND" H 2705 3177 50  0000 C CNN
 F 2 "" H 2700 3350 50  0001 C CNN
@@
 12v-SW
 $Comp
-L Transistor_FET:2N7002 Q?
+L Transistor_FET:2N7002 Q4
 U 1 1 61B4B0F4
 P 4850 4700
-F 0 "Q?" H 5054 4746 50  0000 L CNN
+F 0 "Q4" H 5054 4746 50  0000 L CNN
 F 1 "2N7002" H 5054 4655 50  0000 L CNN
 F 2 "Package_TO_SOT_SMD:SOT-23" H 5050 4625 50  0001 L CIN
@@
 	4950 4450 5600 4450
 $Comp
-L power:GND #PWR?
+L power:GND #PWR05
 U 1 1 61B4B0FF
 P 4950 4900
-F 0 "#PWR?" H 4950 4650 50  0001 C CNN
+F 0 "#PWR05" H 4950 4650 50  0001 C CNN
 F 1 "GND" H 4955 4727 50  0000 C CNN
 F 2 "" H 4950 4900 50  0001 C CNN

Commit message: Finish reroute again
Parts:
- removed JP1: Jumper, Jumper:SolderJumper-2_P1.3mm_Open_RoundedPad1.0x1.5mm, symbol Device:Jumper
- removed TP1: TP_TACH, TestPoint:TestPoint_Pad_D1.0mm, symbol Connector:TestPoint_Small
Connections:
- net TACH-OUT: now also Q3.3 (D), R1.1
Changed lines of the file:
@@
 Comment4 ""
 $EndDescr
-Text HLabel 3900 2850 2    50   Output ~ 0
+Text HLabel 3300 2850 2    50   Output ~ 0
 TACH-OUT
-$Comp
-L Device:Jumper JP1
-U 1 1 5EFA7131
-P 3350 2850
-F 0 "JP1" H 3350 3114 50  0000 C CNN
-F 1 "Jumper" H 3350 3023 50  0000 C CNN
-F 2 "Jumper:SolderJumper-2_P1.3mm_Open_RoundedPad1.0x1.5mm" H 3350 2850 50  0001 C CNN
-F 3 "~" H 3350 2850 50  0001 C CNN
-	1    3350 2850
-	1    0    0    -1
-$EndComp
-$Comp
-L Connector:TestPoint_Small TP1
-U 1 1 60D91417
-P 3700 3050
-F 0 "TP1" H 3748 3096 50  0000 L CNN
-F 1 "TP_TACH" H 3748 3005 50  0000 L CNN
-F 2 "TestPoint:TestPoint_Pad_D1.0mm" H 3900 3050 50  0001 C CNN
-F 3 "~" H 3900 3050 50  0001 C CNN
-	1    3700 3050
-	1    0    0    -1
-$EndComp
-Wire Wire Line
-	3700 3050 3700 2850
-Wire Wire Line
-	3650 2850 3700 2850
-Connection ~ 3700 2850
-Wire Wire Line
-	3700 2850 3900 2850
 $Comp
 L Transistor_FET:2N7002 Q2
@@
 	1    0    0    -1
 $EndComp
-Wire Wire Line
-	2700 2850 3050 2850
 Connection ~ 2700 2850
 Text HLabel 2400 3150 0    50   Input ~ 0
@@
 	1    0    0    -1
 $EndComp
+Wire Wire Line
+	2700 2850 3300 2850
 $EndSCHEMATC
