File: mcu.sch (KiCad schematic (older format))
At the start: 101 parts, among them J3 SWD, J4 USB_B, J5 USB_EXT, J6 Micro_SD_Card_Det, J7 HC-05, Q1 AO3401A, U10 USBLC6-2SC6, U11 MCP2551-I-SN, U12 STM32F429ZGTx, U16 ATECC608A-SSHDA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

Commit message: Swapped the LEDs, added resistor values
Parts:
- D23: value PWR_5V_GREEN -> PWR_3V_GREEN
- D24: value PWR_3V_RED -> PWR_5V_RED
- R74: value null -> 220
- R75: value null -> 330
Changed lines of the file:
@@
 U 1 1 608CDC8A
 P 5150 7250
+AR Path="/608CDC8A" Ref="J5"  Part="1"
+AR Path="/608F155A/608CDC8A" Ref="J5"  Part="1"
 F 0 "J5" H 5258 7631 50  0000 C CNN
 F 1 "USB_EXT" H 5258 7540 50  0000 C CNN
@@
 P 14200 8750
 F 0 "D23" H 14200 8543 50  0000 C CNN
-F 1 "PWR_5V_GREEN" H 14200 8634 50  0000 C CNN
+F 1 "PWR_3V_GREEN" H 14200 8634 50  0000 C CNN
 F 2 "LED_SMD:LED_0603_1608Metric_Pad1.05x0.95mm_HandSolder" V 14200 8750 50  0001 C CNN
 F 3 "https://datasheet.lcsc.com/lcsc/1912111437_TOGIALED-TJ-S1608CY6T5ALC2G-A5_C440518.pdf" V 14200 8750 50  0001 C CNN
@@
 P 13700 8750
 F 0 "R74" V 13504 8750 50  0000 C CNN
-F 1 "null" V 13595 8750 50  0000 C CNN
+F 1 "220" V 13595 8750 50  0000 C CNN
 F 2 "Resistor_SMD:R_0603_1608Metric_Pad0.98x0.95mm_HandSolder" H 13700 8750 50  0001 C CNN
 F 3 "~" H 13700 8750 50  0001 C CNN
@@
 P 13700 9150
 F 0 "R75" V 13504 9150 50  0000 C CNN
-F 1 "null" V 13595 9150 50  0000 C CNN
+F 1 "330" V 13595 9150 50  0000 C CNN
 F 2 "Resistor_SMD:R_0603_1608Metric_Pad0.98x0.95mm_HandSolder" H 13700 9150 50  0001 C CNN
 F 3 "~" H 13700 9150 50  0001 C CNN
@@
 P 14200 9150
 F 0 "D24" H 14200 8943 50  0000 C CNN
-F 1 "PWR_3V_RED" H 14200 9034 50  0000 C CNN
+F 1 "PWR_5V_RED" H 14200 9034 50  0000 C CNN
 F 2 "LED_SMD:LED_0603_1608Metric_Pad1.05x0.95mm_HandSolder" V 14200 9150 50  0001 C CNN
 F 3 "https://datasheet.lcsc.com/lcsc/1811141223_TOGIALED-TJ-S1608SW6TGLC2R-A5_C192315.pdf" V 14200 9150 50  0001 C CNN
