File: Sensors.sch (KiCad schematic (older format))
At the start: 35 parts

Commit message: Starting on layout
Parts:
- C10, C12, C16, C4, C5, C8, C9: renamed from C?; footprint (none) -> Capacitor_SMD:C_0805_2012Metric_Pad1.15x1.40mm_HandSolder
- R43, R44, R45, R46, R47, R48, R49, R50, R51, R52, R53, R54, R55, R56, R57, R58: renamed from R?; footprint (none) -> Resistor_SMD:R_0603_1608Metric_Pad1.05x0.95mm_HandSolder
- U10: renamed from U?; footprint (none) -> speeduino_misc:MPX4250
- gave numbers to parts that had none: 11

Commit message: restart a third time
Parts:
- added TP16: TP_CRANK, TestPoint:TestPoint_Pad_D1.0mm, symbol Connector:TestPoint_Small
- added TP17: TP_CAM, TestPoint:TestPoint_Pad_D1.0mm, symbol Connector:TestPoint_Small
- added TP2: TP_IAT, TestPoint:TestPoint_Pad_D1.0mm, symbol Connector:TestPoint_Small
- added TP3: TP_VBAT, TestPoint:TestPoint_Pad_D1.0mm, symbol Connector:TestPoint_Small
- added TP4: TP_CLT, TestPoint:TestPoint_Pad_D1.0mm, symbol Connector:TestPoint_Small
- added TP5: TP_MAP, TestPoint:TestPoint_Pad_D1.0mm, symbol Connector:TestPoint_Small
- added TP6: TP_TPS, TestPoint:TestPoint_Pad_D1.0mm, symbol Connector:TestPoint_Small
- added TP7: TP_FLEX, TestPoint:TestPoint_Pad_D1.0mm, symbol Connector:TestPoint_Small
- added TP8: TP_O2, TestPoint:TestPoint_Pad_D1.0mm, symbol Connector:TestPoint_Small
- C1: renamed from C2; footprint Capacitor_SMD:C_0805_2012Metric_Pad1.15x1.40mm_HandSolder -> Capacitor_SMD:C_0805_2012Metric_Pad1.18x1.45mm_HandSolder
- C10: renamed from C11; footprint Capacitor_SMD:C_0805_2012Metric_Pad1.15x1.40mm_HandSolder -> Capacitor_SMD:C_0805_2012Metric_Pad1.18x1.45mm_HandSolder
- C11: renamed from C12; footprint Capacitor_SMD:C_0805_2012Metric_Pad1.15x1.40mm_HandSolder -> Capacitor_SMD:C_0805_2012Metric_Pad1.18x1.45mm_HandSolder
- C12: renamed from C13; footprint Capacitor_SMD:C_0805_2012Metric_Pad1.15x1.40mm_HandSolder -> Capacitor_SMD:C_0805_2012Metric_Pad1.18x1.45mm_HandSolder
- C13: renamed from C14; footprint Capacitor_SMD:C_0805_2012Metric_Pad1.15x1.40mm_HandSolder -> Capacitor_SMD:C_0805_2012Metric_Pad1.18x1.45mm_HandSolder
- C14: renamed from C15; footprint Capacitor_SMD:C_0805_2012Metric_Pad1.15x1.40mm_HandSolder -> Capacitor_SMD:C_0805_2012Metric_Pad1.18x1.45mm_HandSolder
- C15: renamed from C16; footprint Capacitor_SMD:C_0805_2012Metric_Pad1.15x1.40mm_HandSolder -> Capacitor_SMD:C_0805_2012Metric_Pad1.18x1.45mm_HandSolder
- C2: renamed from C3; footprint Capacitor_SMD:C_0805_2012Metric_Pad1.15x1.40mm_HandSolder -> Capacitor_SMD:C_0805_2012Metric_Pad1.18x1.45mm_HandSolder
- C3: renamed from C4; footprint Capacitor_SMD:C_0805_2012Metric_Pad1.15x1.40mm_HandSolder -> Capacitor_SMD:C_0805_2012Metric_Pad1.18x1.45mm_HandSolder
- C4: renamed from C5; footprint Capacitor_SMD:C_0805_2012Metric_Pad1.15x1.40mm_HandSolder -> Capacitor_SMD:C_0805_2012Metric_Pad1.18x1.45mm_HandSolder
- C5: renamed from C6; footprint Capacitor_SMD:C_0805_2012Metric_Pad1.15x1.40mm_HandSolder -> Capacitor_SMD:C_0805_2012Metric_Pad1.18x1.45mm_HandSolder
- C6: renamed from C7; footprint Capacitor_SMD:C_0805_2012Metric_Pad1.15x1.40mm_HandSolder -> Capacitor_SMD:C_0805_2012Metric_Pad1.18x1.45mm_HandSolder
- C7: renamed from C8; footprint Capacitor_SMD:C_0805_2012Metric_Pad1.15x1.40mm_HandSolder -> Capacitor_SMD:C_0805_2012Metric_Pad1.18x1.45mm_HandSolder
- C8: renamed from C9; footprint Capacitor_SMD:C_0805_2012Metric_Pad1.15x1.40mm_HandSolder -> Capacitor_SMD:C_0805_2012Metric_Pad1.18x1.45mm_HandSolder
- C9: renamed from C10; footprint Capacitor_SMD:C_0805_2012Metric_Pad1.15x1.40mm_HandSolder -> Capacitor_SMD:C_0805_2012Metric_Pad1.18x1.45mm_HandSolder
- R30: renamed from R43; footprint Resistor_SMD:R_0603_1608Metric_Pad1.05x0.95mm_HandSolder -> Resistor_SMD:R_0805_2012Metric_Pad1.20x1.40mm_HandSolder
- R31: renamed from R44; footprint Resistor_SMD:R_0603_1608Metric_Pad1.05x0.95mm_HandSolder -> Resistor_SMD:R_0805_2012Metric_Pad1.20x1.40mm_HandSolder
- R32: renamed from R45; footprint Resistor_SMD:R_0603_1608Metric_Pad1.05x0.95mm_HandSolder -> Resistor_SMD:R_0805_2012Metric_Pad1.20x1.40mm_HandSolder
- R33: renamed from R46; footprint Resistor_SMD:R_0603_1608Metric_Pad1.05x0.95mm_HandSolder -> Resistor_SMD:R_0805_2012Metric_Pad1.20x1.40mm_HandSolder
- R34: renamed from R47; footprint Resistor_SMD:R_0603_1608Metric_Pad1.05x0.95mm_HandSolder -> Resistor_SMD:R_0805_2012Metric_Pad1.20x1.40mm_HandSolder
- R35: renamed from R48; footprint Resistor_SMD:R_0603_1608Metric_Pad1.05x0.95mm_HandSolder -> Resistor_SMD:R_0805_2012Metric_Pad1.20x1.40mm_HandSolder
- R36: renamed from R49; footprint Resistor_SMD:R_0603_1608Metric_Pad1.05x0.95mm_HandSolder -> Resistor_SMD:R_0805_2012Metric_Pad1.20x1.40mm_HandSolder
- R37: renamed from R50; footprint Resistor_SMD:R_0603_1608Metric_Pad1.05x0.95mm_HandSolder -> Resistor_SMD:R_0805_2012Metric_Pad1.20x1.40mm_HandSolder
- R38: renamed from R51; footprint Resistor_SMD:R_0603_1608Metric_Pad1.05x0.95mm_HandSolder -> Resistor_SMD:R_0805_2012Metric_Pad1.20x1.40mm_HandSolder
- R39: renamed from R52; footprint Resistor_SMD:R_0603_1608Metric_Pad1.05x0.95mm_HandSolder -> Resistor_SMD:R_0805_2012Metric_Pad1.20x1.40mm_HandSolder
- R40: renamed from R53; footprint Resistor_SMD:R_0603_1608Metric_Pad1.05x0.95mm_HandSolder -> Resistor_SMD:R_0805_2012Metric_Pad1.20x1.40mm_HandSolder
- R41: renamed from R54; footprint Resistor_SMD:R_0603_1608Metric_Pad1.05x0.95mm_HandSolder -> Resistor_SMD:R_0805_2012Metric_Pad1.20x1.40mm_HandSolder
- R42: renamed from R55; footprint Resistor_SMD:R_0603_1608Metric_Pad1.05x0.95mm_HandSolder -> Resistor_SMD:R_0805_2012Metric_Pad1.20x1.40mm_HandSolder
- R43: renamed from R56; footprint Resistor_SMD:R_0603_1608Metric_Pad1.05x0.95mm_HandSolder -> Resistor_SMD:R_0805_2012Metric_Pad1.20x1.40mm_HandSolder
- R44: renamed from R57; footprint Resistor_SMD:R_0603_1608Metric_Pad1.05x0.95mm_HandSolder -> Resistor_SMD:R_0805_2012Metric_Pad1.20x1.40mm_HandSolder
- R45: renamed from R58; footprint Resistor_SMD:R_0603_1608Metric_Pad1.05x0.95mm_HandSolder -> Resistor_SMD:R_0805_2012Metric_Pad1.20x1.40mm_HandSolder
- renumbered D15 to D7, D16 to D8, U9 to U6, U10 to U7
Connections:
- net ADC-CLAMP-1: now also TP2.1
- net ADC-CLAMP-10: now also C12.2, R42.1, TP16.1; no longer R45.2
- net ADC-CLAMP-2: now also TP4.1
- net ADC-CLAMP-3: now also TP6.1
- net ADC-CLAMP-4: now also TP8.1
- net ADC-CLAMP-5: now also TP3.1
- net ADC-CLAMP-6: now also TP5.1
- net ADC-CLAMP-8: now also R45.2, TP7.1; no longer C12.2, R42.1
- net ADC-CLAMP-9: now also TP17.1
- net CPU-D12 renamed MCU-CLUTCH
Other:
- moved on the sheet: C13, R40, R43

Commit message: Update Schematic with a bunch of extra stuff
Parts:
- removed C5: 0.1uf, Capacitor_SMD:C_0805_2012Metric_Pad1.18x1.45mm_HandSolder, symbol Device:C
- removed C7: 1uf, Capacitor_SMD:C_0805_2012Metric_Pad1.18x1.45mm_HandSolder, symbol Device:C
- removed C9: 470pf, Capacitor_SMD:C_0805_2012Metric_Pad1.18x1.45mm_HandSolder, symbol Device:C
- removed R38: 470, Resistor_SMD:R_0805_2012Metric_Pad1.20x1.40mm_HandSolder, symbol Device:R
- removed TP5: TP_MAP, TestPoint:TestPoint_Pad_D1.0mm, symbol Connector:TestPoint_Small
- removed U7: MPX4250, speeduino_misc:MPX4250, symbol speeduino_misc:MPX4250
- added C?: 470pf, Capacitor_SMD:C_0805_2012Metric_Pad1.18x1.45mm_HandSolder, symbol Device:C
- added C? (x5): 0.1uf, Capacitor_SMD:C_0805_2012Metric_Pad1.18x1.45mm_HandSolder, symbol Device:C
- added C?: 1uf, Capacitor_SMD:C_0805_2012Metric_Pad1.18x1.45mm_HandSolder, symbol Device:C
- added C? (x4): 0.22uf, Capacitor_SMD:C_0805_2012Metric_Pad1.18x1.45mm_HandSolder, symbol Device:C
- added D?: MM3Zxx, Diode_SMD:D_SOD-323_HandSoldering, symbol Diode:MM3Zxx
- added R?: 470, Resistor_SMD:R_0805_2012Metric_Pad1.20x1.40mm_HandSolder, symbol Device:R
- added R?: 1k, Resistor_SMD:R_0805_2012Metric_Pad1.20x1.40mm_HandSolder, symbol Device:R
- added R? (x8): null, Resistor_SMD:R_0805_2012Metric_Pad1.20x1.40mm_HandSolder, symbol Device:R
- added TP?: TP_MAP, TestPoint:TestPoint_Pad_D1.0mm, symbol Connector:TestPoint_Small
- added TP?: TP_A1, TestPoint:TestPoint_Pad_D1.0mm, symbol Connector:TestPoint_Small
- added TP?: TP_A2, TestPoint:TestPoint_Pad_D1.0mm, symbol Connector:TestPoint_Small
- added TP?: TP_A3, TestPoint:TestPoint_Pad_D1.0mm, symbol Connector:TestPoint_Small
- added TP?: TP_A4, TestPoint:TestPoint_Pad_D1.0mm, symbol Connector:TestPoint_Small
- added U?: MPXH6250A, Sensor_Pressure:Freescale_98ARH99066A, symbol cone-kicad-parts:MPXH6250A
Connections:
- net 5v is gone; now on net VPROT: D8.2 (A), R45.1, U6.16 (V+)
- net ADC-CLAMP-10: now also U6.11 (I10); no longer U6.13 (I12)
- net ADC-CLAMP-6: now also R?.1, TP?.1, U?.4 (VOUT)
- net ADC-CLAMP-8: now also U6.9 (I8); no longer U6.15 (I14)
- net ADC-CLAMP-9: now also U6.10 (I9); no longer U6.14 (I13)
- net GND: now also C?.1, C?.2, C?.2, C?.2, C?.2, C?.2, C?.2, C?.2, C?.2, C?.2, C?.2, D?.2 (A)
- net VPROT: now also C?.1, C?.1, R?.1, R?.1, R?.1, R?.1, U?.2 (VS)
- net ADC-CLAMP-11: now reaches U6.12 (I11)
- net ADC-CLAMP-7: now reaches U6.7 (I7)
- new net: C?.2, R?.2, U?.3 (GND)
- new net: C?.1, R?.1 (x4)
- new net AC-IN: R?.2
- new net ADC-CLAMP-12: U6.13 (I12)
- new net ADC-CLAMP-13: U6.14 (I13)
- new net ADC-CLAMP-14: U6.15 (I14)
- new net MCU-AC: D?.1 (K), R?.1
- new net MCU-ANALOG-1: C?.1, R?.2, R?.2
- new net MCU-ANALOG-2: C?.1, R?.2, R?.2
- new net MCU-ANALOG-3: C?.1, R?.2, R?.2
- new net MCU-ANALOG-4: C?.1, R?.2, R?.2
Other:
- note added: "AC Input\n"
- note added: "Spare Analog 1"
- note added: "Spare Analog 2"
- note added: "Spare Analog 3"
- note added: "Spare Analog 4"
- moved on the sheet: D8, R30, U6

Commit message: Start rerouting again
Parts:
- gave numbers to parts that had none: 28
Connections:
- net ADC-CLAMP-1: now also C4.1, R35.1, TP3.1; no longer C3.1, R34.1, TP2.1
- net ADC-CLAMP-10: no longer C12.2, R42.1, TP16.1
- net ADC-CLAMP-11: now also C55.1, R80.1
- net ADC-CLAMP-12: now also C7.1, R3.1
- net ADC-CLAMP-13: now also C48.1, R10.1
- net ADC-CLAMP-14: now also C12.2, R42.1, TP16.1
- net ADC-CLAMP-2: now also R45.2, TP7.1; no longer C8.1, R37.1, TP4.1
- net ADC-CLAMP-3: now also C3.1, R34.1, TP2.1; no longer C11.1, R41.1, TP6.1
- net ADC-CLAMP-4: now also C8.1, R37.1, TP4.1; no longer C15.1, R44.1, TP8.1
- net ADC-CLAMP-5: now also C11.1, R41.1, TP6.1; no longer C4.1, R35.1, TP3.1
- net ADC-CLAMP-6: now also C15.1, R44.1, TP8.1
- net ADC-CLAMP-7: now also C13.1, R43.1, TP17.1
- net ADC-CLAMP-8: no longer R45.2, TP7.1
- net ADC-CLAMP-9: now also C50.1, R13.1; no longer C13.1, R43.1, TP17.1
