File: daveecu2.kicad_pcb (KiCad board)
At the start: 4 copper layers, 160 x 117.5 mm, 200 parts, among them J1 CONN_BLACK, J2 CONN_GREY, J3 SWD, J4 USB_B, J5 USB_EXT, Q1 AO3401A, Q2 Q_PNP_BEC, U1 VNLD5090, U10 USBLC6-2SC6, U11 MCP2551-I-SN, U12 STM32F429ZGTx, U13 VNLD5090, U14 VNLD5090, U15 MC33814, U2 VNLD5090, U3 VNLD5090, U4 TC4424A, U5 TC4424A, U6 SP720, U7 MPX4250, U8 TPS5430DDA, U9 TPS5430DDA, Y1 25mhz

Commit message: rename project
Parts:
- removed REF**: PinHeader_1x09_P2.54mm_Vertical_SMD_Pin1Left, Connector_PinHeader_2.54mm:PinHeader_1x09_P2.54mm_Vertical_SMD_Pin1Left
- removed REF** (x3): PinHeader_1x02_P2.54mm_Vertical, Connector_PinHeader_2.54mm:PinHeader_1x02_P2.54mm_Vertical
- removed REF**: microSD_HC_Hirose_DM3D-SF, Connector_Card:microSD_HC_Hirose_DM3D-SF
- removed REF**: BatteryHolder_ComfortableElectronic_CH273-2450_1x2450, Battery:BatteryHolder_ComfortableElectronic_CH273-2450_1x2450
Routing:
- net (no net): track 107.8 -> 0.00 mm
- net GND: track 328.4 -> 323.3 mm
- net +3V3: track 111.8 -> 106.9 mm

Commit message: Start rerouting again
Parts:
- removed U15: MC33814, Package_QFP:LQFP-48-1EP_7x7mm_P0.5mm_EP3.6x3.6mm_ThermalVias
- added C42: 12p, Capacitor_SMD:C_0402_1005Metric_Pad0.74x0.62mm_HandSolder, F.Cu at (195.8, 61.4)
- added C52: 12p, Capacitor_SMD:C_0402_1005Metric_Pad0.74x0.62mm_HandSolder, F.Cu at (202.2, 61.4)
- added C53: 10u, Capacitor_SMD:C_0402_1005Metric_Pad0.74x0.62mm_HandSolder, F.Cu at (205.4, 61.4)
- added C54: 100n, Capacitor_SMD:C_0402_1005Metric_Pad0.74x0.62mm_HandSolder, F.Cu at (199.0, 61.4)
- added C55: 0.22uf, Capacitor_SMD:C_0805_2012Metric_Pad1.18x1.45mm_HandSolder, F.Cu at (250.7, 48.7)
- added C56: 47u, Capacitor_SMD:CP_Elec_5x5.8, F.Cu at (212.4, 58.3)
- added C57: 10u, Capacitor_Tantalum_SMD:CP_EIA-7343-20_Kemet-V_Pad2.25x2.55mm_HandSolder, F.Cu at (215.4, 40.5)
- added C58: 0.1u, Capacitor_SMD:C_1206_3216Metric_Pad1.33x1.80mm_HandSolder, F.Cu at (219.3, 45.7)
- added C59: 0.1u, Capacitor_SMD:C_1206_3216Metric_Pad1.33x1.80mm_HandSolder, F.Cu at (213.3, 48.5)
- added C60: 0.1u, Capacitor_SMD:C_1206_3216Metric_Pad1.33x1.80mm_HandSolder, F.Cu at (213.3, 45.1)
- added D22: ESD9B3.3ST5G, Diode_SMD:D_SOD-923, F.Cu at (225.2, 56.7)
- added D23: PWR_5V_GREEN, LED_SMD:LED_0603_1608Metric_Pad1.05x0.95mm_HandSolder, F.Cu at (212.5, 52.0)
- added D24: PWR_3V_RED, LED_SMD:LED_0603_1608Metric_Pad1.05x0.95mm_HandSolder, F.Cu at (216.9, 52.0)
- added D25: ESD9B3.3ST5G, Diode_SMD:D_SOD-923, F.Cu at (231.8, 49.2)
- added D26: ESD9B3.3ST5G, Diode_SMD:D_SOD-923, F.Cu at (222.6, 58.7)
- added D27: ESD9B3.3ST5G, Diode_SMD:D_SOD-923, F.Cu at (227.0, 53.4)
- added D28: ESD9B3.3ST5G, Diode_SMD:D_SOD-923, F.Cu at (222.6, 56.7)
- added D29: ESD9B3.3ST5G, Diode_SMD:D_SOD-923, F.Cu at (229.1, 50.6)
- added D30: ESD9B3.3ST5G, Diode_SMD:D_SOD-923, F.Cu at (228.7, 48.6)
- added D31: 1n41001, Diode_SMD:D_SOD-123, F.Cu at (202.2, 67.3)
- added D32: 1n41001, Diode_SMD:D_SOD-123, F.Cu at (208.0, 67.3)
- added D33: 1n41001, Diode_SMD:D_SOD-123, F.Cu at (202.2, 74.0)
- added D34: MM3Zxx, Diode_SMD:D_SOD-323_HandSoldering, F.Cu at (224.8, 48.5)
- added D35: MM3Zxx, Diode_SMD:D_SOD-323_HandSoldering, F.Cu at (224.8, 45.5)
- added J6: Micro_SD_Card_Det, Connector_Card:microSD_HC_Molex_104031-0811, F.Cu at (149.6, 28.9)
- added J7: HC-05, Connector_PinHeader_2.54mm:PinHeader_1x06_P2.54mm_Vertical, F.Cu at (48.0, 40.3)
- added Q3: 2N7002, Package_TO_SOT_SMD:SOT-23, F.Cu at (245.1, 61.1)
- added Q4: 2N7002, Package_TO_SOT_SMD:SOT-23, F.Cu at (249.5, 61.1)
- added R48: 47, Resistor_SMD:R_0402_1005Metric_Pad0.72x0.64mm_HandSolder, F.Cu at (192.5, 61.4)
- added R49: null, Resistor_SMD:R_0603_1608Metric_Pad0.98x0.95mm_HandSolder, F.Cu at (223.4, 54.5)
- added R50: 4.7k, Resistor_SMD:R_0603_1608Metric_Pad0.98x0.95mm_HandSolder, F.Cu at (231.2, 38.9)
- added R51: 4.7k, Resistor_SMD:R_0603_1608Metric_Pad0.98x0.95mm_HandSolder, F.Cu at (231.2, 41.4)
- added R73: 10k, Resistor_SMD:R_0603_1608Metric_Pad0.98x0.95mm_HandSolder, F.Cu at (221.2, 52.0)
- added R74: null, Resistor_SMD:R_0603_1608Metric_Pad0.98x0.95mm_HandSolder, F.Cu at (229.5, 46.4)
- added R75: null, Resistor_SMD:R_0603_1608Metric_Pad0.98x0.95mm_HandSolder, F.Cu at (225.6, 51.2)
- added R76: 10k, Resistor_SMD:R_0603_1608Metric_Pad0.98x0.95mm_HandSolder, F.Cu at (219.1, 57.1)
- added R77: 10k, Resistor_SMD:R_0603_1608Metric_Pad0.98x0.95mm_HandSolder, F.Cu at (219.1, 59.6)
- added R78: 10k, Resistor_SMD:R_0603_1608Metric_Pad0.98x0.95mm_HandSolder, F.Cu at (219.1, 54.6)
- added R79: 10k, Resistor_SMD:R_0603_1608Metric_Pad0.98x0.95mm_HandSolder, F.Cu at (231.2, 43.9)
- added R80: null, Resistor_SMD:R_0805_2012Metric_Pad1.20x1.40mm_HandSolder, F.Cu at (258.6, 45.1)
- added R81: 1k, Resistor_SMD:R_0603_1608Metric_Pad0.98x0.95mm_HandSolder, F.Cu at (210.2, 77.8)
- added R82: 1k, Resistor_SMD:R_0603_1608Metric_Pad0.98x0.95mm_HandSolder, F.Cu at (210.2, 75.3)
- added R83: 1k, Resistor_SMD:R_0603_1608Metric_Pad0.98x0.95mm_HandSolder, F.Cu at (211.6, 72.7)
- added R84: 1k, Resistor_SMD:R_0603_1608Metric_Pad0.98x0.95mm_HandSolder, F.Cu at (205.9, 76.9)
- added R85: 100k, Resistor_SMD:R_0603_1608Metric_Pad0.98x0.95mm_HandSolder, F.Cu at (211.6, 70.2)
- added R86: 100k, Resistor_SMD:R_0603_1608Metric_Pad0.98x0.95mm_HandSolder, F.Cu at (207.3, 70.2)
- added R87: 100k, Resistor_SMD:R_0603_1608Metric_Pad0.98x0.95mm_HandSolder, F.Cu at (201.5, 76.9)
- added R88: 100k, Resistor_SMD:R_0603_1608Metric_Pad0.98x0.95mm_HandSolder, F.Cu at (207.3, 72.7)
- added TP22: TP_VPROT, TestPoint:TestPoint_Pad_D1.0mm, F.Cu at (233.2, 46.7)
- added U16: ATECC608A-SSHDA, Package_SO:SOIC-8_3.9x4.9mm_P1.27mm, F.Cu at (224.8, 40.8)
- added Y2: Crystal, Crystal:Crystal_SMD_3215-2Pin_3.2x1.5mm, F.Cu at (218.8, 49.1)
- C45: value 22u -> 1uf; footprint Capacitor_SMD:CP_Elec_4x4.5 -> Capacitor_SMD:C_0805_2012Metric_Pad1.18x1.45mm_HandSolder
- C46: value 47u -> 0.1uf; footprint Capacitor_SMD:CP_Elec_5x5.8 -> Capacitor_SMD:C_0805_2012Metric_Pad1.18x1.45mm_HandSolder
- C47: value 0.1 -> 470pf
- C48: value 10u -> 0.22uf; footprint Capacitor_Tantalum_SMD:CP_EIA-7343-20_Kemet-V_Pad2.25x2.55mm_HandSolder -> Capacitor_SMD:C_0805_2012Metric_Pad1.18x1.45mm_HandSolder
- C49, C51: value 0.1u -> 0.1uf; footprint Capacitor_SMD:C_1206_3216Metric_Pad1.33x1.80mm_HandSolder -> Capacitor_SMD:C_0805_2012Metric_Pad1.18x1.45mm_HandSolder
- C50: value 0.1u -> 0.22uf; footprint Capacitor_SMD:C_1206_3216Metric_Pad1.33x1.80mm_HandSolder -> Capacitor_SMD:C_0805_2012Metric_Pad1.18x1.45mm_HandSolder
- C7: value 1uf -> 0.22uf
- C9: value 470pf -> 0.1uf
- D1: value LED -> 1n41001; footprint LED_SMD:LED_0603_1608Metric_Pad1.05x0.95mm_HandSolder -> Diode_SMD:D_SOD-123
- D21: value MM3Zxx -> 1n41001; footprint Diode_SMD:D_SOD-323_HandSoldering -> Diode_SMD:D_SOD-123
- J4: footprint Connector_USB:USB_B_Amphenol_MUSB-D511_Vertical_Rugged -> Connector_USB:USB_B_Lumberg_2411_02_Horizontal
- Q2: value Q_PNP_BEC -> 2N7002
- R1: value 1k -> 10k
- R10, R13: value 1k -> null; footprint Resistor_SMD:R_0603_1608Metric_Pad0.98x0.95mm_HandSolder -> Resistor_SMD:R_0805_2012Metric_Pad1.20x1.40mm_HandSolder
- R11: value 100k -> 470; footprint Resistor_SMD:R_0603_1608Metric_Pad0.98x0.95mm_HandSolder -> Resistor_SMD:R_0805_2012Metric_Pad1.20x1.40mm_HandSolder
- R12, R2: value 100k -> null; footprint Resistor_SMD:R_0603_1608Metric_Pad0.98x0.95mm_HandSolder -> Resistor_SMD:R_0805_2012Metric_Pad1.20x1.40mm_HandSolder
- R3: value 10k -> null; footprint Resistor_SMD:R_0603_1608Metric_Pad0.98x0.95mm_HandSolder -> Resistor_SMD:R_0805_2012Metric_Pad1.20x1.40mm_HandSolder
- R38: value 470 -> null
- R4: value 2.4k -> null; footprint Resistor_SMD:R_0603_1608Metric_Pad0.98x0.95mm_HandSolder -> Resistor_SMD:R_0805_2012Metric_Pad1.20x1.40mm_HandSolder
- R53: value 3.24k -> null
- R9: footprint Resistor_SMD:R_0603_1608Metric_Pad0.98x0.95mm_HandSolder -> Resistor_SMD:R_0805_2012Metric_Pad1.20x1.40mm_HandSolder
- TP12: value TP_VREG -> TP_MAP
- TP13: value TP_VPPREF -> TP_A4
- TP14: value TP_VPPSENS -> TP_A1
- TP15: value TP_VPROT -> TP_A2
- TP5: value TP_MAP -> TP_A3
- U1: value VNLD5090 -> MPXH6250A; footprint Package_SO:SOIC-8_3.9x4.9mm_P1.27mm -> Sensor_Pressure:Freescale_98ARH99066A
- U7: value MPX4250 -> VNLD5090; footprint speeduino_misc:MPX4250 -> Package_SO:SOIC-8_3.9x4.9mm_P1.27mm
- moved TP5 183.9 mm to (267.1, 48.1), turned to 0 degrees
- moved R38 179.7 mm to (263.4, 42.1), turned to 0 degrees
- moved C9 177.2 mm to (258.7, 39.1), turned to 0 degrees
- moved C5 163.4 mm to (245.9, 48.7)
- moved C7 161.1 mm to (245.6, 51.7)
- moved TP15 157.6 mm to (267.3, 45.1), turned to 0 degrees
- moved C51 156.2 mm to (253.9, 39.1), turned to 0 degrees
- moved C46 148.5 mm to (250.4, 51.7), turned to 0 degrees
- moved TP12 146.5 mm to (264.1, 51.1)
- moved TP14 144.0 mm to (264.1, 48.1)
- moved C48 142.7 mm to (263.5, 39.1), turned to 0 degrees
- moved C50 142.1 mm to (240.8, 51.6), turned to 0 degrees
- moved TP13 139.2 mm to (259.3, 54.0)
- moved D20 139.1 mm to (240.9, 48.6), turned to 0 degrees
- moved C47 138.9 mm to (258.7, 42.1)
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Connections:
- C11 pad 1: ADC-CLAMP-3 -> ADC-CLAMP-5
- C12 pad 2: ADC-CLAMP-10 -> ADC-CLAMP-8
- C13 pad 1: ADC-CLAMP-9 -> ADC-CLAMP-7
- C15 pad 1: ADC-CLAMP-4 -> ADC-CLAMP-6
- C17 pad 1: +5V -> VPROT
- C22 pad 1: +5V -> VPROT
- C23 pad 1: +3V3 -> VPROT
- C3 pad 1: ADC-CLAMP-1 -> ADC-CLAMP-3
- C4 pad 1: ADC-CLAMP-5 -> ADC-CLAMP-1
- C45 pad 1: VPPSENS -> VPROT
- C46 pad 1: VPROT -> /Sensors/MCU-ANALOG-4
- C46 pad 2: Net-(C46-Pad2) -> GND
- C47 pad 1: VPPSENS -> GND
- C47 pad 2: GND -> Net-(C47-Pad2)
- C48 pad 1: VBAT -> ADC-CLAMP-13
- C49 pad 1: VBAT -> /Sensors/MCU-ANALOG-1
- C5 pad 1: VPROT -> /Sensors/MCU-ANALOG-3
- C50 pad 1: VPROT -> ADC-CLAMP-9
- C50 pad 2: Net-(C46-Pad2) -> GND
- C51 pad 1: VPROT -> /Sensors/MCU-ANALOG-2
- C51 pad 2: Net-(C46-Pad2) -> GND
- C7 pad 1: VPROT -> ADC-CLAMP-12
- C8 pad 1: ADC-CLAMP-2 -> ADC-CLAMP-4
- C9 pad 1: GND -> VPROT
- C9 pad 2: ADC-CLAMP-6 -> GND
- D1 pad 1: GND -> 12v-SW
- D1 pad 2: Net-(D1-Pad2) -> BOOST
- D20 pad 1: VPROT -> /Sensors/MCU-AC
- D20 pad 2: Net-(C46-Pad2) -> GND
- D21 pad 1: VREG -> 12v-SW
- D21 pad 2: VBAT -> /spare-pwms/VVT-OUT
- D8 pad 2: +5V -> VPROT
- J1 pad A3: Net-(J1-PadA3) -> (no net)
- J1 pad A4: Net-(J1-PadA4) -> (no net)
- J1 pad A5: Net-(J1-PadA5) -> (no net)
- J1 pad A6: Net-(J1-PadA6) -> (no net)
- J1 pad A7: Net-(J1-PadA7) -> (no net)
- J1 pad B1: ST_SIG -> (no net)
- J2 pad A8: Net-(J2-PadA8) -> (no net)
- J2 pad C8: ADC-CLAMP-8 -> ADC-CLAMP-2
- J3 pad 7: Net-(J3-Pad7) -> (no net)
- J3 pad 8: Net-(J3-Pad8) -> (no net)
- L2 pad 2: +5V -> VPROT
- Q2 pad 1: VPPREF -> /FAN+TACH/MCU-FAN
- Q2 pad 2: VREG -> GND
- Q2 pad 3: VPPSENS -> FAN
- R1 pad 1: Net-(R1-Pad1) -> Net-(JP1-Pad1)
- R1 pad 2: /FuelPump/MCU-FP -> 12v-SW
- R10 pad 1: Net-(R10-Pad1) -> ADC-CLAMP-13
- R10 pad 2: /FAN+TACH/MCU-TACH -> /Sensors/MCU-ANALOG-4
- R11 pad 1: Net-(R11-Pad1) -> ADC-CLAMP-6
- R11 pad 2: GND -> Net-(C47-Pad2)
- R12 pad 1: GND -> VPROT
- R12 pad 2: Net-(R10-Pad1) -> /Sensors/MCU-ANALOG-1
- R13 pad 1: 12v-SW -> ADC-CLAMP-9
- R13 pad 2: Net-(JP1-Pad1) -> /Sensors/MCU-ANALOG-1
- R2 pad 1: Net-(R1-Pad1) -> VPROT
- R2 pad 2: GND -> /Sensors/MCU-ANALOG-3
- R3 pad 1: Net-(R3-Pad1) -> ADC-CLAMP-12
- R3 pad 2: GND -> /Sensors/MCU-ANALOG-3
- R34 pad 1: ADC-CLAMP-1 -> ADC-CLAMP-3
- R35 pad 1: ADC-CLAMP-5 -> ADC-CLAMP-1
- R37 pad 1: ADC-CLAMP-2 -> ADC-CLAMP-4
- R38 pad 1: Net-(R38-Pad1) -> VPROT
- R38 pad 2: ADC-CLAMP-6 -> /Sensors/MCU-ANALOG-2
- R4 pad 1: Net-(D1-Pad2) -> VPROT
- R4 pad 2: ST_SIG -> /Sensors/MCU-ANALOG-4
- R41 pad 1: ADC-CLAMP-3 -> ADC-CLAMP-5
- R42 pad 1: ADC-CLAMP-10 -> ADC-CLAMP-8
- R43 pad 1: ADC-CLAMP-9 -> ADC-CLAMP-7
- R44 pad 1: ADC-CLAMP-4 -> ADC-CLAMP-6
- R45 pad 1: +5V -> VPROT
- R45 pad 2: ADC-CLAMP-8 -> ADC-CLAMP-2
- R55 pad 2: +5V -> VPROT
- R9 pad 1: Net-(R11-Pad1) -> /Sensors/MCU-AC
- R9 pad 2: /FAN+TACH/MCU-FAN -> (no net)
- RV1 pad 2: VBAT -> 12v-SW
- TP10 pad 1: +5V -> VPROT
- TP12 pad 1: VREG -> ADC-CLAMP-6
- TP13 pad 1: VPPREF -> (no net)
- TP14 pad 1: VPPSENS -> (no net)
- TP15 pad 1: VPROT -> (no net)
- TP16 pad 1: ADC-CLAMP-10 -> ADC-CLAMP-8
- TP17 pad 1: ADC-CLAMP-9 -> ADC-CLAMP-7
- TP2 pad 1: ADC-CLAMP-1 -> ADC-CLAMP-3
- TP3 pad 1: ADC-CLAMP-5 -> ADC-CLAMP-1
- TP4 pad 1: ADC-CLAMP-2 -> ADC-CLAMP-4
- TP5 pad 1: ADC-CLAMP-6 -> (no net)
- TP6 pad 1: ADC-CLAMP-3 -> ADC-CLAMP-5
- TP7 pad 1: ADC-CLAMP-8 -> ADC-CLAMP-2
- TP8 pad 1: ADC-CLAMP-4 -> ADC-CLAMP-6
- U1 pad 1: GND -> (no net)
- U1 pad 2: Net-(R1-Pad1) -> VPROT
- U1 pad 3: Net-(U1-Pad3) -> Net-(C47-Pad2)
- U1 pad 4: Net-(R3-Pad1) -> ADC-CLAMP-6
- U1 pad 5: 12v-SW -> (no net)
- U1 pad 6: ST_SIG -> (no net)
- U1 pad 7: ST_SIG -> (no net)
- U1 pad 8: 12v-SW -> (no net)
- U11 pad 3: +3V3 -> VPROT
- U11 pad 5: +3V3 -> VPROT
- U12 pad 1: Net-(U12-Pad1) -> (no net)
- U12 pad 10: Net-(U12-Pad10) -> (no net)
- U12 pad 100: Net-(U12-Pad100) -> (no net)
- U12 pad 101: Net-(U12-Pad101) -> (no net)
- U12 pad 102: Net-(U12-Pad102) -> (no net)
- U12 pad 11: Net-(U12-Pad11) -> (no net)
- U12 pad 110: Net-(U12-Pad110) -> (no net)
- U12 pad 111: Net-(U12-Pad111) -> SDIO_D2
- U12 pad 112: Net-(U12-Pad112) -> SDIO_D3
- U12 pad 113: Net-(U12-Pad113) -> SDIO_CK
- U12 pad 116: ADC-CLAMP-10 -> SDIO_CMD
- U12 pad 117: ADC-CLAMP-9 -> ADC-CLAMP-7
- U12 pad 118: Net-(U12-Pad118) -> ADC-CLAMP-8
- U12 pad 119: ADC-CLAMP-8 -> ADC-CLAMP-2
- U12 pad 12: Net-(U12-Pad12) -> (no net)
- U12 pad 122: Net-(U12-Pad122) -> (no net)
- U12 pad 123: Net-(U12-Pad123) -> (no net)
- U12 pad 124: Net-(U12-Pad124) -> (no net)
- U12 pad 125: Net-(U12-Pad125) -> (no net)
- U12 pad 126: Net-(U12-Pad126) -> (no net)
- U12 pad 127: Net-(U12-Pad127) -> (no net)
- U12 pad 128: Net-(U12-Pad128) -> (no net)
- U12 pad 129: Net-(U12-Pad129) -> (no net)
- U12 pad 13: Net-(U12-Pad13) -> (no net)
- U12 pad 132: Net-(U12-Pad132) -> (no net)
- U12 pad 134: Net-(U12-Pad134) -> (no net)
- U12 pad 135: Net-(U12-Pad135) -> (no net)
- U12 pad 136: Net-(U12-Pad136) -> I2C1_SDL
- U12 pad 137: Net-(U12-Pad137) -> I2C1_SDA
- U12 pad 14: Net-(U12-Pad14) -> (no net)
- U12 pad 140: /FuelPump/MCU-FP -> /FAN+TACH/MCU-FP
- U12 pad 141: Net-(U12-Pad141) -> (no net)
- U12 pad 142: Net-(U12-Pad142) -> (no net)
- U12 pad 15: Net-(U12-Pad15) -> (no net)
- U12 pad 2: Net-(U12-Pad2) -> (no net)
- U12 pad 22: Net-(U12-Pad22) -> (no net)
- U12 pad 26: Net-(U12-Pad26) -> (no net)
- U12 pad 27: Net-(U12-Pad27) -> (no net)
- U12 pad 28: Net-(U12-Pad28) -> (no net)
- U12 pad 29: ADC-CLAMP-4 -> ADC-CLAMP-6
- U12 pad 3: Net-(U12-Pad3) -> (no net)
- U12 pad 34: ADC-CLAMP-1 -> /Ignitors/MCU-IGN-1
- U12 pad 35: ADC-CLAMP-3 -> /Ignitors/MCU-IGN-2
- U12 pad 37: ADC-CLAMP-2 -> ADC-CLAMP-4
- U12 pad 4: Net-(U12-Pad4) -> /mcu/MCU-PWM2
- U12 pad 40: /mc33814/MCU-SPI1-CS -> (no net)
- U12 pad 41: /mc33814/MCU-SPI1-SCK -> (no net)
- U12 pad 42: /mcu/MCU-SPI1-MISO -> (no net)
- U12 pad 43: /mc33814/MCU-SPI1-MISO -> (no net)
- U12 pad 44: ADC-CLAMP-5 -> ADC-CLAMP-1
- U12 pad 45: /mcu/MCU-BARO -> ADC-CLAMP-6
- U12 pad 46: /Ignitors/MCU-IGN-3 -> ADC-CLAMP-3
- U12 pad 47: /Ignitors/MCU-IGN-4 -> ADC-CLAMP-5
- U12 pad 48: Net-(U12-Pad48) -> (no net)
- U12 pad 49: Net-(U12-Pad49) -> (no net)
- U12 pad 5: Net-(U12-Pad5) -> /mcu/MCU-PWM3
- U12 pad 50: Net-(U12-Pad50) -> (no net)
- U12 pad 53: Net-(U12-Pad53) -> (no net)
- U12 pad 54: Net-(U12-Pad54) -> (no net)
- U12 pad 55: Net-(U12-Pad55) -> (no net)
- U12 pad 56: Net-(U12-Pad56) -> (no net)
- U12 pad 57: Net-(U12-Pad57) -> (no net)
- U12 pad 58: Net-(U12-Pad58) -> (no net)
- U12 pad 59: Net-(U12-Pad59) -> (no net)
- U12 pad 63: Net-(U12-Pad63) -> (no net)
- U12 pad 65: Net-(U12-Pad65) -> (no net)
- U12 pad 68: Net-(U12-Pad68) -> (no net)
- U12 pad 69: /mc33814/MCU-RIN1 -> /Ignitors/MCU-IGN-3
- U12 pad 7: Net-(U12-Pad7) -> (no net)
- U12 pad 70: /mc33814/MCU-RIN2 -> /Ignitors/MCU-IGN-4
- U12 pad 73: Net-(U12-Pad73) -> /Sensors/MCU-CLUTCH
- U12 pad 74: /mcu/MCU-AC -> /Sensors/MCU-AC
- U12 pad 76: /Sensors/MCU-CLUTCH -> (no net)
- U12 pad 77: Net-(U12-Pad77) -> (no net)
- U12 pad 78: Net-(U12-Pad78) -> (no net)
- U12 pad 79: Net-(U12-Pad79) -> (no net)
- U12 pad 8: Net-(U12-Pad8) -> (no net)
- U12 pad 80: Net-(U12-Pad80) -> (no net)
- U12 pad 81: Net-(U12-Pad81) -> /mcu/MCU-VVT
- U12 pad 82: Net-(U12-Pad82) -> /mcu/MCU-PWM1
- U12 pad 85: Net-(U12-Pad85) -> (no net)
- U12 pad 86: Net-(U12-Pad86) -> (no net)
- U12 pad 87: Net-(U12-Pad87) -> /Sensors/MCU-ANALOG-1
- U12 pad 88: Net-(U12-Pad88) -> /Sensors/MCU-ANALOG-2
- U12 pad 89: Net-(U12-Pad89) -> /Sensors/MCU-ANALOG-3
- U12 pad 9: Net-(U12-Pad9) -> (no net)
- U12 pad 90: Net-(U12-Pad90) -> /Sensors/MCU-ANALOG-4
- U12 pad 91: Net-(U12-Pad91) -> (no net)
- U12 pad 92: Net-(U12-Pad92) -> (no net)
- U12 pad 93: Net-(U12-Pad93) -> (no net)
- U12 pad 96: /Ignitors/MCU-IGN-1 -> (no net)
- U12 pad 97: /Ignitors/MCU-IGN-2 -> (no net)
- U12 pad 98: Net-(U12-Pad98) -> SDIO_D0
- U12 pad 99: Net-(U12-Pad99) -> SDIO_D1
- U13 pad 2: Net-(U13-Pad2) -> (no net)
- U13 pad 4: Net-(U13-Pad4) -> (no net)
- U14 pad 2: Net-(U14-Pad2) -> (no net)
- U14 pad 4: Net-(U14-Pad4) -> (no net)
- U2 pad 2: Net-(U2-Pad2) -> (no net)
- U2 pad 4: Net-(U2-Pad4) -> (no net)
- U3 pad 1: Net-(R11-Pad1) -> Net-(R81-Pad1)
- U3 pad 2: Net-(U3-Pad2) -> (no net)
- U3 pad 3: Net-(R10-Pad1) -> Net-(R82-Pad1)
- U3 pad 4: Net-(U3-Pad4) -> (no net)
- U3 pad 6: Net-(JP1-Pad1) -> /spare-pwms/HC-1
- U3 pad 8: FAN -> /spare-pwms/VVT-OUT
- U4 pad 1: Net-(U4-Pad1) -> (no net)
- U4 pad 6: +5V -> VPROT
- U4 pad 8: Net-(U4-Pad8) -> (no net)
- U5 pad 1: Net-(U5-Pad1) -> (no net)
- U5 pad 6: +5V -> VPROT
- U5 pad 8: Net-(U5-Pad8) -> (no net)
- U6 pad 10: Net-(U6-Pad10) -> ADC-CLAMP-9
- U6 pad 11: Net-(U6-Pad11) -> (no net)
- U6 pad 12: Net-(U6-Pad12) -> ADC-CLAMP-11
- U6 pad 13: ADC-CLAMP-10 -> ADC-CLAMP-12
- U6 pad 14: ADC-CLAMP-9 -> ADC-CLAMP-13
- U6 pad 15: ADC-CLAMP-8 -> (no net)
- U6 pad 16: +5V -> VPROT
- U6 pad 7: Net-(U6-Pad7) -> ADC-CLAMP-7
- U6 pad 9: Net-(U6-Pad9) -> ADC-CLAMP-8
- U7 pad 1: Net-(R38-Pad1) -> Net-(R83-Pad1)
- U7 pad 2: GND -> (no net)
- U7 pad 3: VPROT -> Net-(R84-Pad1)
- U7 pad 5: (no net) -> GND
- U7 pad 6: (no net) -> /spare-pwms/HC-3
- U8 pad 2: Net-(U8-Pad2) -> (no net)
- U8 pad 3: Net-(U8-Pad3) -> (no net)
- U8 pad 7: +5V -> VPROT
- U9 pad 2: Net-(U9-Pad2) -> (no net)
- U9 pad 3: Net-(U9-Pad3) -> (no net)
Routing:
- net GND: track 323.3 -> 0.00 mm, vias 80 -> 0
- net +5V: track 250.9 -> 0.00 mm, vias 14 -> 0
- net BOOST: track 212.5 -> 0.00 mm, vias 3 -> 0
- net 12v-SW: track 211.1 -> 0.00 mm, vias 7 -> 0
- net IDLE: track 210.1 -> 0.00 mm, vias 3 -> 0
- net FAN: track 203.4 -> 0.00 mm, vias 3 -> 0
- net VBAT: track 195.7 -> 0.00 mm, vias 1 -> 0
- net Net-(JP1-Pad1): track 191.4 -> 0.00 mm, vias 2 -> 0
- net /FuelPump/MCU-FP: track 157.0 -> 0.00 mm, vias 3 -> 0
- net NRST: track 149.3 -> 0.00 mm, vias 5 -> 0
- net MCU-CAN-TX: track 147.5 -> 0.00 mm, vias 3 -> 0
- net MCU-CAN-RX: track 146.0 -> 0.00 mm, vias 3 -> 0
- net VPROT: track 141.1 -> 0.00 mm, vias 5 -> 0
- net ADC-CLAMP-8: track 139.6 -> 0.00 mm, vias 1 -> 0
- net ADC-CLAMP-10: track 137.7 -> 0.00 mm, vias 2 -> 0
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- removed copper zone on In2.Cu, net +3V3
- removed copper zone on In2.Cu, net +5V
- removed copper zone on In2.Cu, net 12v-SW
- removed copper zone on B.Cu, net GND
- removed copper zone on F.Cu, net GND
- removed copper zone on In1.Cu, net GND
- removed copper zone on In2.Cu, net USB_CONN_VBUS
Other:
- board text removed: "FUEL"
- board text removed: "IGN1"
- board text removed: "IGN2"
- board text removed: "IGN3"
- board text removed: "IGN4"
- board text removed: "INJ1"
- board text removed: "INJ2"
- board text removed: "INJ3"
- board text removed: "INJ4"

Commit message: Layout checkpoint: everything fits on the board
Parts:
- TP22: value TP_VPROT -> TP_REG_IN
- moved Q4 232.0 mm to (18.8, 85.2), turned to 180 degrees
- moved Q3 223.2 mm to (23.2, 85.2), turned to 180 degrees
- moved TP12 221.6 mm to (47.8, 99.3)
- moved R4 220.1 mm to (57.2, 104.7), turned to 270 degrees
- moved TP5 219.4 mm to (50.5, 82.8), turned to 180 degrees
- moved TP15 219.1 mm to (51.7, 84.2), turned to 45 degrees
- moved C48 216.1 mm to (51.1, 79.1), turned to 45 degrees
- moved Q2 214.3 mm to (27.7, 85.2), turned to 180 degrees
- moved TP14 213.9 mm to (53.6, 85.8), turned to 45 degrees
- moved R1 213.5 mm to (27.7, 81.6), turned to 180 degrees
- moved TP13 212.2 mm to (48.9, 81.3), turned to 45 degrees
- moved R13 210.4 mm to (68.4, 104.8), turned to 270 degrees
- moved R38 206.9 mm to (64.5, 99.1), turned to 270 degrees
- moved R10 206.8 mm to (61.3, 104.7), turned to 270 degrees
- moved R2 204.7 mm to (57.2, 99.2), turned to 270 degrees
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Connections:
- C12 pad 2: ADC-CLAMP-8 -> ADC-CLAMP-14
- C42 pad 1: HSE_OUT -> LSE_OUT
- C46 pad 1: /Sensors/MCU-ANALOG-4 -> /Sensors/ANALOG-4-IN
- C49 pad 1: /Sensors/MCU-ANALOG-1 -> /Sensors/ANALOG-1-IN
- C5 pad 1: /Sensors/MCU-ANALOG-3 -> /Sensors/ANALOG-3-IN
- C51 pad 1: /Sensors/MCU-ANALOG-2 -> /Sensors/ANALOG-2-IN
- D35 pad 1: (no net) -> VREG
- J1 pad A3: (no net) -> Net-(J1-PadA3)
- J1 pad A4: (no net) -> Net-(J1-PadA4)
- J1 pad A5: (no net) -> Net-(J1-PadA5)
- J1 pad A6: (no net) -> Net-(J1-PadA6)
- J1 pad A7: (no net) -> Net-(J1-PadA7)
- J1 pad B1: (no net) -> ST_SIG
- J2 pad A8: (no net) -> Net-(J2-PadA8)
- J3 pad 7: (no net) -> Net-(J3-Pad7)
- J3 pad 8: (no net) -> Net-(J3-Pad8)
- J6 pad 10: (no net) -> Net-(J6-Pad10)
- J6 pad 9: (no net) -> Net-(J6-Pad9)
- J7 pad 1: (no net) -> Net-(J7-Pad1)
- J7 pad 6: (no net) -> Net-(J7-Pad6)
- R10 pad 2: /Sensors/MCU-ANALOG-4 -> /Sensors/ANALOG-4-IN
- R12 pad 2: /Sensors/MCU-ANALOG-1 -> /Sensors/ANALOG-1-IN
- R13 pad 2: /Sensors/MCU-ANALOG-1 -> /Sensors/ANALOG-1-IN
- R2 pad 2: /Sensors/MCU-ANALOG-3 -> /Sensors/ANALOG-3-IN
- R3 pad 2: /Sensors/MCU-ANALOG-3 -> /Sensors/ANALOG-3-IN
- R38 pad 2: /Sensors/MCU-ANALOG-2 -> /Sensors/ANALOG-2-IN
- R4 pad 2: /Sensors/MCU-ANALOG-4 -> /Sensors/ANALOG-4-IN
- R42 pad 1: ADC-CLAMP-8 -> ADC-CLAMP-14
- R48 pad 2: HSE_IN -> LSE_IN
- R80 pad 2: /Sensors/MCU-ANALOG-2 -> /Sensors/ANALOG-2-IN
- R9 pad 2: (no net) -> /Sensors/AC-IN
- TP13 pad 1: (no net) -> ADC-CLAMP-13
- TP14 pad 1: (no net) -> ADC-CLAMP-9
- TP15 pad 1: (no net) -> ADC-CLAMP-11
- TP16 pad 1: ADC-CLAMP-8 -> ADC-CLAMP-14
- TP22 pad 1: VPROT -> 12v-SW
- TP5 pad 1: (no net) -> ADC-CLAMP-12
- U1 pad 1: (no net) -> Net-(U1-Pad1)
- U1 pad 5: (no net) -> Net-(U1-Pad5)
- U1 pad 6: (no net) -> Net-(U1-Pad6)
- U1 pad 7: (no net) -> Net-(U1-Pad7)
- U1 pad 8: (no net) -> Net-(U1-Pad8)
- U12 pad 1: (no net) -> Net-(U12-Pad1)
- U12 pad 10: (no net) -> Net-(U12-Pad10)
- U12 pad 100: (no net) -> /mcu/MCU-CEL
- U12 pad 101: (no net) -> /mcu/MCU-RN1
- U12 pad 102: (no net) -> /mcu/MCU-RN2
- U12 pad 11: (no net) -> Net-(U12-Pad11)
- U12 pad 110: (no net) -> Net-(U12-Pad110)
- U12 pad 118: ADC-CLAMP-8 -> ADC-CLAMP-14
- U12 pad 12: (no net) -> Net-(U12-Pad12)
- U12 pad 122: (no net) -> Net-(U12-Pad122)
- U12 pad 123: (no net) -> Net-(U12-Pad123)
- U12 pad 124: (no net) -> Net-(U12-Pad124)
- U12 pad 125: (no net) -> Net-(U12-Pad125)
- U12 pad 126: (no net) -> Net-(U12-Pad126)
- U12 pad 127: (no net) -> Net-(U12-Pad127)
- U12 pad 128: (no net) -> Net-(U12-Pad128)
- U12 pad 129: (no net) -> Net-(U12-Pad129)
- U12 pad 13: (no net) -> Net-(U12-Pad13)
- U12 pad 132: (no net) -> Net-(U12-Pad132)
- U12 pad 134: (no net) -> Net-(U12-Pad134)
- U12 pad 135: (no net) -> Net-(U12-Pad135)
- U12 pad 14: (no net) -> Net-(U12-Pad14)
- U12 pad 141: (no net) -> Net-(U12-Pad141)
- U12 pad 142: (no net) -> Net-(U12-Pad142)
- U12 pad 15: (no net) -> Net-(U12-Pad15)
- U12 pad 2: (no net) -> Net-(U12-Pad2)
- U12 pad 22: (no net) -> Net-(U12-Pad22)
- U12 pad 26: (no net) -> Net-(U12-Pad26)
- U12 pad 27: (no net) -> Net-(U12-Pad27)
- U12 pad 28: (no net) -> Net-(U12-Pad28)
- U12 pad 3: (no net) -> Net-(U12-Pad3)
- U12 pad 40: (no net) -> /mcu/MCU-SPI1-CS
- U12 pad 41: (no net) -> /mcu/MCU-SPI1-SCK
- U12 pad 42: (no net) -> /mcu/MCU-SPI1-MISO
- U12 pad 43: (no net) -> /mcu/MCU-SPI1-MOSI
- U12 pad 48: (no net) -> Net-(U12-Pad48)
- U12 pad 49: (no net) -> Net-(U12-Pad49)
- U12 pad 50: (no net) -> Net-(U12-Pad50)
- U12 pad 53: (no net) -> Net-(U12-Pad53)
- U12 pad 54: (no net) -> Net-(U12-Pad54)
- U12 pad 55: (no net) -> Net-(U12-Pad55)
- U12 pad 56: (no net) -> Net-(U12-Pad56)
- U12 pad 57: (no net) -> Net-(U12-Pad57)
- U12 pad 58: (no net) -> Net-(U12-Pad58)
- U12 pad 59: (no net) -> Net-(U12-Pad59)
- U12 pad 63: (no net) -> Net-(U12-Pad63)
- U12 pad 65: (no net) -> Net-(U12-Pad65)
- U12 pad 68: (no net) -> Net-(U12-Pad68)
- U12 pad 7: (no net) -> Net-(U12-Pad7)
- U12 pad 76: (no net) -> Net-(U12-Pad76)
- U12 pad 77: (no net) -> Net-(U12-Pad77)
- U12 pad 78: (no net) -> Net-(U12-Pad78)
- U12 pad 79: (no net) -> Net-(U12-Pad79)
- U12 pad 8: (no net) -> LSE_IN
- U12 pad 80: (no net) -> Net-(U12-Pad80)
- U12 pad 85: (no net) -> Net-(U12-Pad85)
- U12 pad 86: (no net) -> Net-(U12-Pad86)
- U12 pad 87: /Sensors/MCU-ANALOG-1 -> ADC-CLAMP-9
- U12 pad 88: /Sensors/MCU-ANALOG-2 -> ADC-CLAMP-11
- U12 pad 89: /Sensors/MCU-ANALOG-3 -> ADC-CLAMP-12
- U12 pad 9: (no net) -> LSE_OUT
- U12 pad 90: /Sensors/MCU-ANALOG-4 -> ADC-CLAMP-13
- U12 pad 91: (no net) -> Net-(U12-Pad91)
- U12 pad 92: (no net) -> Net-(U12-Pad92)
- U12 pad 93: (no net) -> Net-(U12-Pad93)
- U12 pad 96: (no net) -> Net-(U12-Pad96)
- U12 pad 97: (no net) -> Net-(U12-Pad97)
- U13 pad 2: (no net) -> Net-(U13-Pad2)
- U13 pad 4: (no net) -> Net-(U13-Pad4)
- U14 pad 2: (no net) -> Net-(U14-Pad2)
- U14 pad 4: (no net) -> Net-(U14-Pad4)
- U2 pad 2: (no net) -> Net-(U2-Pad2)
- U2 pad 4: (no net) -> Net-(U2-Pad4)
- U3 pad 2: (no net) -> Net-(U3-Pad2)
- U3 pad 4: (no net) -> Net-(U3-Pad4)
- U4 pad 1: (no net) -> Net-(U4-Pad1)
- U4 pad 8: (no net) -> Net-(U4-Pad8)
- U5 pad 1: (no net) -> Net-(U5-Pad1)
- U5 pad 8: (no net) -> Net-(U5-Pad8)
- U6 pad 11: (no net) -> ADC-CLAMP-10
- U6 pad 15: (no net) -> ADC-CLAMP-14
- U7 pad 2: (no net) -> Net-(U7-Pad2)
- U7 pad 4: (no net) -> Net-(U7-Pad4)
- U8 pad 2: (no net) -> Net-(U8-Pad2)
- U8 pad 3: (no net) -> Net-(U8-Pad3)
- U9 pad 2: (no net) -> Net-(U9-Pad2)
- U9 pad 3: (no net) -> Net-(U9-Pad3)
- Y2 pad 1: HSE_OUT -> LSE_OUT
Routing:
- net LSE_OUT: track 0.00 -> 10.8 mm
- net /mcu/MCU-PWM3: track 0.00 -> 6.63 mm
- net /mcu/MCU-PWM2: track 0.00 -> 6.59 mm
- net Net-(C52-Pad1): track 0.00 -> 4.83 mm
- net GND: track 0.00 -> 3.73 mm, vias 0 -> 3
- net +3V3: track 76.9 -> 78.9 mm
- net LSE_IN: track 0.00 -> 1.70 mm

Commit message: Finish reroute again
Parts:
- removed JP1: Jumper, Jumper:SolderJumper-2_P1.3mm_Open_RoundedPad1.0x1.5mm
- removed TP1: TP_TACH, TestPoint:TestPoint_Pad_D1.0mm
- moved TP9 96.0 mm to (31.6, 29.1)
- moved J3 96.0 mm to (36.2, 26.5)
- moved C24 83.9 mm to (86.2, 30.7)
- moved U11 83.9 mm to (80.6, 30.7)
- moved C23 83.9 mm to (76.2, 30.7)
- moved R58 83.9 mm to (85.1, 30.7)
- moved R4 80.5 mm to (108.7, 42.7), turned to 45 degrees
- moved R33 80.1 mm to (109.7, 60.2), turned to 45 degrees
- moved C46 79.5 mm to (107.2, 41.3), turned to 225 degrees
- moved R10 78.7 mm to (105.8, 39.8), turned to 45 degrees
- moved D7 77.8 mm to (111.2, 61.5), turned to 45 degrees
- moved R32 76.6 mm to (96.5, 91.4), turned to 135 degrees
- moved R35 76.2 mm to (90.6, 82.7), turned to 315 degrees
- moved Q3 76.2 mm to (92.3, 117.3), turned to 270 degrees
- moved R1 76.1 mm to (94.9, 117.3), turned to 270 degrees
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Connections:
- C11 pad 1: ADC-CLAMP-5 -> ADC-CLAMP-14
- C12 pad 2: ADC-CLAMP-14 -> ADC-CLAMP-5
- C13 pad 1: ADC-CLAMP-7 -> ADC-CLAMP-6
- C15 pad 1: ADC-CLAMP-6 -> ADC-CLAMP-11
- C3 pad 1: ADC-CLAMP-3 -> ADC-CLAMP-13
- C4 pad 1: ADC-CLAMP-1 -> ADC-CLAMP-12
- C46 pad 1: /Sensors/ANALOG-4-IN -> A4
- C48 pad 1: ADC-CLAMP-13 -> ADC-CLAMP-4
- C49 pad 1: /Sensors/ANALOG-1-IN -> A1
- C5 pad 1: /Sensors/ANALOG-3-IN -> A3
- C50 pad 1: ADC-CLAMP-9 -> ADC-CLAMP-1
- C51 pad 1: /Sensors/ANALOG-2-IN -> A2
- C55 pad 1: ADC-CLAMP-11 -> ADC-CLAMP-2
- C7 pad 1: ADC-CLAMP-12 -> ADC-CLAMP-3
- C8 pad 1: ADC-CLAMP-4 -> ADC-CLAMP-10
- D21 pad 2: /spare-pwms/VVT-OUT -> VVT
- D31 pad 2: /spare-pwms/HC-1 -> HC1
- D32 pad 2: /spare-pwms/HC-2 -> HC2
- D33 pad 2: /spare-pwms/HC-3 -> HC3
- D35 pad 1: VREG -> (no net)
- J1 pad A1: VBAT -> (no net)
- J1 pad A3: Net-(J1-PadA3) -> GND
- J1 pad A4: Net-(J1-PadA4) -> GND
- J1 pad A5: Net-(J1-PadA5) -> GND
- J1 pad A6: Net-(J1-PadA6) -> GND
- J1 pad A7: Net-(J1-PadA7) -> VPROT
- J1 pad A8: VPROT -> VBAT
- J1 pad B1: ST_SIG -> GND
- J1 pad B5: GND -> A4
- J1 pad B6: GND -> A3
- J1 pad B7: GND -> A2
- J1 pad B8: GND -> A1
- J1 pad C1: IGN-2 -> IGN-1
- J1 pad C2: IGN-1 -> IGN-2
- J1 pad C3: IGN-4 -> IGN-3
- J1 pad C4: IGN-3 -> IGN-4
- J1 pad C5: INJ-2 -> INJ-1
- J1 pad C6: INJ-1 -> INJ-2
- J1 pad C7: INJ-4 -> INJ-3
- J1 pad C8: INJ-3 -> INJ-4
- J2 pad A1: CRANK -> AC
- J2 pad A2: CAM -> CLUTCH
- J2 pad A3: CLUTCH -> TPS
- J2 pad A4: O2 -> IAT
- J2 pad A5: TPS -> CLT
- J2 pad A6: CLT -> O2
- J2 pad A7: IAT -> CAM
- J2 pad A8: Net-(J2-PadA8) -> CRANK
- J2 pad B1: CANH -> HC2
- J2 pad B2: CANL -> HC3
- J2 pad B3: FP -> VVT
- J2 pad B4: GND -> HC1
- J2 pad B7: GND -> IDLE
- J2 pad B8: GND -> BOOST
- J2 pad C1: TACH -> GND
- J2 pad C2: FAN -> GND
- J2 pad C3: IDLE -> FP
- J2 pad C4: BOOST -> FAN
- J2 pad C5: GND -> TACH
- J2 pad C6: GND -> CANH
- J2 pad C7: GND -> CANL
- J2 pad C8: ADC-CLAMP-2 -> ADC-CLAMP-7
- J3 pad 7: Net-(J3-Pad7) -> (no net)
- J3 pad 8: Net-(J3-Pad8) -> (no net)
- J6 pad 10: Net-(J6-Pad10) -> (no net)
- J6 pad 11: USB_CONN_SHIELD -> Net-(J6-Pad11)
- J6 pad 9: Net-(J6-Pad9) -> (no net)
- J7 pad 1: Net-(J7-Pad1) -> (no net)
- J7 pad 6: Net-(J7-Pad6) -> (no net)
- Q3 pad 3: Net-(JP1-Pad1) -> TACH
- R1 pad 1: Net-(JP1-Pad1) -> TACH
- R10 pad 1: ADC-CLAMP-13 -> ADC-CLAMP-4
- R10 pad 2: /Sensors/ANALOG-4-IN -> A4
- R11 pad 1: ADC-CLAMP-6 -> ADC-CLAMP-9
- R12 pad 2: /Sensors/ANALOG-1-IN -> A1
- R13 pad 1: ADC-CLAMP-9 -> ADC-CLAMP-1
- R13 pad 2: /Sensors/ANALOG-1-IN -> A1
- R2 pad 2: /Sensors/ANALOG-3-IN -> A3
- R3 pad 1: ADC-CLAMP-12 -> ADC-CLAMP-3
- R3 pad 2: /Sensors/ANALOG-3-IN -> A3
- R34 pad 1: ADC-CLAMP-3 -> ADC-CLAMP-13
- R35 pad 1: ADC-CLAMP-1 -> ADC-CLAMP-12
- R37 pad 1: ADC-CLAMP-4 -> ADC-CLAMP-10
- R38 pad 2: /Sensors/ANALOG-2-IN -> A2
- R4 pad 2: /Sensors/ANALOG-4-IN -> A4
- R41 pad 1: ADC-CLAMP-5 -> ADC-CLAMP-14
- R42 pad 1: ADC-CLAMP-14 -> ADC-CLAMP-5
- R43 pad 1: ADC-CLAMP-7 -> ADC-CLAMP-6
- R44 pad 1: ADC-CLAMP-6 -> ADC-CLAMP-11
- R45 pad 2: ADC-CLAMP-2 -> ADC-CLAMP-7
- R76 pad 2: +3V3 -> SDIO_VDD
- R77 pad 2: +3V3 -> SDIO_VDD
- R78 pad 2: +3V3 -> SDIO_VDD
- R79 pad 2: +3V3 -> SDIO_VDD
- R80 pad 1: ADC-CLAMP-11 -> ADC-CLAMP-2
- R80 pad 2: /Sensors/ANALOG-2-IN -> A2
- R9 pad 2: /Sensors/AC-IN -> AC
- TP12 pad 1: ADC-CLAMP-6 -> ADC-CLAMP-9
- TP13 pad 1: ADC-CLAMP-13 -> ADC-CLAMP-4
- TP14 pad 1: ADC-CLAMP-9 -> ADC-CLAMP-1
- TP15 pad 1: ADC-CLAMP-11 -> ADC-CLAMP-2
- TP16 pad 1: ADC-CLAMP-14 -> ADC-CLAMP-5
- TP17 pad 1: ADC-CLAMP-7 -> ADC-CLAMP-6
- TP2 pad 1: ADC-CLAMP-3 -> ADC-CLAMP-13
- TP3 pad 1: ADC-CLAMP-1 -> ADC-CLAMP-12
- TP4 pad 1: ADC-CLAMP-4 -> ADC-CLAMP-10
- TP5 pad 1: ADC-CLAMP-12 -> ADC-CLAMP-3
- TP6 pad 1: ADC-CLAMP-5 -> ADC-CLAMP-14
- TP7 pad 1: ADC-CLAMP-2 -> ADC-CLAMP-7
- TP8 pad 1: ADC-CLAMP-6 -> ADC-CLAMP-11
- U1 pad 1: Net-(U1-Pad1) -> (no net)
- U1 pad 4: ADC-CLAMP-6 -> ADC-CLAMP-9
- U1 pad 5: Net-(U1-Pad5) -> (no net)
- U1 pad 6: Net-(U1-Pad6) -> (no net)
- U1 pad 7: Net-(U1-Pad7) -> (no net)
- U1 pad 8: Net-(U1-Pad8) -> (no net)
- U12 pad 1: Net-(U12-Pad1) -> (no net)
- U12 pad 10: Net-(U12-Pad10) -> (no net)
- U12 pad 100: /mcu/MCU-CEL -> (no net)
- U12 pad 101: /mcu/MCU-RN1 -> (no net)
- U12 pad 102: /mcu/MCU-RN2 -> (no net)
- U12 pad 11: Net-(U12-Pad11) -> (no net)
- U12 pad 110: Net-(U12-Pad110) -> (no net)
- U12 pad 117: ADC-CLAMP-7 -> ADC-CLAMP-6
- U12 pad 118: ADC-CLAMP-14 -> ADC-CLAMP-5
- U12 pad 119: ADC-CLAMP-2 -> ADC-CLAMP-7
- U12 pad 12: Net-(U12-Pad12) -> (no net)
- U12 pad 122: Net-(U12-Pad122) -> (no net)
- U12 pad 123: Net-(U12-Pad123) -> (no net)
- U12 pad 124: Net-(U12-Pad124) -> (no net)
- U12 pad 125: Net-(U12-Pad125) -> (no net)
- U12 pad 126: Net-(U12-Pad126) -> (no net)
- U12 pad 127: Net-(U12-Pad127) -> (no net)
- U12 pad 128: Net-(U12-Pad128) -> (no net)
- U12 pad 129: Net-(U12-Pad129) -> (no net)
- U12 pad 13: Net-(U12-Pad13) -> (no net)
- U12 pad 132: Net-(U12-Pad132) -> (no net)
- U12 pad 134: Net-(U12-Pad134) -> (no net)
- U12 pad 135: Net-(U12-Pad135) -> (no net)
- U12 pad 14: Net-(U12-Pad14) -> (no net)
- U12 pad 141: Net-(U12-Pad141) -> (no net)
- U12 pad 142: Net-(U12-Pad142) -> (no net)
- U12 pad 15: Net-(U12-Pad15) -> (no net)
- U12 pad 2: Net-(U12-Pad2) -> (no net)
- U12 pad 22: Net-(U12-Pad22) -> (no net)
- U12 pad 26: Net-(U12-Pad26) -> (no net)
- U12 pad 27: Net-(U12-Pad27) -> (no net)
- U12 pad 28: Net-(U12-Pad28) -> (no net)
- U12 pad 29: ADC-CLAMP-6 -> ADC-CLAMP-11
- U12 pad 3: Net-(U12-Pad3) -> (no net)
- U12 pad 36: ADC-CLAMP-6 -> ADC-CLAMP-9
- U12 pad 37: ADC-CLAMP-4 -> ADC-CLAMP-10
- U12 pad 4: /mcu/MCU-PWM2 -> /mcu/MCU-PWM3
- U12 pad 40: /mcu/MCU-SPI1-CS -> (no net)
- U12 pad 41: /mcu/MCU-SPI1-SCK -> (no net)
- U12 pad 42: /mcu/MCU-SPI1-MISO -> (no net)
- U12 pad 43: /mcu/MCU-SPI1-MOSI -> (no net)
- U12 pad 44: ADC-CLAMP-1 -> ADC-CLAMP-12
- U12 pad 45: ADC-CLAMP-6 -> (no net)
- U12 pad 46: ADC-CLAMP-3 -> ADC-CLAMP-13
- U12 pad 47: ADC-CLAMP-5 -> ADC-CLAMP-14
- U12 pad 48: Net-(U12-Pad48) -> (no net)
- U12 pad 49: Net-(U12-Pad49) -> (no net)
- U12 pad 5: /mcu/MCU-PWM3 -> /mcu/MCU-PWM2
- U12 pad 50: Net-(U12-Pad50) -> (no net)
- U12 pad 53: Net-(U12-Pad53) -> (no net)
- U12 pad 54: Net-(U12-Pad54) -> (no net)
- U12 pad 55: Net-(U12-Pad55) -> (no net)
- U12 pad 56: Net-(U12-Pad56) -> (no net)
- U12 pad 57: Net-(U12-Pad57) -> (no net)
- U12 pad 58: Net-(U12-Pad58) -> (no net)
- U12 pad 59: Net-(U12-Pad59) -> (no net)
- U12 pad 63: Net-(U12-Pad63) -> (no net)
- U12 pad 65: Net-(U12-Pad65) -> (no net)
- U12 pad 68: Net-(U12-Pad68) -> (no net)
- U12 pad 7: Net-(U12-Pad7) -> (no net)
- U12 pad 76: Net-(U12-Pad76) -> (no net)
- U12 pad 77: Net-(U12-Pad77) -> (no net)
- U12 pad 78: Net-(U12-Pad78) -> (no net)
- U12 pad 79: Net-(U12-Pad79) -> (no net)
- U12 pad 80: Net-(U12-Pad80) -> (no net)
- U12 pad 85: Net-(U12-Pad85) -> (no net)
- U12 pad 86: Net-(U12-Pad86) -> (no net)
- U12 pad 87: ADC-CLAMP-9 -> ADC-CLAMP-1
- U12 pad 88: ADC-CLAMP-11 -> ADC-CLAMP-2
- U12 pad 89: ADC-CLAMP-12 -> ADC-CLAMP-3
- U12 pad 90: ADC-CLAMP-13 -> ADC-CLAMP-4
- U12 pad 91: Net-(U12-Pad91) -> (no net)
- U12 pad 92: Net-(U12-Pad92) -> (no net)
- U12 pad 93: Net-(U12-Pad93) -> (no net)
- U12 pad 96: Net-(U12-Pad96) -> (no net)
- U12 pad 97: Net-(U12-Pad97) -> (no net)
- U13 pad 2: Net-(U13-Pad2) -> (no net)
- U13 pad 4: Net-(U13-Pad4) -> (no net)
- U14 pad 2: Net-(U14-Pad2) -> (no net)
- U14 pad 4: Net-(U14-Pad4) -> (no net)
- U2 pad 2: Net-(U2-Pad2) -> (no net)
- U2 pad 4: Net-(U2-Pad4) -> (no net)
- U3 pad 2: Net-(U3-Pad2) -> (no net)
- U3 pad 4: Net-(U3-Pad4) -> (no net)
- U3 pad 6: /spare-pwms/HC-1 -> HC1
- U3 pad 8: /spare-pwms/VVT-OUT -> VVT
- U4 pad 1: Net-(U4-Pad1) -> (no net)
- U4 pad 8: Net-(U4-Pad8) -> (no net)
- U5 pad 1: Net-(U5-Pad1) -> (no net)
- U5 pad 8: Net-(U5-Pad8) -> (no net)
- U6 pad 9: ADC-CLAMP-8 -> (no net)
- U7 pad 2: Net-(U7-Pad2) -> (no net)
- U7 pad 4: Net-(U7-Pad4) -> (no net)
- U7 pad 6: /spare-pwms/HC-3 -> HC3
- U7 pad 8: /spare-pwms/HC-2 -> HC2
- U8 pad 2: Net-(U8-Pad2) -> (no net)
- U8 pad 3: Net-(U8-Pad3) -> (no net)
- U9 pad 2: Net-(U9-Pad2) -> (no net)
- U9 pad 3: Net-(U9-Pad3) -> (no net)
Routing:
- net VPROT: track 0.00 -> 419.6 mm, vias 0 -> 19
- net GND: track 3.73 -> 290.5 mm, vias 3 -> 93
- net 12v-SW: track 0.00 -> 196.2 mm, vias 0 -> 4
- net CANH: track 0.00 -> 187.2 mm, vias 0 -> 1
- net CANL: track 0.00 -> 182.4 mm, vias 0 -> 1
- net NRST: track 0.00 -> 145.7 mm, vias 0 -> 2
- net CAM: track 0.00 -> 145.3 mm, vias 0 -> 1
- net CRANK: track 0.00 -> 138.7 mm, vias 0 -> 1
- net ADC-CLAMP-7: track 0.00 -> 136.7 mm, vias 0 -> 3
- net /mcu/MCU-VVT: track 0.00 -> 134.5 mm, vias 0 -> 3
- net /mcu/MCU-PWM1: track 0.00 -> 128.5 mm, vias 0 -> 3
- net BOOST: track 0.00 -> 127.1 mm, vias 0 -> 1
- net ADC-CLAMP-4: track 0.00 -> 117.0 mm, vias 0 -> 2
- net SDIO_CMD: track 0.00 -> 116.6 mm, vias 0 -> 3
- net IDLE: track 0.00 -> 112.9 mm, vias 0 -> 1
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- added copper zone on In1.Cu, net +3V3
- added copper zone on B.Cu, net GND
- added copper zone on F.Cu, net GND
- added copper zone on In1.Cu, net GND
- added copper zone on In1.Cu, net SDIO_VDD
- added copper zone on In1.Cu, net VPROT

Commit message: Reload netlist for new LED nets
Parts:
- D23: value PWR_5V_GREEN -> PWR_3V_GREEN
- D24: value PWR_3V_RED -> PWR_5V_RED
- R74: value null -> 220
- R75: value null -> 330
