File: Ignitors.sch (KiCad schematic (older format))
At the start: 11 parts

Commit message: Starting on layout
Parts:
- added D11, D12: LED, LED_SMD:LED_0603_1608Metric, symbol Device:LED
- added JP2, JP3: Jumper_3_Open, Connector_PinHeader_2.54mm:PinHeader_1x03_P2.54mm_Vertical_SMD_Pin1Left, symbol Jumper:Jumper_3_Open
- added R27, R28: 1k, Resistor_SMD:R_0603_1608Metric_Pad1.05x0.95mm_HandSolder, symbol Device:R
- added R31, R32: 100k, Resistor_SMD:R_0603_1608Metric_Pad1.05x0.95mm_HandSolder, symbol Device:R
- added R35, R36: 2.4k, Resistor_SMD:R_0603_1608Metric_Pad1.05x0.95mm_HandSolder, symbol Device:R
- added R39, R40: 10, Resistor_SMD:R_0603_1608Metric_Pad1.05x0.95mm_HandSolder, symbol Device:R
- added U7: TC4424A, Package_SO:SOIC-8_3.9x4.9mm_P1.27mm, symbol speeduino_ic_automotive:TC4424A
- D13, D14: renamed from D?; footprint (none) -> LED_SMD:LED_0603_1608Metric
- R29, R30, R33, R34, R37, R38, R41, R42: renamed from R?; footprint (none) -> Resistor_SMD:R_0603_1608Metric_Pad1.05x0.95mm_HandSolder
- gave numbers to parts that had none: 1
Connections:
- net 5v: now also U7.6 (VDD)
- net GND: now also D11.1 (K), D12.1 (K), R31.2, R32.1, U7.3 (GND)
- net at R38.2, R42.2, U8.5 (OUT_B): now also JP3.1 (A)
- net at R37.1, R41.1, U8.7 (OUT_A): now also JP2.1 (A)
- new net: R27.1, R31.1, U7.2 (IN_A)
- new net: R28.1, R32.2, U7.4 (IN_B)
- new net: R36.2, R40.2, U7.5 (OUT_B)
- new net: R35.1, R39.1, U7.7 (OUT_A)
- new net: JP3.3 (B), R40.1
- new net: D12.2 (A), R36.1
- new net: D11.2 (A), R35.2
- new net: JP2.3 (B), R39.2
- new net CPU-D32: R27.2
- new net CPU-D33: R28.2
- new net IGN-3-OUT: JP3.2 (C)
- new net IGN-4-OUT: JP2.2 (C)
Other:
- moved on the sheet: D13, D14, R29, R30, R33, R34, R37, R38, R41, R42, U8

Commit message: restart a third time
Parts:
- removed D11, D12: LED, LED_SMD:LED_0603_1608Metric, symbol Device:LED
- removed JP2, JP3: Jumper_3_Open, Connector_PinHeader_2.54mm:PinHeader_1x03_P2.54mm_Vertical_SMD_Pin1Left, symbol Jumper:Jumper_3_Open
- removed R35, R36: 2.4k, Resistor_SMD:R_0603_1608Metric_Pad1.05x0.95mm_HandSolder, symbol Device:R
- removed R39, R40: 10, Resistor_SMD:R_0603_1608Metric_Pad1.05x0.95mm_HandSolder, symbol Device:R
- added D3, D4: LED, LED_SMD:LED_0603_1608Metric_Pad1.05x0.95mm_HandSolder, symbol Device:LED
- added R22, R23: 10, Resistor_SMD:R_0603_1608Metric_Pad0.98x0.95mm_HandSolder, symbol Device:R
- added R26, R27: 2.4k, Resistor_SMD:R_0603_1608Metric_Pad0.98x0.95mm_HandSolder, symbol Device:R
- D5: renamed from D13; footprint LED_SMD:LED_0603_1608Metric -> LED_SMD:LED_0603_1608Metric_Pad1.05x0.95mm_HandSolder
- D6: renamed from D14; footprint LED_SMD:LED_0603_1608Metric -> LED_SMD:LED_0603_1608Metric_Pad1.05x0.95mm_HandSolder
- R14: renamed from R27; footprint Resistor_SMD:R_0603_1608Metric_Pad1.05x0.95mm_HandSolder -> Resistor_SMD:R_0603_1608Metric_Pad0.98x0.95mm_HandSolder
- R15: renamed from R28; footprint Resistor_SMD:R_0603_1608Metric_Pad1.05x0.95mm_HandSolder -> Resistor_SMD:R_0603_1608Metric_Pad0.98x0.95mm_HandSolder
- R16: renamed from R29; footprint Resistor_SMD:R_0603_1608Metric_Pad1.05x0.95mm_HandSolder -> Resistor_SMD:R_0603_1608Metric_Pad0.98x0.95mm_HandSolder
- R17: renamed from R30; footprint Resistor_SMD:R_0603_1608Metric_Pad1.05x0.95mm_HandSolder -> Resistor_SMD:R_0603_1608Metric_Pad0.98x0.95mm_HandSolder
- R18: renamed from R31; footprint Resistor_SMD:R_0603_1608Metric_Pad1.05x0.95mm_HandSolder -> Resistor_SMD:R_0603_1608Metric_Pad0.98x0.95mm_HandSolder
- R19: renamed from R32; footprint Resistor_SMD:R_0603_1608Metric_Pad1.05x0.95mm_HandSolder -> Resistor_SMD:R_0603_1608Metric_Pad0.98x0.95mm_HandSolder
- R20: renamed from R33; footprint Resistor_SMD:R_0603_1608Metric_Pad1.05x0.95mm_HandSolder -> Resistor_SMD:R_0603_1608Metric_Pad0.98x0.95mm_HandSolder
- R21: renamed from R34; footprint Resistor_SMD:R_0603_1608Metric_Pad1.05x0.95mm_HandSolder -> Resistor_SMD:R_0603_1608Metric_Pad0.98x0.95mm_HandSolder
- R24: renamed from R41; footprint Resistor_SMD:R_0603_1608Metric_Pad1.05x0.95mm_HandSolder -> Resistor_SMD:R_0603_1608Metric_Pad0.98x0.95mm_HandSolder
- R25: renamed from R42; footprint Resistor_SMD:R_0603_1608Metric_Pad1.05x0.95mm_HandSolder -> Resistor_SMD:R_0603_1608Metric_Pad0.98x0.95mm_HandSolder
- R28: renamed from R37; footprint Resistor_SMD:R_0603_1608Metric_Pad1.05x0.95mm_HandSolder -> Resistor_SMD:R_0603_1608Metric_Pad0.98x0.95mm_HandSolder
- R29: renamed from R38; footprint Resistor_SMD:R_0603_1608Metric_Pad1.05x0.95mm_HandSolder -> Resistor_SMD:R_0603_1608Metric_Pad0.98x0.95mm_HandSolder
- renumbered U7 to U4, U8 to U5
Connections:
- net GND: now also D3.1 (K), D4.1 (K)
- net IGN-1-OUT: now also R24.1; no longer R24.2
- net IGN-2-OUT: now also R25.2; no longer R25.1
- net IGN-3-OUT: now also R22.1
- net IGN-4-OUT: now also R23.2
- net at U4.5 (OUT_B): now also R23.1, R27.2
- net at U4.7 (OUT_A): now also R22.2, R26.1
- net at R28.1, U5.7 (OUT_A): now also R24.2; no longer R24.1
- net at R29.2, U5.5 (OUT_B): now also R25.1; no longer R25.2
- net CPU-D32 renamed MCU-IGN-3
- net CPU-D33 renamed MCU-IGN-4
- net CPU-D39 renamed MCU-IGN-1
- net CPU-D41 renamed MCU-IGN-2
- new net: D4.2 (A), R27.1
- new net: D3.2 (A), R26.2
Other:
- moved on the sheet: D5, D6, R24, R25, R28, R29

Commit message: Changed ignition drivers, set the proper package and datasheet on them
Parts:
- removed U4, U5: TC4424A, Package_SO:SOIC-8_3.9x4.9mm_P1.27mm, symbol speeduino_ic_automotive:TC4424A
- added U3, U4, U5, U6: TC4422A, Package_DFN_QFN:DFN-8-1EP_6x5mm_P1.27mm_EP4x4mm, symbol Driver_FET:TC4422
Connections:
- wire segments 40 -> 56
Other:
- moved on the sheet: D3, D4, D5, R14, R15, R16, R18, R19, R20, R22, R23, R24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

Commit message: Changed ignitor names back to U?
Parts:
- renumbered U3 to U?, U4 to U?, U5 to U?, U6 to U?
Changed lines of the file:
@@
 	4400 4650 4800 4650
 $Comp
-L Driver_FET:TC4422 U3
+L Driver_FET:TC4422 U?
 U 1 1 6096AFF0
 P 3350 2050
-F 0 "U3" H 3894 2096 50  0000 L CNN
+F 0 "U?" H 3894 2096 50  0000 L CNN
 F 1 "TC4422A" H 3894 2005 50  0000 L CNN
 F 2 "Package_DFN_QFN:DFN-8-1EP_6x5mm_P1.27mm_EP4x4mm" H 3350 1250 50  0001 C CNN
@@
 	3350 1650 2750 1650
 $Comp
-L Driver_FET:TC4422 U4
+L Driver_FET:TC4422 U?
 U 1 1 60973F5E
 P 3350 3350
-F 0 "U4" H 3894 3396 50  0000 L CNN
+F 0 "U?" H 3894 3396 50  0000 L CNN
 F 1 "TC4422A" H 3894 3305 50  0000 L CNN
 F 2 "Package_DFN_QFN:DFN-8-1EP_6x5mm_P1.27mm_EP4x4mm" H 3350 2550 50  0001 C CNN
@@
 	3350 2950 2750 2950
 $Comp
-L Driver_FET:TC4422 U5
+L Driver_FET:TC4422 U?
 U 1 1 6098A9E1
 P 3350 4650
-F 0 "U5" H 3894 4696 50  0000 L CNN
+F 0 "U?" H 3894 4696 50  0000 L CNN
 F 1 "TC4422A" H 3894 4605 50  0000 L CNN
 F 2 "Package_DFN_QFN:DFN-8-1EP_6x5mm_P1.27mm_EP4x4mm" H 3350 3850 50  0001 C CNN
@@
 	3350 4250 2750 4250
 $Comp
-L Driver_FET:TC4422 U6
+L Driver_FET:TC4422 U?
 U 1 1 6098EF46
 P 3350 5950
-F 0 "U6" H 3894 5996 50  0000 L CNN
+F 0 "U?" H 3894 5996 50  0000 L CNN
 F 1 "TC4422A" H 3894 5905 50  0000 L CNN
 F 2 "Package_DFN_QFN:DFN-8-1EP_6x5mm_P1.27mm_EP4x4mm" H 3350 5150 50  0001 C CNN
